File: pcb_files/mouse/_saved_mouse.sch (KiCad schematic (older format))
At the start: 27 parts, among them M1 Motor_DC, M2 Motor_DC, M3 Motor_DC, Q0 Q_Photo_NPN, Q1 Q_Photo_NPN, Q2 Q_Photo_NPN, Q3 Q_Photo_NPN, U1 Teensy3.2, U2 SN754410NE, U3 LM1084-5.0, U4 Encoder_3081, U5 Encoder_3081, U6 NRF24L01_Breakout

Commit message: added status LEDs, buzzer
Parts:
- added D? (x2): LED, symbol Device:LED
- added R? (x3): R, symbol Device:R
Connections:
- net labels added: STATUS_LED_0, STATUS_LED_1
- wire segments 70 -> 74
Changed lines of the file:
@@
 	1    0    0    -1
 $EndComp
+$Comp
+L Device:R R?
+U 1 1 5D28EC87
+P 10150 2200
+F 0 "R?" V 9943 2200 50  0000 C CNN
+F 1 "R" V 10034 2200 50  0000 C CNN
+F 2 "" V 10080 2200 50  0001 C CNN
+F 3 "~" H 10150 2200 50  0001 C CNN
+	1    10150 2200
+	0    1    1    0
+$EndComp
+Wire Wire Line
+	10400 2200 10300 2200
+Text Label 10400 2400 2    50   ~ 0
+GND
+Wire Wire Line
+	9550 2550 9800 2550
+Wire Wire Line
+	9800 2550 9800 2200
+Wire Wire Line
+	9800 2200 10000 2200
+$Comp
+L Device:LED D?
+U 1 1 5D292553
+P 5900 3400
+F 0 "D?" H 5891 3616 50  0000 C CNN
+F 1 "LED" H 5900 3550 50  0000 C CNN
+F 2 "" H 5900 3400 50  0001 C CNN
+F 3 "~" H 5900 3400 50  0001 C CNN
+	1    5900 3400
+	0    -1   -1   0
+$EndComp
+$Comp
+L Device:R R?
+U 1 1 5D292B44
+P 5900 3100
+F 0 "R?" H 5830 3054 50  0000 R CNN
+F 1 "R" H 5830 3145 50  0000 R CNN
+F 2 "" V 5830 3100 50  0001 C CNN
+F 3 "~" H 5900 3100 50  0001 C CNN
+	1    5900 3100
+	-1   0    0    1
+$EndComp
+$Comp
+L Device:LED D?
+U 1 1 5D2990A5
+P 6300 3400
+F 0 "D?" H 6291 3616 50  0000 C CNN
+F 1 "LED" H 6300 3550 50  0000 C CNN
+F 2 "" H 6300 3400 50  0001 C CNN
+F 3 "~" H 6300 3400 50  0001 C CNN
+	1    6300 3400
+	0    -1   -1   0
+$EndComp
+$Comp
+L Device:R R?
+U 1 1 5D2990AB
+P 6300 3100
+F 0 "R?" H 6230 3054 50  0000 R CNN
+F 1 "R" H 6230 3145 50  0000 R CNN
+F 2 "" V 6230 3100 50  0001 C CNN
+F 3 "~" H 6300 3100 50  0001 C CNN
+	1    6300 3100
+	-1   0    0    1
+$EndComp
+Text Label 5900 2950 1    50   ~ 0
+STATUS_LED_0
+Text Label 6300 2950 1    50   ~ 0
+STATUS_LED_1
+Text Label 5900 3550 3    50   ~ 0
+GND
+Text Label 6300 3550 3    50   ~ 0
+GND
 $EndSCHEMATC
