File: pcb_files/mouse/_saved_mouse.sch (KiCad schematic (older format))
At the start: 66 parts, among them J2 BT_Conn, J4 I2C_Conn, M1 Motor_DC, M2 Motor_DC, M3 CASTER_BALL, Q0 Q_Photo_NPN, Q1 Q_Photo_NPN, Q2 Q_Photo_NPN, Q3 Q_Photo_NPN, SW1 SW_Push, T0 Q_NMOS_DGS, T1 Q_NMOS_DGS, T2 Q_NMOS_DGS, T3 Q_NMOS_DGS, U1 Teensy3.2, U2 SN754410NE, U4 Encoder_3081, U5 Encoder_3081, U6 LM2596S-5

Commit message: updates
Parts:
- removed D4: STATUS_0, misc:3528_SMD_LED, symbol Device:LED
- removed R18: R, Resistor_THT:R_Axial_DIN0309_L9.0mm_D3.2mm_P15.24mm_Horizontal, symbol Device:R
- added MH? (x4): M4, symbol Mechanical:MountingHole
- added R? (x2): 4.7k, symbol Device:R
- U4, U5: footprint Connector_PinSocket_2.54mm:PinSocket_1x06_P2.54mm_Vertical -> Connector_PinSocket_2.00mm:PinSocket_1x06_P2.00mm_Vertical
- gave numbers to parts that had none: 6
Connections:
- net labels removed: STATUS_LED_0
- wire segments 136 -> 142
Changed lines of the file:
@@
 F 0 "U4" H 3000 10317 50  0000 C CNN
 F 1 "Encoder_3081" H 3000 10226 50  0000 C CNN
-F 2 "Connector_PinSocket_2.54mm:PinSocket_1x06_P2.54mm_Vertical" H 3150 9200 50  0001 L CNN
+F 2 "Connector_PinSocket_2.00mm:PinSocket_1x06_P2.00mm_Vertical" H 3150 9200 50  0001 L CNN
 F 3 "http://ams.com/eng/content/download/438063/1340357/246195" H 850 11300 50  0001 C CNN
 	1    3000 9700
@@
 F 0 "U5" H 3000 9017 50  0000 C CNN
 F 1 "Encoder_3081" H 3000 8926 50  0000 C CNN
-F 2 "Connector_PinSocket_2.54mm:PinSocket_1x06_P2.54mm_Vertical" H 3150 7900 50  0001 L CNN
+F 2 "Connector_PinSocket_2.00mm:PinSocket_1x06_P2.00mm_Vertical" H 3150 7900 50  0001 L CNN
 F 3 "http://ams.com/eng/content/download/438063/1340357/246195" H 850 10000 50  0001 C CNN
 	1    3000 8400
@@
 	15200 6700 15200 6900
 $Comp
-L Device:LED D4
-U 1 1 5D292553
-P 14300 7500
-F 0 "D4" H 14291 7716 50  0000 C CNN
-F 1 "STATUS_0" H 14300 7650 50  0000 C CNN
-F 2 "misc:3528_SMD_LED" H 14300 7500 50  0001 C CNN
-F 3 "~" H 14300 7500 50  0001 C CNN
-	1    14300 7500
-	0    -1   -1   0
-$EndComp
-$Comp
-L Device:R R18
-U 1 1 5D292B44
-P 14300 7200
-F 0 "R18" H 14230 7154 50  0000 R CNN
-F 1 "R" H 14230 7245 50  0000 R CNN
-F 2 "Resistor_THT:R_Axial_DIN0309_L9.0mm_D3.2mm_P15.24mm_Horizontal" V 14230 7200 50  0001 C CNN
-F 3 "~" H 14300 7200 50  0001 C CNN
-	1    14300 7200
-	-1   0    0    1
-$EndComp
-$Comp
 L Device:LED D5
 U 1 1 5D2990A5
@@
 	-1   0    0    1
 $EndComp
-Text Label 14300 7050 1    50   ~ 0
-STATUS_LED_0
 Text Label 14700 7050 1    50   ~ 0
 STATUS_LED_1
-Text Label 14300 7650 3    50   ~ 0
-GND
 Text Label 14700 7650 3    50   ~ 0
 GND
 Text Label 7650 5100 2    50   ~ 0
-STATUS_LED_0
+RGB_DATA
 Text Label 7650 5200 2    50   ~ 0
 STATUS_LED_1
@@
 Text Label 7650 6500 2    50   ~ 0
 i2c_SCL
-Text Label 13600 7250 0    50   ~ 0
+Text Label 13975 7250 0    50   ~ 0
 i2c_SCL
 Text Label 13600 7750 0    50   ~ 0
@@
 	1    0    0    -1
 $EndComp
-Text Label 13600 7350 0    50   ~ 0
+Text Label 13950 7350 0    50   ~ 0
 i2c_SDA
 $Comp
@@
 $EndComp
 $Comp
-L mouse-rescue:EG1218-dk_Slide-Switches S?
+L mouse-rescue:EG1218-dk_Slide-Switches S1
 U 1 1 5E819689
 P 12250 1775
-F 0 "S?" H 12250 2054 50  0000 C CNN
+F 0 "S1" H 12250 2054 50  0000 C CNN
 F 1 "EG1218" H 12250 1963 50  0000 C CNN
 F 2 "misc:Switch_amazon" H 12450 1975 50  0001 L CNN
@@
 $EndComp
 $Comp
-L Device:Battery_Cell BT?
+L Device:Battery_Cell BT1
 U 1 1 5E820C97
 P 11950 2225
-F 0 "BT?" H 11700 2325 50  0000 L CNN
+F 0 "BT1" H 11700 2325 50  0000 L CNN
 F 1 "Battery_Cell" H 11400 2225 50  0000 L CNN
 F 2 "Connector_PinSocket_2.54mm:PinSocket_1x02_P2.54mm_Vertical" V 11950 2285 50  0001 C CNN
@@
 5v
 $Comp
-L Device:L L?
+L Device:L L1
 U 1 1 5E8A9E63
 P 14400 2075
-F 0 "L?" V 14590 2075 50  0000 C CNN
+F 0 "L1" V 14590 2075 50  0000 C CNN
 F 1 "33uH" V 14499 2075 50  0000 C CNN
 F 2 "" H 14400 2075 50  0001 C CNN
@@
 	14800 2075 14700 2075
 $Comp
-L Device:D_Schottky D?
+L Device:D_Schottky D12
 U 1 1 5E8B6F40
 P 14150 2225
-F 0 "D?" V 14104 2304 50  0000 L CNN
+F 0 "D12" V 14104 2304 50  0000 L CNN
 F 1 "1n5824" V 14195 2304 50  0000 L CNN
 F 2 "" H 14150 2225 50  0001 C CNN
@@
 GND
 $Comp
-L Device:CP1 C?
+L Device:CP1 C10
 U 1 1 5E8B972D
 P 14700 2225
-F 0 "C?" H 14815 2271 50  0000 L CNN
+F 0 "C10" H 14815 2271 50  0000 L CNN
 F 1 "220uF" H 14815 2180 50  0000 L CNN
 F 2 "" H 14700 2225 50  0001 C CNN
@@
 	14700 2075 14550 2075
 $Comp
-L Device:CP1 C?
+L Device:CP1 C9
 U 1 1 5E8BA3C3
 P 12700 2025
-F 0 "C?" H 12500 1975 50  0000 L CNN
+F 0 "C9" H 12500 1975 50  0000 L CNN
 F 1 "680uF" H 12450 1875 50  0000 L CNN
 F 2 "" H 12700 2025 50  0001 C CNN
@@
 NoConn ~ 1675 7050
 NoConn ~ 1675 7550
+Wire Wire Line
+	13600 7350 13700 7350
+Wire Wire Line
+	13600 7250 13900 7250
+Wire Wire Line
+	13900 7250 13900 7000
+Connection ~ 13900 7250
+Wire Wire Line
+	13900 7250 13975 7250
+Wire Wire Line
+	13700 7350 13700 7050
+Connection ~ 13700 7350
+Wire Wire Line
+	13700 7350 13950 7350
+$Comp
+L Device:R R?
+U 1 1 5E798BF8
+P 13700 6900
+F 0 "R?" H 13525 6950 50  0000 L CNN
+F 1 "4.7k" H 13475 6850 50  0000 L CNN
+F 2 "" V 13630 6900 50  0001 C CNN
+F 3 "~" H 13700 6900 50  0001 C CNN
+	1    13700 6900
+	1    0    0    -1
+$EndComp
+$Comp
+L Device:R R?
+U 1 1 5E798D08
+P 13900 6850
+F 0 "R?" H 13970 6896 50  0000 L CNN
+F 1 "4.7k" H 13970 6805 50  0000 L CNN
+F 2 "" V 13830 6850 50  0001 C CNN
+F 3 "~" H 13900 6850 50  0001 C CNN
+	1    13900 6850
+	1    0    0    -1
+$EndComp
+$Comp
+L Mechanical:MountingHole MH?
+U 1 1 5E799FC8
+P 14800 5875
+F 0 "MH?" H 14900 5921 50  0000 L CNN
+F 1 "M4" H 14900 5830 50  0000 L CNN
+F 2 "" H 14800 5875 50  0001 C CNN
+F 3 "~" H 14800 5875 50  0001 C CNN
+	1    14800 5875
+	1    0    0    -1
+$EndComp
+$Comp
+L Mechanical:MountingHole MH?
+U 1 1 5E79A0A3
+P 13975 5900
+F 0 "MH?" H 14075 5946 50  0000 L CNN
+F 1 "M4" H 14075 5855 50  0000 L CNN
+F 2 "" H 13975 5900 50  0001 C CNN
+F 3 "~" H 13975 5900 50  0001 C CNN
+	1    13975 5900
+	1    0    0    -1
+$EndComp
+$Comp
+L Mechanical:MountingHole MH?
+U 1 1 5E79A15B
+P 13975 5500
+F 0 "MH?" H 14075 5546 50  0000 L CNN
+F 1 "M4" H 14075 5455 50  0000 L CNN
+F 2 "" H 13975 5500 50  0001 C CNN
+F 3 "~" H 13975 5500 50  0001 C CNN
+	1    13975 5500
+	1    0    0    -1
+$EndComp
+$Comp
+L Mechanical:MountingHole MH?
+U 1 1 5E79A200
+P 14800 5500
+F 0 "MH?" H 14900 5546 50  0000 L CNN
+F 1 "M4" H 14900 5455 50  0000 L CNN
+F 2 "" H 14800 5500 50  0001 C CNN
+F 3 "~" H 14800 5500 50  0001 C CNN
+	1    14800 5500
+	1    0    0    -1
+$EndComp
 $EndSCHEMATC
