File: pcb_files/mouse/_saved_mouse.sch (KiCad schematic (older format))
At the start: 72 parts, among them J2 BT_Conn, J4 I2C_Conn, M1 Motor_DC, M2 Motor_DC, M3 CASTER_BALL, Q0 Q_Photo_NPN, Q1 Q_Photo_NPN, Q2 Q_Photo_NPN, Q3 Q_Photo_NPN, SW1 TL3315NF160Q, SW2 TL3315NF160Q, T0 Q_NMOS_DGS, T1 Q_NMOS_DGS, T2 Q_NMOS_DGS, T3 Q_NMOS_DGS, U1 Teensy3.2, U2 SN754410NE, U3 LM1084-5.0, U4 Encoder_3081, U5 Encoder_3081

Commit message: reworked mouse shape
Parts:
- MH1, MH2, MH3, MH4: value M4 -> M3
- R1, R10, R11, R12, R13, R14, R15, R16, R2, R3, R4, R5, R6, R7, R8, R9: footprint Resistor_THT:R_Axial_DIN0309_L9.0mm_D3.2mm_P12.70mm_Horizontal -> Resistor_SMD:R_1206_3216Metric_Pad1.42x1.75mm_HandSolder
Changed lines of the file:
@@
 F 0 "R8" H 6020 1396 50  0000 L CNN
 F 1 "33" H 6020 1305 50  0000 L CNN
-F 2 "Resistor_THT:R_Axial_DIN0309_L9.0mm_D3.2mm_P12.70mm_Horizontal" V 5880 1350 50  0001 C CNN
+F 2 "Resistor_SMD:R_1206_3216Metric_Pad1.42x1.75mm_HandSolder" V 5880 1350 50  0001 C CNN
 F 3 "~" H 5950 1350 50  0001 C CNN
 	1    5950 1350
@@
 F 0 "R1" H 1490 3506 50  0000 L CNN
 F 1 "R" H 1490 3415 50  0000 L CNN
-F 2 "Resistor_THT:R_Axial_DIN0309_L9.0mm_D3.2mm_P12.70mm_Horizontal" V 1350 3460 50  0001 C CNN
+F 2 "Resistor_SMD:R_1206_3216Metric_Pad1.42x1.75mm_HandSolder" V 1350 3460 50  0001 C CNN
 F 3 "~" H 1420 3460 50  0001 C CNN
 	1    1420 3460
@@
 F 0 "R2" H 2390 3506 50  0000 L CNN
 F 1 "R" H 2390 3415 50  0000 L CNN
-F 2 "Resistor_THT:R_Axial_DIN0309_L9.0mm_D3.2mm_P12.70mm_Horizontal" V 2250 3460 50  0001 C CNN
+F 2 "Resistor_SMD:R_1206_3216Metric_Pad1.42x1.75mm_HandSolder" V 2250 3460 50  0001 C CNN
 F 3 "~" H 2320 3460 50  0001 C CNN
 	1    2320 3460
@@
 F 0 "R3" H 3290 3506 50  0000 L CNN
 F 1 "R" H 3290 3415 50  0000 L CNN
-F 2 "Resistor_THT:R_Axial_DIN0309_L9.0mm_D3.2mm_P12.70mm_Horizontal" V 3150 3460 50  0001 C CNN
+F 2 "Resistor_SMD:R_1206_3216Metric_Pad1.42x1.75mm_HandSolder" V 3150 3460 50  0001 C CNN
 F 3 "~" H 3220 3460 50  0001 C CNN
 	1    3220 3460
@@
 F 0 "R4" H 4140 3506 50  0000 L CNN
 F 1 "R" H 4140 3415 50  0000 L CNN
-F 2 "Resistor_THT:R_Axial_DIN0309_L9.0mm_D3.2mm_P12.70mm_Horizontal" V 4000 3460 50  0001 C CNN
+F 2 "Resistor_SMD:R_1206_3216Metric_Pad1.42x1.75mm_HandSolder" V 4000 3460 50  0001 C CNN
 F 3 "~" H 4070 3460 50  0001 C CNN
 	1    4070 3460
@@
 F 0 "R16" V 5593 2200 50  0000 C CNN
 F 1 "47k" V 5684 2200 50  0000 C CNN
-F 2 "Resistor_THT:R_Axial_DIN0309_L9.0mm_D3.2mm_P12.70mm_Horizontal" V 5730 2200 50  0001 C CNN
+F 2 "Resistor_SMD:R_1206_3216Metric_Pad1.42x1.75mm_HandSolder" V 5730 2200 50  0001 C CNN
 F 3 "~" H 5800 2200 50  0001 C CNN
 	1    5800 2200
@@
 F 0 "R12" V 5193 1800 50  0000 C CNN
 F 1 "1k" V 5284 1800 50  0000 C CNN
-F 2 "Resistor_THT:R_Axial_DIN0309_L9.0mm_D3.2mm_P12.70mm_Horizontal" V 5330 1800 50  0001 C CNN
+F 2 "Resistor_SMD:R_1206_3216Metric_Pad1.42x1.75mm_HandSolder" V 5330 1800 50  0001 C CNN
 F 3 "~" H 5400 1800 50  0001 C CNN
 	1    5400 1800
@@
 F 0 "R7" H 4520 1396 50  0000 L CNN
 F 1 "33" H 4520 1305 50  0000 L CNN
-F 2 "Resistor_THT:R_Axial_DIN0309_L9.0mm_D3.2mm_P12.70mm_Horizontal" V 4380 1350 50  0001 C CNN
+F 2 "Resistor_SMD:R_1206_3216Metric_Pad1.42x1.75mm_HandSolder" V 4380 1350 50  0001 C CNN
 F 3 "~" H 4450 1350 50  0001 C CNN
 	1    4450 1350
@@
 F 0 "R15" V 4093 2200 50  0000 C CNN
 F 1 "47k" V 4184 2200 50  0000 C CNN
-F 2 "Resistor_THT:R_Axial_DIN0309_L9.0mm_D3.2mm_P12.70mm_Horizontal" V 4230 2200 50  0001 C CNN
+F 2 "Resistor_SMD:R_1206_3216Metric_Pad1.42x1.75mm_HandSolder" V 4230 2200 50  0001 C CNN
 F 3 "~" H 4300 2200 50  0001 C CNN
 	1    4300 2200
@@
 F 0 "R11" V 3693 1800 50  0000 C CNN
 F 1 "1k" V 3784 1800 50  0000 C CNN
-F 2 "Resistor_THT:R_Axial_DIN0309_L9.0mm_D3.2mm_P12.70mm_Horizontal" V 3830 1800 50  0001 C CNN
+F 2 "Resistor_SMD:R_1206_3216Metric_Pad1.42x1.75mm_HandSolder" V 3830 1800 50  0001 C CNN
 F 3 "~" H 3900 1800 50  0001 C CNN
 	1    3900 1800
@@
 F 0 "R5" H 1520 1396 50  0000 L CNN
 F 1 "33" H 1520 1305 50  0000 L CNN
-F 2 "Resistor_THT:R_Axial_DIN0309_L9.0mm_D3.2mm_P12.70mm_Horizontal" V 1380 1350 50  0001 C CNN
+F 2 "Resistor_SMD:R_1206_3216Metric_Pad1.42x1.75mm_HandSolder" V 1380 1350 50  0001 C CNN
 F 3 "~" H 1450 1350 50  0001 C CNN
 	1    1450 1350
@@
 F 0 "R13" V 1093 2200 50  0000 C CNN
 F 1 "47k" V 1184 2200 50  0000 C CNN
-F 2 "Resistor_THT:R_Axial_DIN0309_L9.0mm_D3.2mm_P12.70mm_Horizontal" V 1230 2200 50  0001 C CNN
+F 2 "Resistor_SMD:R_1206_3216Metric_Pad1.42x1.75mm_HandSolder" V 1230 2200 50  0001 C CNN
 F 3 "~" H 1300 2200 50  0001 C CNN
 	1    1300 2200
@@
 F 0 "R9" V 693 1800 50  0000 C CNN
 F 1 "1k" V 784 1800 50  0000 C CNN
-F 2 "Resistor_THT:R_Axial_DIN0309_L9.0mm_D3.2mm_P12.70mm_Horizontal" V 830 1800 50  0001 C CNN
+F 2 "Resistor_SMD:R_1206_3216Metric_Pad1.42x1.75mm_HandSolder" V 830 1800 50  0001 C CNN
 F 3 "~" H 900 1800 50  0001 C CNN
 	1    900  1800
@@
 F 0 "R6" H 3020 1396 50  0000 L CNN
 F 1 "33" H 3020 1305 50  0000 L CNN
-F 2 "Resistor_THT:R_Axial_DIN0309_L9.0mm_D3.2mm_P12.70mm_Horizontal" V 2880 1350 50  0001 C CNN
+F 2 "Resistor_SMD:R_1206_3216Metric_Pad1.42x1.75mm_HandSolder" V 2880 1350 50  0001 C CNN
 F 3 "~" H 2950 1350 50  0001 C CNN
 	1    2950 1350
@@
 F 0 "R14" V 2593 2200 50  0000 C CNN
 F 1 "47k" V 2684 2200 50  0000 C CNN
-F 2 "Resistor_THT:R_Axial_DIN0309_L9.0mm_D3.2mm_P12.70mm_Horizontal" V 2730 2200 50  0001 C CNN
+F 2 "Resistor_SMD:R_1206_3216Metric_Pad1.42x1.75mm_HandSolder" V 2730 2200 50  0001 C CNN
 F 3 "~" H 2800 2200 50  0001 C CNN
 	1    2800 2200
@@
 F 0 "R10" V 2193 1800 50  0000 C CNN
 F 1 "1k" V 2284 1800 50  0000 C CNN
-F 2 "Resistor_THT:R_Axial_DIN0309_L9.0mm_D3.2mm_P12.70mm_Horizontal" V 2330 1800 50  0001 C CNN
+F 2 "Resistor_SMD:R_1206_3216Metric_Pad1.42x1.75mm_HandSolder" V 2330 1800 50  0001 C CNN
 F 3 "~" H 2400 1800 50  0001 C CNN
 	1    2400 1800
@@
 P 14800 5875
 F 0 "MH4" H 14900 5921 50  0000 L CNN
-F 1 "M4" H 14900 5830 50  0000 L CNN
+F 1 "M3" H 14900 5830 50  0000 L CNN
 F 2 "MountingHole:MountingHole_3.2mm_M3" H 14800 5875 50  0001 C CNN
 F 3 "~" H 14800 5875 50  0001 C CNN
@@
 P 13975 5900
 F 0 "MH2" H 14075 5946 50  0000 L CNN
-F 1 "M4" H 14075 5855 50  0000 L CNN
+F 1 "M3" H 14075 5855 50  0000 L CNN
 F 2 "MountingHole:MountingHole_3.2mm_M3" H 13975 5900 50  0001 C CNN
 F 3 "~" H 13975 5900 50  0001 C CNN
@@
 P 13975 5500
 F 0 "MH1" H 14075 5546 50  0000 L CNN
-F 1 "M4" H 14075 5455 50  0000 L CNN
+F 1 "M3" H 14075 5455 50  0000 L CNN
 F 2 "MountingHole:MountingHole_3.2mm_M3" H 13975 5500 50  0001 C CNN
 F 3 "~" H 13975 5500 50  0001 C CNN
@@
 P 14800 5500
 F 0 "MH3" H 14900 5546 50  0000 L CNN
-F 1 "M4" H 14900 5455 50  0000 L CNN
+F 1 "M3" H 14900 5455 50  0000 L CNN
 F 2 "MountingHole:MountingHole_3.2mm_M3" H 14800 5500 50  0001 C CNN
 F 3 "~" H 14800 5500 50  0001 C CNN
