File: pcb_files/mouse/mouse.sch (KiCad schematic (older format))
At the start: 32 parts, among them M1 Motor_DC, M2 Motor_DC, M3 CASTER_BALL, Q0 Q_Photo_NPN, Q1 Q_Photo_NPN, Q2 Q_Photo_NPN, Q3 Q_Photo_NPN, U1 Teensy3.2, U2 SN754410NE, U3 LM1084-5.0, U4 Encoder_3081, U5 Encoder_3081, U6 NRF24L01_Breakout

Commit message: removed wirless module
Parts:
- removed U6: NRF24L01_Breakout, Connector_PinSocket_2.54mm:PinSocket_2x04_P2.54mm_Vertical, symbol RF:NRF24L01_Breakout
- added R?: R, symbol Device:R
- added SW?: SW_Push, symbol Switch:SW_Push
Connections:
- net labels removed: Emiter_2, u1_CE, u1_CS, u1_MISO, u1_MOSI, u1_SCK
- wire segments 72 -> 77
Changed lines of the file:
@@
 EESchema Schematic File Version 4
 LIBS:mouse-cache
-EELAYER 26 0
+EELAYER 29 0
 EELAYER END
 $Descr A4 11693 8268
@@
 $EndComp
 $Comp
-L RF:NRF24L01_Breakout U6
-U 1 1 5D1C0351
-P 6400 1750
-F 0 "U6" H 6878 1728 50  0000 L CNN
-F 1 "NRF24L01_Breakout" H 6878 1637 50  0000 L CNN
-F 2 "Connector_PinSocket_2.54mm:PinSocket_2x04_P2.54mm_Vertical" H 6550 2350 50  0001 L CIN
-F 3 "http://www.nordicsemi.com/eng/content/download/2730/34105/file/nRF24L01_Product_Specification_v2_0.pdf" H 6400 1650 50  0001 C CNN
-	1    6400 1750
-	1    0    0    -1
-$EndComp
-$Comp
 L Device:Battery_Cell BT1
 U 1 1 5D1C070D
@@
 Wire Wire Line
 	10250 6200 9000 6200
-Text Label 6400 1150 0    50   ~ 0
-3.3v
 Text Label 7550 3450 2    50   ~ 0
 3.3v
-Text Label 6400 2350 0    50   ~ 0
-GND
-Text Label 7550 3250 2    50   ~ 0
-u1_MISO
-Text Label 7550 3150 2    50   ~ 0
-u1_MOSI
-Text Label 7550 3850 2    50   ~ 0
-u1_SCK
-Text Label 7550 3050 2    50   ~ 0
-u1_CS
-Text Label 7550 2950 2    50   ~ 0
-u1_CE
-Text Label 5900 1450 2    50   ~ 0
-u1_MOSI
-Text Label 5900 1550 2    50   ~ 0
-u1_MISO
-Text Label 5900 1650 2    50   ~ 0
-u1_SCK
-Text Label 5900 1750 2    50   ~ 0
-u1_CS
-Text Label 5900 1950 2    50   ~ 0
-u1_CE
 Text Label 4300 5100 2    50   ~ 0
 5v
@@
 Emitter_1
 Text Label 2550 1450 3    50   ~ 0
-Emiter_2
+Emitter_2
 Text Label 3050 1450 3    50   ~ 0
 Emitter_3
@@
 Text Label 7550 2550 2    50   ~ 0
 Buzzer
+Text Label 7550 2750 2    50   ~ 0
+M1_forward
+Text Label 7550 2850 2    50   ~ 0
+M1_backward
+Text Label 7550 2950 2    50   ~ 0
+M2_forward
+Text Label 7550 3050 2    50   ~ 0
+M2_backward
+$Comp
+L Switch:SW_Push SW?
+U 1 1 5D2BB906
+P 6270 2200
+F 0 "SW?" H 6270 2485 50  0000 C CNN
+F 1 "SW_Push" H 6270 2394 50  0000 C CNN
+F 2 "" H 6270 2400 50  0001 C CNN
+F 3 "~" H 6270 2400 50  0001 C CNN
+	1    6270 2200
+	1    0    0    -1
+$EndComp
+Wire Wire Line
+	7550 2250 7460 2250
+Wire Wire Line
+	7460 2250 7460 1990
+Wire Wire Line
+	7460 1990 6470 1990
+Wire Wire Line
+	6470 1990 6470 2200
+Text Label 6070 2200 2    50   ~ 0
+3.3v
+Wire Wire Line
+	6470 2200 6470 2270
+Connection ~ 6470 2200
+$Comp
+L Device:R R?
+U 1 1 5D2C4CD1
+P 6470 2420
+F 0 "R?" H 6540 2466 50  0000 L CNN
+F 1 "R" H 6540 2375 50  0000 L CNN
+F 2 "" V 6400 2420 50  0001 C CNN
+F 3 "~" H 6470 2420 50  0001 C CNN
+	1    6470 2420
+	1    0    0    -1
+$EndComp
+Text Label 6470 2570 3    50   ~ 0
+GND
 $EndSCHEMATC

Commit message: update
Parts:
- added MH_GND, MH_SCL, MH_SDA, MH_vBatt: MountingHole_Pad, symbol Mechanical:MountingHole_Pad
Connections:
- net labels added: i2c_SCL, i2c_SDA
Changed lines of the file:
@@
 EESchema Schematic File Version 4
 LIBS:mouse-cache
-EELAYER 29 0
+EELAYER 26 0
 EELAYER END
 $Descr A4 11693 8268
@@
 Text Label 7550 4250 2    50   ~ 0
 Reciever_3
-Text Label 7550 4350 2    50   ~ 0
+Text Label 7550 3150 2    50   ~ 0
 Emitter_0
 Connection ~ 9000 6200
@@
 Text Label 7700 6200 2    50   ~ 0
 5v
-Text Label 7550 4450 2    50   ~ 0
+Text Label 7550 3250 2    50   ~ 0
 Emitter_1
 Text Label 7550 4550 2    50   ~ 0
@@
 Text Label 6470 2570 3    50   ~ 0
 GND
+$Comp
+L Mechanical:MountingHole_Pad MH_SCL
+U 1 1 5D2CDA5E
+P 5550 1300
+F 0 "MH_SCL" V 5504 1450 50  0000 L CNN
+F 1 "MountingHole_Pad" V 5595 1450 50  0000 L CNN
+F 2 "" H 5550 1300 50  0001 C CNN
+F 3 "~" H 5550 1300 50  0001 C CNN
+	1    5550 1300
+	0    1    1    0
+$EndComp
+$Comp
+L Mechanical:MountingHole_Pad MH_SDA
+U 1 1 5D2CDD65
+P 5550 1050
+F 0 "MH_SDA" V 5504 1200 50  0000 L CNN
+F 1 "MountingHole_Pad" V 5595 1200 50  0000 L CNN
+F 2 "" H 5550 1050 50  0001 C CNN
+F 3 "~" H 5550 1050 50  0001 C CNN
+	1    5550 1050
+	0    1    1    0
+$EndComp
+Text Label 7550 4350 2    50   ~ 0
+i2c_SDA
+Text Label 7550 4450 2    50   ~ 0
+i2c_SCL
+Text Label 5450 1050 2    50   ~ 0
+i2c_SDA
+Text Label 5450 1300 2    50   ~ 0
+i2c_SCL
+$Comp
+L Mechanical:MountingHole_Pad MH_GND
+U 1 1 5D2D0AFA
+P 5550 1550
+F 0 "MH_GND" V 5504 1700 50  0000 L CNN
+F 1 "MountingHole_Pad" V 5595 1700 50  0000 L CNN
+F 2 "" H 5550 1550 50  0001 C CNN
+F 3 "~" H 5550 1550 50  0001 C CNN
+	1    5550 1550
+	0    1    1    0
+$EndComp
+$Comp
+L Mechanical:MountingHole_Pad MH_vBatt
+U 1 1 5D2D0CC0
+P 5550 800
+F 0 "MH_vBatt" V 5504 950 50  0000 L CNN
+F 1 "MountingHole_Pad" V 5595 950 50  0000 L CNN
+F 2 "" H 5550 800 50  0001 C CNN
+F 3 "~" H 5550 800 50  0001 C CNN
+	1    5550 800
+	0    1    1    0
+$EndComp
+Text Label 5450 800  2    50   ~ 0
+vBatt
+Text Label 5450 1550 2    50   ~ 0
+GND
 $EndSCHEMATC

Commit message: update
Parts:
- gave numbers to parts that had none: 2
- renumbered MH_GND to MH_GND1, MH_SCL to MH_SCL1, MH_SDA to MH_SDA1, MH_vBatt to MH_vBatt1
Changed lines of the file:
@@
 M2_backward
 $Comp
-L Switch:SW_Push SW?
+L Switch:SW_Push SW1
 U 1 1 5D2BB906
 P 6270 2200
-F 0 "SW?" H 6270 2485 50  0000 C CNN
+F 0 "SW1" H 6270 2485 50  0000 C CNN
 F 1 "SW_Push" H 6270 2394 50  0000 C CNN
 F 2 "" H 6270 2400 50  0001 C CNN
@@
 Connection ~ 6470 2200
 $Comp
-L Device:R R?
+L Device:R R11
 U 1 1 5D2C4CD1
 P 6470 2420
-F 0 "R?" H 6540 2466 50  0000 L CNN
+F 0 "R11" H 6540 2466 50  0000 L CNN
 F 1 "R" H 6540 2375 50  0000 L CNN
 F 2 "" V 6400 2420 50  0001 C CNN
@@
 GND
 $Comp
-L Mechanical:MountingHole_Pad MH_SCL
+L Mechanical:MountingHole_Pad MH_SCL1
 U 1 1 5D2CDA5E
 P 5550 1300
-F 0 "MH_SCL" V 5504 1450 50  0000 L CNN
+F 0 "MH_SCL1" V 5504 1450 50  0000 L CNN
 F 1 "MountingHole_Pad" V 5595 1450 50  0000 L CNN
 F 2 "" H 5550 1300 50  0001 C CNN
@@
 $EndComp
 $Comp
-L Mechanical:MountingHole_Pad MH_SDA
+L Mechanical:MountingHole_Pad MH_SDA1
 U 1 1 5D2CDD65
 P 5550 1050
-F 0 "MH_SDA" V 5504 1200 50  0000 L CNN
+F 0 "MH_SDA1" V 5504 1200 50  0000 L CNN
 F 1 "MountingHole_Pad" V 5595 1200 50  0000 L CNN
 F 2 "" H 5550 1050 50  0001 C CNN
@@
 i2c_SCL
 $Comp
-L Mechanical:MountingHole_Pad MH_GND
+L Mechanical:MountingHole_Pad MH_GND1
 U 1 1 5D2D0AFA
 P 5550 1550
-F 0 "MH_GND" V 5504 1700 50  0000 L CNN
+F 0 "MH_GND1" V 5504 1700 50  0000 L CNN
 F 1 "MountingHole_Pad" V 5595 1700 50  0000 L CNN
 F 2 "" H 5550 1550 50  0001 C CNN
@@
 $EndComp
 $Comp
-L Mechanical:MountingHole_Pad MH_vBatt
+L Mechanical:MountingHole_Pad MH_vBatt1
 U 1 1 5D2D0CC0
 P 5550 800
-F 0 "MH_vBatt" V 5504 950 50  0000 L CNN
+F 0 "MH_vBatt1" V 5504 950 50  0000 L CNN
 F 1 "MountingHole_Pad" V 5595 950 50  0000 L CNN
 F 2 "" H 5550 800 50  0001 C CNN
