File: pcb_files/mouse/mouse.sch (KiCad schematic (older format))
At the start: 49 parts, among them M1 Motor_DC, M2 Motor_DC, M3 CASTER_BALL, Q0 Q_NMOS_DGS, Q0 Q_Photo_NPN, Q1 Q_NMOS_DGS, Q1 Q_Photo_NPN, Q2 Q_NMOS_DGS, Q2 Q_Photo_NPN, Q3 Q_NMOS_DGS, Q3 Q_Photo_NPN, SW1 SW_Push, U1 Teensy3.2, U2 SN754410NE, U3 LM1084-5.0, U4 Encoder_3081, U5 Encoder_3081

Commit message: started new pcb
Parts:
- R1, R17, R18, R19, R2, R20, R3, R4, R5, R6, R7, R8: footprint Resistor_THT:R_Axial_DIN0207_L6.3mm_D2.5mm_P2.54mm_Vertical -> Resistor_THT:R_Axial_DIN0309_L9.0mm_D3.2mm_P15.24mm_Horizontal
- R10, R11, R12, R13, R14, R15, R16, R9: footprint (none) -> Resistor_THT:R_Axial_DIN0309_L9.0mm_D3.2mm_P15.24mm_Horizontal
- T0: renamed from Q0; footprint (none) -> misc:TN0104(TO-92)
- T1: renamed from Q1; footprint (none) -> misc:TN0104(TO-92)
- T2: renamed from Q2; footprint (none) -> misc:TN0104(TO-92)
- T3: renamed from Q3; footprint (none) -> misc:TN0104(TO-92)
Changed lines of the file:
@@
 F 0 "R8" H 6020 1396 50  0000 L CNN
 F 1 "33" H 6020 1305 50  0000 L CNN
-F 2 "Resistor_THT:R_Axial_DIN0207_L6.3mm_D2.5mm_P2.54mm_Vertical" V 5880 1350 50  0001 C CNN
+F 2 "Resistor_THT:R_Axial_DIN0309_L9.0mm_D3.2mm_P15.24mm_Horizontal" V 5880 1350 50  0001 C CNN
 F 3 "~" H 5950 1350 50  0001 C CNN
 	1    5950 1350
@@
 F 0 "R1" H 1490 3506 50  0000 L CNN
 F 1 "R" H 1490 3415 50  0000 L CNN
-F 2 "Resistor_THT:R_Axial_DIN0207_L6.3mm_D2.5mm_P2.54mm_Vertical" V 1350 3460 50  0001 C CNN
+F 2 "Resistor_THT:R_Axial_DIN0309_L9.0mm_D3.2mm_P15.24mm_Horizontal" V 1350 3460 50  0001 C CNN
 F 3 "~" H 1420 3460 50  0001 C CNN
 	1    1420 3460
@@
 F 0 "R2" H 2390 3506 50  0000 L CNN
 F 1 "R" H 2390 3415 50  0000 L CNN
-F 2 "Resistor_THT:R_Axial_DIN0207_L6.3mm_D2.5mm_P2.54mm_Vertical" V 2250 3460 50  0001 C CNN
+F 2 "Resistor_THT:R_Axial_DIN0309_L9.0mm_D3.2mm_P15.24mm_Horizontal" V 2250 3460 50  0001 C CNN
 F 3 "~" H 2320 3460 50  0001 C CNN
 	1    2320 3460
@@
 F 0 "R3" H 3290 3506 50  0000 L CNN
 F 1 "R" H 3290 3415 50  0000 L CNN
-F 2 "Resistor_THT:R_Axial_DIN0207_L6.3mm_D2.5mm_P2.54mm_Vertical" V 3150 3460 50  0001 C CNN
+F 2 "Resistor_THT:R_Axial_DIN0309_L9.0mm_D3.2mm_P15.24mm_Horizontal" V 3150 3460 50  0001 C CNN
 F 3 "~" H 3220 3460 50  0001 C CNN
 	1    3220 3460
@@
 F 0 "R4" H 4140 3506 50  0000 L CNN
 F 1 "R" H 4140 3415 50  0000 L CNN
-F 2 "Resistor_THT:R_Axial_DIN0207_L6.3mm_D2.5mm_P2.54mm_Vertical" V 4000 3460 50  0001 C CNN
+F 2 "Resistor_THT:R_Axial_DIN0309_L9.0mm_D3.2mm_P15.24mm_Horizontal" V 4000 3460 50  0001 C CNN
 F 3 "~" H 4070 3460 50  0001 C CNN
 	1    4070 3460
@@
 F 0 "R20" V 10693 2650 50  0000 C CNN
 F 1 "R" V 10784 2650 50  0000 C CNN
-F 2 "Resistor_THT:R_Axial_DIN0207_L6.3mm_D2.5mm_P2.54mm_Vertical" V 10830 2650 50  0001 C CNN
+F 2 "Resistor_THT:R_Axial_DIN0309_L9.0mm_D3.2mm_P15.24mm_Horizontal" V 10830 2650 50  0001 C CNN
 F 3 "~" H 10900 2650 50  0001 C CNN
 	1    10900 2650
@@
 F 0 "R18" H 9930 2754 50  0000 R CNN
 F 1 "R" H 9930 2845 50  0000 R CNN
-F 2 "Resistor_THT:R_Axial_DIN0207_L6.3mm_D2.5mm_P2.54mm_Vertical" V 9930 2800 50  0001 C CNN
+F 2 "Resistor_THT:R_Axial_DIN0309_L9.0mm_D3.2mm_P15.24mm_Horizontal" V 9930 2800 50  0001 C CNN
 F 3 "~" H 10000 2800 50  0001 C CNN
 	1    10000 2800
@@
 F 0 "R19" H 10330 2754 50  0000 R CNN
 F 1 "R" H 10330 2845 50  0000 R CNN
-F 2 "Resistor_THT:R_Axial_DIN0207_L6.3mm_D2.5mm_P2.54mm_Vertical" V 10330 2800 50  0001 C CNN
+F 2 "Resistor_THT:R_Axial_DIN0309_L9.0mm_D3.2mm_P15.24mm_Horizontal" V 10330 2800 50  0001 C CNN
 F 3 "~" H 10400 2800 50  0001 C CNN
 	1    10400 2800
@@
 F 0 "R17" H 8945 1096 50  0000 L CNN
 F 1 "R" H 8945 1005 50  0000 L CNN
-F 2 "Resistor_THT:R_Axial_DIN0207_L6.3mm_D2.5mm_P2.54mm_Vertical" V 8805 1050 50  0001 C CNN
+F 2 "Resistor_THT:R_Axial_DIN0309_L9.0mm_D3.2mm_P15.24mm_Horizontal" V 8805 1050 50  0001 C CNN
 F 3 "~" H 8875 1050 50  0001 C CNN
 	1    8875 1050
@@
 	7900 5350 9000 5350
 $Comp
-L Device:Q_NMOS_DGS Q3
+L Device:Q_NMOS_DGS T3
 U 1 1 5E006E8C
 P 5850 1800
-F 0 "Q3" H 6055 1846 50  0000 L CNN
+F 0 "T3" H 6055 1846 50  0000 L CNN
 F 1 "Q_NMOS_DGS" H 6055 1755 50  0000 L CNN
-F 2 "" H 6050 1900 50  0001 C CNN
+F 2 "misc:TN0104(TO-92)" H 6050 1900 50  0001 C CNN
 F 3 "~" H 5850 1800 50  0001 C CNN
 	1    5850 1800
@@
 F 0 "R16" V 5593 2200 50  0000 C CNN
 F 1 "47k" V 5684 2200 50  0000 C CNN
-F 2 "" V 5730 2200 50  0001 C CNN
+F 2 "Resistor_THT:R_Axial_DIN0309_L9.0mm_D3.2mm_P15.24mm_Horizontal" V 5730 2200 50  0001 C CNN
 F 3 "~" H 5800 2200 50  0001 C CNN
 	1    5800 2200
@@
 F 0 "R12" V 5193 1800 50  0000 C CNN
 F 1 "1k" V 5284 1800 50  0000 C CNN
-F 2 "" V 5330 1800 50  0001 C CNN
+F 2 "Resistor_THT:R_Axial_DIN0309_L9.0mm_D3.2mm_P15.24mm_Horizontal" V 5330 1800 50  0001 C CNN
 F 3 "~" H 5400 1800 50  0001 C CNN
 	1    5400 1800
@@
 F 0 "R7" H 4520 1396 50  0000 L CNN
 F 1 "33" H 4520 1305 50  0000 L CNN
-F 2 "Resistor_THT:R_Axial_DIN0207_L6.3mm_D2.5mm_P2.54mm_Vertical" V 4380 1350 50  0001 C CNN
+F 2 "Resistor_THT:R_Axial_DIN0309_L9.0mm_D3.2mm_P15.24mm_Horizontal" V 4380 1350 50  0001 C CNN
 F 3 "~" H 4450 1350 50  0001 C CNN
 	1    4450 1350
@@
 $EndComp
 $Comp
-L Device:Q_NMOS_DGS Q2
+L Device:Q_NMOS_DGS T2
 U 1 1 5E01EC76
 P 4350 1800
-F 0 "Q2" H 4555 1846 50  0000 L CNN
+F 0 "T2" H 4555 1846 50  0000 L CNN
 F 1 "Q_NMOS_DGS" H 4555 1755 50  0000 L CNN
-F 2 "" H 4550 1900 50  0001 C CNN
+F 2 "misc:TN0104(TO-92)" H 4550 1900 50  0001 C CNN
 F 3 "~" H 4350 1800 50  0001 C CNN
 	1    4350 1800
@@
 F 0 "R15" V 4093 2200 50  0000 C CNN
 F 1 "47k" V 4184 2200 50  0000 C CNN
-F 2 "" V 4230 2200 50  0001 C CNN
+F 2 "Resistor_THT:R_Axial_DIN0309_L9.0mm_D3.2mm_P15.24mm_Horizontal" V 4230 2200 50  0001 C CNN
 F 3 "~" H 4300 2200 50  0001 C CNN
 	1    4300 2200
@@
 F 0 "R11" V 3693 1800 50  0000 C CNN
 F 1 "1k" V 3784 1800 50  0000 C CNN
-F 2 "" V 3830 1800 50  0001 C CNN
+F 2 "Resistor_THT:R_Axial_DIN0309_L9.0mm_D3.2mm_P15.24mm_Horizontal" V 3830 1800 50  0001 C CNN
 F 3 "~" H 3900 1800 50  0001 C CNN
 	1    3900 1800
@@
 F 0 "R5" H 1520 1396 50  0000 L CNN
 F 1 "33" H 1520 1305 50  0000 L CNN
-F 2 "Resistor_THT:R_Axial_DIN0207_L6.3mm_D2.5mm_P2.54mm_Vertical" V 1380 1350 50  0001 C CNN
+F 2 "Resistor_THT:R_Axial_DIN0309_L9.0mm_D3.2mm_P15.24mm_Horizontal" V 1380 1350 50  0001 C CNN
 F 3 "~" H 1450 1350 50  0001 C CNN
 	1    1450 1350
@@
 $EndComp
 $Comp
-L Device:Q_NMOS_DGS Q0
+L Device:Q_NMOS_DGS T0
 U 1 1 5E02C7FB
 P 1350 1800
-F 0 "Q0" H 1555 1846 50  0000 L CNN
+F 0 "T0" H 1555 1846 50  0000 L CNN
 F 1 "Q_NMOS_DGS" H 1555 1755 50  0000 L CNN
-F 2 "" H 1550 1900 50  0001 C CNN
+F 2 "misc:TN0104(TO-92)" H 1550 1900 50  0001 C CNN
 F 3 "~" H 1350 1800 50  0001 C CNN
 	1    1350 1800
@@
 F 0 "R13" V 1093 2200 50  0000 C CNN
 F 1 "47k" V 1184 2200 50  0000 C CNN
-F 2 "" V 1230 2200 50  0001 C CNN
+F 2 "Resistor_THT:R_Axial_DIN0309_L9.0mm_D3.2mm_P15.24mm_Horizontal" V 1230 2200 50  0001 C CNN
 F 3 "~" H 1300 2200 50  0001 C CNN
 	1    1300 2200
@@
 F 0 "R9" V 693 1800 50  0000 C CNN
 F 1 "1k" V 784 1800 50  0000 C CNN
-F 2 "" V 830 1800 50  0001 C CNN
+F 2 "Resistor_THT:R_Axial_DIN0309_L9.0mm_D3.2mm_P15.24mm_Horizontal" V 830 1800 50  0001 C CNN
 F 3 "~" H 900 1800 50  0001 C CNN
 	1    900  1800
@@
 F 0 "R6" H 3020 1396 50  0000 L CNN
 F 1 "33" H 3020 1305 50  0000 L CNN
-F 2 "Resistor_THT:R_Axial_DIN0207_L6.3mm_D2.5mm_P2.54mm_Vertical" V 2880 1350 50  0001 C CNN
+F 2 "Resistor_THT:R_Axial_DIN0309_L9.0mm_D3.2mm_P15.24mm_Horizontal" V 2880 1350 50  0001 C CNN
 F 3 "~" H 2950 1350 50  0001 C CNN
 	1    2950 1350
@@
 $EndComp
 $Comp
-L Device:Q_NMOS_DGS Q1
+L Device:Q_NMOS_DGS T1
 U 1 1 5E0358BD
 P 2850 1800
-F 0 "Q1" H 3055 1846 50  0000 L CNN
+F 0 "T1" H 3055 1846 50  0000 L CNN
 F 1 "Q_NMOS_DGS" H 3055 1755 50  0000 L CNN
-F 2 "" H 3050 1900 50  0001 C CNN
+F 2 "misc:TN0104(TO-92)" H 3050 1900 50  0001 C CNN
 F 3 "~" H 2850 1800 50  0001 C CNN
 	1    2850 1800
@@
 F 0 "R14" V 2593 2200 50  0000 C CNN
 F 1 "47k" V 2684 2200 50  0000 C CNN
-F 2 "" V 2730 2200 50  0001 C CNN
+F 2 "Resistor_THT:R_Axial_DIN0309_L9.0mm_D3.2mm_P15.24mm_Horizontal" V 2730 2200 50  0001 C CNN
 F 3 "~" H 2800 2200 50  0001 C CNN
 	1    2800 2200
@@
 F 0 "R10" V 2193 1800 50  0000 C CNN
 F 1 "1k" V 2284 1800 50  0000 C CNN
-F 2 "" V 2330 1800 50  0001 C CNN
+F 2 "Resistor_THT:R_Axial_DIN0309_L9.0mm_D3.2mm_P15.24mm_Horizontal" V 2330 1800 50  0001 C CNN
 F 3 "~" H 2400 1800 50  0001 C CNN
 	1    2400 1800

Commit message: added resistor layout
Changed lines of the file:
@@
 Text Label 5120 3110 0    50   ~ 0
 GND
+Text Label 9550 4350 0    50   ~ 0
+Reciever_0
+Text Label 9550 4550 0    50   ~ 0
+Reciever_1
+Text Label 7550 3950 2    50   ~ 0
+Reciever_2
 Text Label 7550 4150 2    50   ~ 0
-Reciever_0
-Text Label 7550 4050 2    50   ~ 0
-Reciever_1
-Text Label 7550 4250 2    50   ~ 0
-Reciever_2
-Text Label 7550 3950 2    50   ~ 0
 Reciever_3
-Text Label 9550 4350 0    50   ~ 0
+Text Label 9550 4450 0    50   ~ 0
 Emitter_0
 Connection ~ 9000 6200
@@
 Text Label 7700 6200 2    50   ~ 0
 5v
-Text Label 9550 4450 0    50   ~ 0
+Text Label 7550 4550 2    50   ~ 0
 Emitter_1
-Text Label 7550 4550 2    50   ~ 0
+Text Label 7550 4050 2    50   ~ 0
 Emitter_2
-Text Label 9550 4550 0    50   ~ 0
+Text Label 7550 4250 2    50   ~ 0
 Emitter_3
 $Comp

Commit message: draft 1 layout
Changed lines of the file:
@@
 Text Label 10900 2300 1    50   ~ 0
 Buzzer
-Text Label 7550 2950 2    50   ~ 0
+Text Label 7550 3850 2    50   ~ 0
 Buzzer
 Text Label 7550 2150 2    50   ~ 0
@@
 Text Label 7550 2850 2    50   ~ 0
 M1_encoder_A
-Text Label 7550 3850 2    50   ~ 0
+Text Label 7550 2950 2    50   ~ 0
 M1_encoder_B
 Text Label 7550 2650 2    50   ~ 0

Commit message: added filter capictors
Parts:
- added C2: 0.1uF, Capacitor_SMD:C_0603_1608Metric_Pad1.05x0.95mm_HandSolder, symbol Device:CP1_Small
- added C3: 1.0uF, Capacitor_SMD:C_0603_1608Metric_Pad1.05x0.95mm_HandSolder, symbol Device:CP1_Small
- added CP1: 10uF (Tantalum), Capacitor_SMD:C_0603_1608Metric_Pad1.05x0.95mm_HandSolder, symbol Device:CP1
Connections:
- wire segments 106 -> 112
Other:
- moved on the sheet: U2
Changed lines of the file:
@@
-$EndComp
-$Comp
-L SN754410NE:SN754410NE U2
-U 1 1 5D1BEE18
-P 5000 5700
-F 0 "U2" H 5000 6670 50  0000 C CNN
-F 1 "SN754410NE" H 5000 6579 50  0000 C CNN
-F 2 "SN754410NE.kicad_mod:DIP254P762X508-16" H 5000 5700 50  0001 L BNN
-F 3 "PDIP-16 Texas Instruments" H 5000 5700 50  0001 L BNN
-F 4 "Texas Instruments" H 5000 5700 50  0001 L BNN "Field4"
-F 5 "None" H 5000 5700 50  0001 L BNN "Field5"
-F 6 "Unavailable" H 5000 5700 50  0001 L BNN "Field6"
-F 7 "Peripheral Drivers and Actuators Quad Half-Hs" H 5000 5700 50  0001 L BNN "Field7"
-F 8 "SN754410NE" H 5000 5700 50  0001 L BNN "Field8"
-	1    5000 5700
-	1    0    0    -1
 $EndComp
 $Comp
@@
 	8700 5650 8700 5800
 Wire Wire Line
-	8700 5800 8350 5800
-Wire Wire Line
 	9550 4050 10250 4050
 Wire Wire Line
@@
 Text Label 7550 3450 2    50   ~ 0
 3.3v
-Text Label 4300 5100 2    50   ~ 0
+Text Label 4450 5050 2    50   ~ 0
 5v
 Wire Wire Line
@@
 Text Label 7600 5500 2    50   ~ 0
 vBatt
-Text Label 4300 5200 2    50   ~ 0
+Text Label 4450 5150 2    50   ~ 0
 5v
-Text Label 4300 5400 2    50   ~ 0
+Text Label 5050 5350 2    50   ~ 0
 M1_speed
-Text Label 4300 5500 2    50   ~ 0
+Text Label 5050 5450 2    50   ~ 0
 M2_speed
-Text Label 4300 5700 2    50   ~ 0
+Text Label 5050 5650 2    50   ~ 0
 M1_forward
-Text Label 4300 5800 2    50   ~ 0
+Text Label 5050 5750 2    50   ~ 0
 M1_backward
-Text Label 4300 5900 2    50   ~ 0
+Text Label 5050 5850 2    50   ~ 0
 M2_forward
-Text Label 4300 6000 2    50   ~ 0
+Text Label 5050 5950 2    50   ~ 0
 M2_backward
 Wire Wire Line
-	4300 6200 4150 6200
-Wire Wire Line
-	4150 6200 4150 6300
-Wire Wire Line
-	4150 6500 4300 6500
-Wire Wire Line
-	4300 6400 4150 6400
-Connection ~ 4150 6400
-Wire Wire Line
-	4150 6400 4150 6500
-Wire Wire Line
-	4300 6300 4150 6300
-Connection ~ 4150 6300
-Wire Wire Line
-	4150 6300 4150 6350
-Wire Wire Line
-	4150 6350 4000 6350
-Connection ~ 4150 6350
-Wire Wire Line
-	4150 6350 4150 6400
-Text Label 4000 6350 2    50   ~ 0
+	5050 6150 4900 6150
+Wire Wire Line
+	4900 6150 4900 6250
+Wire Wire Line
+	4900 6450 5050 6450
+Wire Wire Line
+	5050 6350 4900 6350
+Connection ~ 4900 6350
+Wire Wire Line
+	4900 6350 4900 6450
+Wire Wire Line
+	5050 6250 4900 6250
+Connection ~ 4900 6250
+Wire Wire Line
+	4900 6250 4900 6300
+Wire Wire Line
+	4900 6300 4750 6300
+Connection ~ 4900 6300
+Wire Wire Line
+	4900 6300 4900 6350
+Text Label 4750 6300 2    50   ~ 0
 GND
 Text Label 7550 2450 2    50   ~ 0
@@
 Text Label 7550 2550 2    50   ~ 0
 M2_speed
-Text Label 5700 5100 0    50   ~ 0
+Text Label 6450 5050 0    50   ~ 0
 OUT1
-Text Label 5700 5200 0    50   ~ 0
+Text Label 6450 5150 0    50   ~ 0
 OUT2
-Text Label 5700 5300 0    50   ~ 0
+Text Label 6450 5250 0    50   ~ 0
 OUT3
-Text Label 5700 5400 0    50   ~ 0
+Text Label 6450 5350 0    50   ~ 0
 OUT4
 Text Label 3200 5250 0    50   ~ 0
@@
 Emitter_0
 Connection ~ 9000 6200
-Wire Wire Line
-	8350 5800 8350 6000
-Wire Wire Line
-	8350 6000 7700 6000
-Connection ~ 8350 5800
-Wire Wire Line
-	8350 5800 7900 5800
 Text Label 7700 6000 2    50   ~ 0
 GND
@@
 	9000 5950 9000 6200
 Wire Wire Line
-	7700 6200 9000 6200
+	7700 6200 8150 6200
 Text Label 7700 6200 2    50   ~ 0
 5v
@@
 Text Label 6650 2400 0    50   ~ 0
 GND
+$Comp
+L Device:CP1 CP1
+U 1 1 5E08B3B9
+P 8150 6050
+F 0 "CP1" H 8035 6004 50  0000 R CNN
+F 1 "10uF (Tantalum)" H 8035 6095 50  0000 R CNN
+F 2 "Capacitor_SMD:C_0603_1608Metric_Pad1.05x0.95mm_HandSolder" H 8150 6050 50  0001 C CNN
+F 3 "~" H 8150 6050 50  0001 C CNN
+	1    8150 6050
+	-1   0    0    1
+$EndComp
+Wire Wire Line
+	7900 5800 8150 5800
+Wire Wire Line
+	7700 6000 7900 6000
+Wire Wire Line
+	7900 6000 7900 5800
+Connection ~ 7900 5800
+Connection ~ 8150 6200
+Wire Wire Line
+	8150 5900 8150 5800
+Wire Wire Line
+	8150 6200 9000 6200
+Connection ~ 8150 5800
+Wire Wire Line
+	8150 5800 8700 5800
+$Comp
+L SN754410NE:SN754410NE U2
+U 1 1 5D1BEE18
+P 5750 5650
+F 0 "U2" H 5750 6620 50  0000 C CNN
+F 1 "SN754410NE" H 5750 6529 50  0000 C CNN
+F 2 "SN754410NE.kicad_mod:DIP254P762X508-16" H 5750 5650 50  0001 L BNN
+F 3 "PDIP-16 Texas Instruments" H 5750 5650 50  0001 L BNN
+F 4 "Texas Instruments" H 5750 5650 50  0001 L BNN "Field4"
+F 5 "None" H 5750 5650 50  0001 L BNN "Field5"
+F 6 "Unavailable" H 5750 5650 50  0001 L BNN "Field6"
+F 7 "Peripheral Drivers and Actuators Quad Half-Hs" H 5750 5650 50  0001 L BNN "Field7"
+F 8 "SN754410NE" H 5750 5650 50  0001 L BNN "Field8"
+	1    5750 5650
+	1    0    0    -1
+$EndComp
+$Comp
+L Device:CP1_Small C2
+U 1 1 5E0B1B16
+P 4550 4950
+F 0 "C2" H 4450 4900 50  0000 R CNN
+F 1 "0.1uF" H 4459 4995 50  0000 R CNN
+F 2 "Capacitor_SMD:C_0603_1608Metric_Pad1.05x0.95mm_HandSolder" H 4550 4950 50  0001 C CNN
+F 3 "~" H 4550 4950 50  0001 C CNN
+	1    4550 4950
+	-1   0    0    1
+$EndComp
+$Comp
+L Device:CP1_Small C3
+U 1 1 5E0B1E54
+P 4550 5250
+F 0 "C3" H 4350 5300 50  0000 L CNN
+F 1 "1.0uF" H 4250 5200 50  0000 L CNN
+F 2 "Capacitor_SMD:C_0603_1608Metric_Pad1.05x0.95mm_HandSolder" H 4550 5250 50  0001 C CNN
+F 3 "~" H 4550 5250 50  0001 C CNN
+	1    4550 5250
+	1    0    0    -1
+$EndComp
+Wire Wire Line
+	5050 5050 4550 5050
+Connection ~ 5050 5050
+Wire Wire Line
+	4450 5150 4550 5150
+Connection ~ 4550 5050
+Wire Wire Line
+	4550 5050 4450 5050
+Connection ~ 4550 5150
+Wire Wire Line
+	4550 5150 5050 5150
+Text Label 4550 4850 2    50   ~ 0
+GND
+Text Label 4550 5350 3    50   ~ 0
+GND
 $EndSCHEMATC

Commit message: started new design
Parts:
- removed MH_GND1, MH_SCL1, MH_SDA1, MH_vBatt1: MountingHole_Pad, Connector_PinHeader_2.54mm:PinHeader_1x01_P2.54mm_Vertical, symbol Mechanical:MountingHole_Pad
- added J2: BT_Conn, Connector_PinSocket_2.54mm:PinSocket_1x02_P2.54mm_Vertical, symbol Connector:Conn_01x02_Male
- added J4: I2C_Conn, Connector_PinSocket_2.54mm:PinSocket_1x02_P2.54mm_Vertical, symbol Connector:Conn_01x02_Male
- added S1: EG1218, misc:Switch_amazon, symbol dk_Slide-Switches:EG1218
Connections:
- wire segments 112 -> 114
Changed lines of the file:
@@
 $EndComp
-Wire Wire Line
-	7900 5500 7900 5350
 Wire Wire Line
 	8700 5650 8700 5800
@@
 Text Label 8275 900  2    50   ~ 0
 GND
-$Comp
-L Mechanical:MountingHole_Pad MH_SCL1
-U 1 1 5D2CDA5E
-P 9900 1250
-F 0 "MH_SCL1" V 9854 1400 50  0000 L CNN
-F 1 "MountingHole_Pad" V 9945 1400 50  0000 L CNN
-F 2 "Connector_PinHeader_2.54mm:PinHeader_1x01_P2.54mm_Vertical" H 9900 1250 50  0001 C CNN
-F 3 "~" H 9900 1250 50  0001 C CNN
-	1    9900 1250
-	0    1    1    0
-$EndComp
-$Comp
-L Mechanical:MountingHole_Pad MH_SDA1
-U 1 1 5D2CDD65
-P 9900 1000
-F 0 "MH_SDA1" V 9854 1150 50  0000 L CNN
-F 1 "MountingHole_Pad" V 9945 1150 50  0000 L CNN
-F 2 "Connector_PinHeader_2.54mm:PinHeader_1x01_P2.54mm_Vertical" H 9900 1000 50  0001 C CNN
-F 3 "~" H 9900 1000 50  0001 C CNN
-	1    9900 1000
-	0    1    1    0
-$EndComp
 Text Label 7550 4350 2    50   ~ 0
 i2c_SDA
 Text Label 7550 4450 2    50   ~ 0
 i2c_SCL
-Text Label 9800 1000 2    50   ~ 0
-i2c_SDA
-Text Label 9800 1250 2    50   ~ 0
+Text Label 10250 1050 0    50   ~ 0
 i2c_SCL
-$Comp
-L Mechanical:MountingHole_Pad MH_GND1
-U 1 1 5D2D0AFA
-P 9900 1500
-F 0 "MH_GND1" V 9854 1650 50  0000 L CNN
-F 1 "MountingHole_Pad" V 9945 1650 50  0000 L CNN
-F 2 "Connector_PinHeader_2.54mm:PinHeader_1x01_P2.54mm_Vertical" H 9900 1500 50  0001 C CNN
-F 3 "~" H 9900 1500 50  0001 C CNN
-	1    9900 1500
-	0    1    1    0
-$EndComp
-$Comp
-L Mechanical:MountingHole_Pad MH_vBatt1
-U 1 1 5D2D0CC0
-P 9900 750
-F 0 "MH_vBatt1" V 9854 900 50  0000 L CNN
-F 1 "MountingHole_Pad" V 9945 900 50  0000 L CNN
-F 2 "Connector_PinHeader_2.54mm:PinHeader_1x01_P2.54mm_Vertical" H 9900 750 50  0001 C CNN
-F 3 "~" H 9900 750 50  0001 C CNN
-	1    9900 750
-	0    1    1    0
-$EndComp
-Text Label 9800 750  2    50   ~ 0
+Text Label 10250 1550 0    50   ~ 0
 vBatt
-Text Label 9800 1500 2    50   ~ 0
+Text Label 10250 1450 0    50   ~ 0
 GND
 Text Label 9100 675  0    50   ~ 0
@@
 Text Label 7550 3550 2    50   ~ 0
 GND
-Wire Wire Line
-	7900 5350 9000 5350
 $Comp
 L Device:Q_NMOS_DGS T3
@@
 Wire Wire Line
 	5050 5050 4550 5050
-Connection ~ 5050 5050
 Wire Wire Line
 	4450 5150 4550 5150
@@
 Text Label 4550 5350 3    50   ~ 0
 GND
+$Comp
+L dk_Slide-Switches:EG1218 S1
+U 1 1 5E600D6A
+P 8350 5200
+F 0 "S1" H 8350 5479 50  0000 C CNN
+F 1 "EG1218" H 8350 5388 50  0000 C CNN
+F 2 "misc:Switch_amazon" H 8550 5400 50  0001 L CNN
+F 3 "http://spec_sheets.e-switch.com/specs/P040040.pdf" H 8550 5500 60  0001 L CNN
+F 4 "EG1903-ND" H 8550 5600 60  0001 L CNN "Digi-Key_PN"
+F 5 "EG1218" H 8550 5700 60  0001 L CNN "MPN"
+F 6 "Switches" H 8550 5800 60  0001 L CNN "Category"
+F 7 "Slide Switches" H 8550 5900 60  0001 L CNN "Family"
+F 8 "http://spec_sheets.e-switch.com/specs/P040040.pdf" H 8550 6000 60  0001 L CNN "DK_Datasheet_Link"
+F 9 "/product-detail/en/e-switch/EG1218/EG1903-ND/101726" H 8550 6100 60  0001 L CNN "DK_Detail_Page"
+F 10 "SWITCH SLIDE SPDT 200MA 30V" H 8550 6200 60  0001 L CNN "Description"
+F 11 "E-Switch" H 8550 6300 60  0001 L CNN "Manufacturer"
+F 12 "Active" H 8550 6400 60  0001 L CNN "Status"
+	1    8350 5200
+	1    0    0    -1
+$EndComp
+Wire Wire Line
+	8550 5300 9000 5300
+Wire Wire Line
+	9000 5300 9000 5350
+Wire Wire Line
+	8150 5200 7900 5200
+Wire Wire Line
+	7900 5200 7900 5500
+$Comp
+L Connector:Conn_01x02_Male J4
+U 1 1 5E60A04C
+P 10050 1450
+F 0 "J4" H 10156 1628 50  0000 C CNN
+F 1 "I2C_Conn" H 10150 1550 50  0000 C CNN
+F 2 "Connector_PinSocket_2.54mm:PinSocket_1x02_P2.54mm_Vertical" H 10050 1450 50  0001 C CNN
+F 3 "~" H 10050 1450 50  0001 C CNN
+	1    10050 1450
+	1    0    0    -1
+$EndComp
+Text Label 10250 1150 0    50   ~ 0
+i2c_SDA
+$Comp
+L Connector:Conn_01x02_Male J2
+U 1 1 5E60EB54
+P 10050 1050
+F 0 "J2" H 10156 1228 50  0000 C CNN
+F 1 "BT_Conn" H 10150 1150 50  0000 C CNN
+F 2 "Connector_PinSocket_2.54mm:PinSocket_1x02_P2.54mm_Vertical" H 10050 1050 50  0001 C CNN
+F 3 "~" H 10050 1050 50  0001 C CNN
+	1    10050 1050
+	1    0    0    -1
+$EndComp
 $EndSCHEMATC
