File: pcb_files/mouse/mouse.sch (KiCad schematic (older format))
At the start: 70 parts, among them J2 BT_Conn, J4 I2C_Conn, M1 Motor_DC, M2 Motor_DC, M3 CASTER_BALL, Q0 Q_Photo_NPN, Q1 Q_Photo_NPN, Q2 Q_Photo_NPN, Q3 Q_Photo_NPN, SW1 SW_Push, T0 Q_NMOS_DGS, T1 Q_NMOS_DGS, T2 Q_NMOS_DGS, T3 Q_NMOS_DGS, U1 Teensy3.2, U2 SN754410NE, U4 Encoder_3081, U5 Encoder_3081, U6 LM2596S-5

Commit message: test1
Parts:
- added MH?: MountingHole, symbol Mechanical:MountingHole
Changed lines of the file:
@@
+	1    0    0    -1
+$EndComp
+$Comp
+L Mechanical:MountingHole MH?
+U 1 1 5E7A547E
+P 13225 5675
+F 0 "MH?" H 13325 5721 50  0000 L CNN
+F 1 "MountingHole" H 13325 5630 50  0000 L CNN
+F 2 "" H 13225 5675 50  0001 C CNN
+F 3 "~" H 13225 5675 50  0001 C CNN
+	1    13225 5675
 	1    0    0    -1
 $EndComp

Commit message: paired footprints with almost all compoennts
Parts:
- removed MH?: MountingHole, symbol Mechanical:MountingHole
- C1, C4, C5, C6, C7, C8: value 104 -> 0.1uF; footprint (none) -> Capacitor_SMD:C_1206_3216Metric_Pad1.42x1.75mm_HandSolder
- C10: footprint (none) -> Capacitor_Tantalum_SMD:CP_EIA-7343-15_Kemet-W_Pad2.25x2.55mm_HandSolder
- C2, C3: footprint Capacitor_SMD:C_0603_1608Metric_Pad1.05x0.95mm_HandSolder -> Capacitor_SMD:C_1206_3216Metric_Pad1.42x1.75mm_HandSolder
- C9: footprint (none) -> Capacitor_THT:CP_Radial_D10.0mm_P5.00mm
- D12: footprint (none) -> Diode_THT:D_DO-201AD_P12.70mm_Horizontal
- L1: value 33uH -> 22uH
- MH1, MH2, MH3, MH4: renamed from MH?; footprint (none) -> MountingHole:MountingHole_4.3mm_M4
- R1, R10, R11, R12, R13, R14, R15, R16, R17, R2, R3, R4, R5, R6, R7, R8, R9: footprint Resistor_THT:R_Axial_DIN0309_L9.0mm_D3.2mm_P15.24mm_Horizontal -> Resistor_THT:R_Axial_DIN0309_L9.0mm_D3.2mm_P12.70mm_Horizontal
- gave numbers to parts that had none: 2

Commit message: Created footprint for inductor
Parts:
- R18, R21: footprint (none) -> Resistor_SMD:R_1206_3216Metric_Pad1.42x1.75mm_HandSolder
Changed lines of the file:
@@
 F 0 "R18" H 13525 6950 50  0000 L CNN
 F 1 "4.7k" H 13475 6850 50  0000 L CNN
-F 2 "" V 13630 6900 50  0001 C CNN
+F 2 "Resistor_SMD:R_1206_3216Metric_Pad1.42x1.75mm_HandSolder" V 13630 6900 50  0001 C CNN
 F 3 "~" H 13700 6900 50  0001 C CNN
 	1    13700 6900
@@
 F 0 "R21" H 13970 6896 50  0000 L CNN
 F 1 "4.7k" H 13970 6805 50  0000 L CNN
-F 2 "" V 13830 6850 50  0001 C CNN
+F 2 "Resistor_SMD:R_1206_3216Metric_Pad1.42x1.75mm_HandSolder" V 13830 6850 50  0001 C CNN
 F 3 "~" H 13900 6850 50  0001 C CNN
 	1    13900 6850

Commit message: reverted back to LDO
Parts:
- removed D12: 1n5824, Diode_THT:D_DO-201AD_P12.70mm_Horizontal, symbol Device:D_Schottky
- removed L1: 22uH, symbol Device:L
- removed U6: LM2596S-5, Package_TO_SOT_SMD:TO-263-5_TabPin3, symbol Regulator_Switching:LM2596S-5
- added U3: LM1084-5.0, Package_TO_SOT_SMD:TO-263-3_TabPin2, symbol Regulator_Linear:LM1084-5.0
- C10: value 220uF -> 10uF(Tantalum); footprint Capacitor_Tantalum_SMD:CP_EIA-7343-15_Kemet-W_Pad2.25x2.55mm_HandSolder -> Capacitor_SMD:C_1206_3216Metric_Pad1.42x1.75mm_HandSolder
- C9: value 680uF -> 10uF; footprint Capacitor_THT:CP_Radial_D10.0mm_P5.00mm -> Capacitor_SMD:C_1206_3216Metric_Pad1.42x1.75mm_HandSolder
- R19, R20: footprint Resistor_THT:R_Axial_DIN0309_L9.0mm_D3.2mm_P15.24mm_Horizontal -> Resistor_SMD:R_1206_3216Metric_Pad1.42x1.75mm_HandSolder
Connections:
- wire segments 142 -> 137
Changed lines of the file:
@@
 F 0 "R20" V 14993 7050 50  0000 C CNN
 F 1 "R" V 15084 7050 50  0000 C CNN
-F 2 "Resistor_THT:R_Axial_DIN0309_L9.0mm_D3.2mm_P15.24mm_Horizontal" V 15130 7050 50  0001 C CNN
+F 2 "Resistor_SMD:R_1206_3216Metric_Pad1.42x1.75mm_HandSolder" V 15130 7050 50  0001 C CNN
 F 3 "~" H 15200 7050 50  0001 C CNN
 	1    15200 7050
@@
 F 0 "R19" H 14630 7154 50  0000 R CNN
 F 1 "R" H 14630 7245 50  0000 R CNN
-F 2 "Resistor_THT:R_Axial_DIN0309_L9.0mm_D3.2mm_P15.24mm_Horizontal" V 14630 7200 50  0001 C CNN
+F 2 "Resistor_SMD:R_1206_3216Metric_Pad1.42x1.75mm_HandSolder" V 14630 7200 50  0001 C CNN
 F 3 "~" H 14700 7200 50  0001 C CNN
 	1    14700 7200
@@
 	11750 8700 11550 8700
 $Comp
-L Regulator_Switching:LM2596S-5 U6
-U 1 1 5E812135
-P 13850 1475
-F 0 "U6" H 13850 1842 50  0000 C CNN
-F 1 "LM2596S-5" H 13850 1751 50  0000 C CNN
-F 2 "Package_TO_SOT_SMD:TO-263-5_TabPin3" H 13900 1225 50  0001 L CIN
-F 3 "http://www.ti.com/lit/ds/symlink/lm2596.pdf" H 13850 1475 50  0001 C CNN
-	1    13850 1475
-	1    0    0    -1
-$EndComp
-$Comp
 L mouse-rescue:EG1218-dk_Slide-Switches S1
 U 1 1 5E819689
-P 12650 1275
-F 0 "S1" H 12650 1554 50  0000 C CNN
-F 1 "EG1218" H 12650 1463 50  0000 C CNN
-F 2 "misc:Switch_amazon" H 12850 1475 50  0001 L CNN
-F 3 "http://spec_sheets.e-switch.com/specs/P040040.pdf" H 12850 1575 60  0001 L CNN
-F 4 "EG1903-ND" H 12850 1675 60  0001 L CNN "Digi-Key_PN"
-F 5 "EG1218" H 12850 1775 60  0001 L CNN "MPN"
-F 6 "Switches" H 12850 1875 60  0001 L CNN "Category"
-F 7 "Slide Switches" H 12850 1975 60  0001 L CNN "Family"
-F 8 "http://spec_sheets.e-switch.com/specs/P040040.pdf" H 12850 2075 60  0001 L CNN "DK_Datasheet_Link"
-F 9 "/product-detail/en/e-switch/EG1218/EG1903-ND/101726" H 12850 2175 60  0001 L CNN "DK_Detail_Page"
-F 10 "SWITCH SLIDE SPDT 200MA 30V" H 12850 2275 60  0001 L CNN "Description"
-F 11 "E-Switch" H 12850 2375 60  0001 L CNN "Manufacturer"
-F 12 "Active" H 12850 2475 60  0001 L CNN "Status"
-	1    12650 1275
+P 12875 3525
+F 0 "S1" H 12875 3804 50  0000 C CNN
+F 1 "EG1218" H 12875 3713 50  0000 C CNN
+F 2 "misc:Switch_amazon" H 13075 3725 50  0001 L CNN
+F 3 "http://spec_sheets.e-switch.com/specs/P040040.pdf" H 13075 3825 60  0001 L CNN
+F 4 "EG1903-ND" H 13075 3925 60  0001 L CNN "Digi-Key_PN"
+F 5 "EG1218" H 13075 4025 60  0001 L CNN "MPN"
+F 6 "Switches" H 13075 4125 60  0001 L CNN "Category"
+F 7 "Slide Switches" H 13075 4225 60  0001 L CNN "Family"
+F 8 "http://spec_sheets.e-switch.com/specs/P040040.pdf" H 13075 4325 60  0001 L CNN "DK_Datasheet_Link"
+F 9 "/product-detail/en/e-switch/EG1218/EG1903-ND/101726" H 13075 4425 60  0001 L CNN "DK_Detail_Page"
+F 10 "SWITCH SLIDE SPDT 200MA 30V" H 13075 4525 60  0001 L CNN "Description"
+F 11 "E-Switch" H 13075 4625 60  0001 L CNN "Manufacturer"
+F 12 "Active" H 13075 4725 60  0001 L CNN "Status"
+	1    12875 3525
 	1    0    0    -1
 $EndComp
@@
 L Device:Battery_Cell BT1
 U 1 1 5E820C97
-P 12350 1725
-F 0 "BT1" H 12100 1825 50  0000 L CNN
-F 1 "Battery_Cell" H 11800 1725 50  0000 L CNN
-F 2 "Connector_PinSocket_2.54mm:PinSocket_1x02_P2.54mm_Vertical" V 12350 1785 50  0001 C CNN
-F 3 "~" V 12350 1785 50  0001 C CNN
-	1    12350 1725
-	1    0    0    -1
-$EndComp
-Text Label 13350 2025 3    50   ~ 0
-GND
-Text Label 13850 1775 3    50   ~ 0
-GND
-Text Label 12350 1825 3    50   ~ 0
-GND
-Wire Wire Line
-	12450 1275 12350 1275
-Wire Wire Line
-	12350 1275 12350 1525
-Wire Wire Line
-	12350 1275 12200 1275
-Connection ~ 12350 1275
-Text Label 12200 1275 2    50   ~ 0
-vBatt
-Wire Wire Line
-	13350 1575 13350 2025
-Text Label 13100 2025 3    50   ~ 0
-GND
-Text Label 15200 1575 0    50   ~ 0
-5v
-$Comp
-L Device:L L1
-U 1 1 5E8A9E63
-P 14800 1575
-F 0 "L1" V 14990 1575 50  0000 C CNN
-F 1 "22uH" V 14899 1575 50  0000 C CNN
-F 2 "" H 14800 1575 50  0001 C CNN
-F 3 "~" H 14800 1575 50  0001 C CNN
-	1    14800 1575
-	0    -1   -1   0
-$EndComp
-Wire Wire Line
-	15200 1575 15100 1575
-$Comp
-L Device:D_Schottky D12
-U 1 1 5E8B6F40
-P 14550 1725
-F 0 "D12" V 14504 1804 50  0000 L CNN
-F 1 "1n5824" V 14595 1804 50  0000 L CNN
-F 2 "Diode_THT:D_DO-201AD_P12.70mm_Horizontal" H 14550 1725 50  0001 C CNN
-F 3 "~" H 14550 1725 50  0001 C CNN
-	1    14550 1725
-	0    1    1    0
-$EndComp
-Text Label 14550 1875 3    50   ~ 0
-GND
+P 12650 4100
+F 0 "BT1" H 12400 4200 50  0000 L CNN
+F 1 "Battery_Cell" H 12100 4100 50  0000 L CNN
+F 2 "Connector_PinSocket_2.54mm:PinSocket_1x02_P2.54mm_Vertical" V 12650 4160 50  0001 C CNN
+F 3 "~" V 12650 4160 50  0001 C CNN
+	1    12650 4100
+	1    0    0    -1
+$EndComp
 $Comp
 L Device:CP1 C10
 U 1 1 5E8B972D
-P 15100 1725
-F 0 "C10" H 15215 1771 50  0000 L CNN
-F 1 "220uF" H 15215 1680 50  0000 L CNN
-F 2 "Capacitor_Tantalum_SMD:CP_EIA-7343-15_Kemet-W_Pad2.25x2.55mm_HandSolder" H 15100 1725 50  0001 C CNN
-F 3 "~" H 15100 1725 50  0001 C CNN
-	1    15100 1725
-	1    0    0    -1
-$EndComp
-Connection ~ 15100 1575
-Wire Wire Line
-	15100 1575 14950 1575
-$Comp
-L Device:CP1 C9
-U 1 1 5E8BA3C3
-P 13100 1525
-F 0 "C9" H 12900 1475 50  0000 L CNN
-F 1 "680uF" H 12850 1375 50  0000 L CNN
-F 2 "Capacitor_THT:CP_Radial_D10.0mm_P5.00mm" H 13100 1525 50  0001 C CNN
-F 3 "~" H 13100 1525 50  0001 C CNN
-	1    13100 1525
-	1    0    0    -1
-$EndComp
-Wire Wire Line
-	12850 1375 13100 1375
-Connection ~ 13100 1375
-Wire Wire Line
-	13100 1375 13350 1375
-Wire Wire Line
-	13100 1675 13100 2025
-Wire Wire Line
-	14350 1575 14550 1575
-Connection ~ 14550 1575
-Wire Wire Line
-	14550 1575 14650 1575
-Wire Wire Line
-	14350 1375 14500 1375
-Wire Wire Line
-	14500 1375 14500 1225
-Wire Wire Line
-	14500 1225 15100 1225
-Wire Wire Line
-	15100 1225 15100 1575
-Text Label 15100 1875 3    50   ~ 0
-GND
+P 14325 3575
+F 0 "C10" H 14440 3621 50  0000 L CNN
+F 1 "10uF(Tantalum)" H 14440 3530 50  0000 L CNN
+F 2 "Capacitor_SMD:C_1206_3216Metric_Pad1.42x1.75mm_HandSolder" H 14325 3575 50  0001 C CNN
+F 3 "~" H 14325 3575 50  0001 C CNN
+	1    14325 3575
+	1    0    0    -1
+$EndComp
 Text Label 9650 6100 0    50   ~ 0
 5v
@@
 	1    0    0    -1
 $EndComp
+$Comp
+L Regulator_Linear:LM1084-5.0 U3
+U 1 1 5E7860F1
+P 13700 3425
+F 0 "U3" H 13700 3667 50  0000 C CNN
+F 1 "LM1084-5.0" H 13700 3576 50  0000 C CNN
+F 2 "Package_TO_SOT_SMD:TO-263-3_TabPin2" H 13700 3675 50  0001 C CIN
+F 3 "http://www.ti.com/lit/ds/symlink/lm1084.pdf" H 13700 3425 50  0001 C CNN
+	1    13700 3425
+	1    0    0    -1
+$EndComp
+Wire Wire Line
+	13700 3725 13700 3975
+Text Label 13700 3975 3    50   ~ 0
+GND
+Wire Wire Line
+	14000 3425 14325 3425
+Text Label 14500 3425 0    50   ~ 0
+5v
+Text Label 12650 4200 3    50   ~ 0
+GND
+Wire Wire Line
+	12650 3900 12650 3675
+Wire Wire Line
+	12650 3525 12675 3525
+Wire Wire Line
+	13400 3425 13275 3425
+Connection ~ 14325 3425
+Wire Wire Line
+	14325 3425 14500 3425
+$Comp
+L Device:CP1 C9
+U 1 1 5E79A9AD
+P 13275 3000
+F 0 "C9" H 13390 3046 50  0000 L CNN
+F 1 "10uF" H 13390 2955 50  0000 L CNN
+F 2 "Capacitor_SMD:C_1206_3216Metric_Pad1.42x1.75mm_HandSolder" H 13275 3000 50  0001 C CNN
+F 3 "~" H 13275 3000 50  0001 C CNN
+	1    13275 3000
+	-1   0    0    1
+$EndComp
+Text Label 13275 2850 0    50   ~ 0
+GND
+Wire Wire Line
+	13275 3150 13275 3425
+Connection ~ 13275 3425
+Wire Wire Line
+	13275 3425 13075 3425
+Wire Wire Line
+	12650 3675 12425 3675
+Connection ~ 12650 3675
+Wire Wire Line
+	12650 3675 12650 3525
+Text Label 12425 3675 2    50   ~ 0
+vBatt
 $EndSCHEMATC

Commit message: added rgb led, and button
Parts:
- removed D5: STATUS_1, misc:3528_SMD_LED, symbol Device:LED
- added C11, C12: 0.1uF, Capacitor_SMD:C_1206_3216Metric_Pad1.42x1.75mm_HandSolder, symbol Device:C
- added D4, D5: WS2812B, LED_SMD:LED_WS2812B_PLCC4_5.0x5.0mm_P3.2mm, symbol LED:WS2812B
- added SW2: SW_Push, keyswitches:MX, symbol Switch:SW_Push
- R19: footprint Resistor_SMD:R_1206_3216Metric_Pad1.42x1.75mm_HandSolder -> Resistor_THT:R_Axial_DIN0309_L9.0mm_D3.2mm_P12.70mm_Horizontal
Connections:
- net labels added: PUSH_SW1
- net labels removed: STATUS_LED_1
- wire segments 137 -> 151
Changed lines of the file:
@@
 Wire Wire Line
 	15200 6700 15200 6900
-$Comp
-L Device:LED D5
-U 1 1 5D2990A5
-P 14700 7500
-F 0 "D5" H 14691 7716 50  0000 C CNN
-F 1 "STATUS_1" H 14700 7650 50  0000 C CNN
-F 2 "misc:3528_SMD_LED" H 14700 7500 50  0001 C CNN
-F 3 "~" H 14700 7500 50  0001 C CNN
-	1    14700 7500
-	0    -1   -1   0
-$EndComp
-$Comp
-L Device:R R19
-U 1 1 5D2990AB
-P 14700 7200
-F 0 "R19" H 14630 7154 50  0000 R CNN
-F 1 "R" H 14630 7245 50  0000 R CNN
-F 2 "Resistor_SMD:R_1206_3216Metric_Pad1.42x1.75mm_HandSolder" V 14630 7200 50  0001 C CNN
-F 3 "~" H 14700 7200 50  0001 C CNN
-	1    14700 7200
-	-1   0    0    1
-$EndComp
-Text Label 14700 7050 1    50   ~ 0
-STATUS_LED_1
-Text Label 14700 7650 3    50   ~ 0
-GND
 Text Label 7650 5100 2    50   ~ 0
 RGB_DATA
-Text Label 7650 5200 2    50   ~ 0
-STATUS_LED_1
 Text Label 15200 6700 1    50   ~ 0
 Buzzer
@@
 Text Label 12425 3675 2    50   ~ 0
 vBatt
+Text Label 11100 7575 3    50   ~ 0
+3.3v
+$Comp
+L Device:R R19
+U 1 1 5E7B1BAC
+P 11100 7425
+F 0 "R19" H 11170 7471 50  0000 L CNN
+F 1 "R" H 11170 7380 50  0000 L CNN
+F 2 "Resistor_THT:R_Axial_DIN0309_L9.0mm_D3.2mm_P12.70mm_Horizontal" V 11030 7425 50  0001 C CNN
+F 3 "~" H 11100 7425 50  0001 C CNN
+	1    11100 7425
+	1    0    0    -1
+$EndComp
+Text Label 10500 7275 2    50   ~ 0
+GND
+Text Label 11325 7050 0    50   ~ 0
+PUSH_SW1
+$Comp
+L Switch:SW_Push SW2
+U 1 1 5E7B1BB4
+P 10700 7275
+F 0 "SW2" H 10700 7560 50  0000 C CNN
+F 1 "SW_Push" H 10700 7469 50  0000 C CNN
+F 2 "keyswitches:MX" H 10700 7475 50  0001 C CNN
+F 3 "~" H 10700 7475 50  0001 C CNN
+	1    10700 7275
+	1    0    0    -1
+$EndComp
+Wire Wire Line
+	11100 7275 10975 7275
+Wire Wire Line
+	10975 7275 10975 7150
+Wire Wire Line
+	10975 7150 11150 7150
+Wire Wire Line
+	11150 7150 11150 7050
+Wire Wire Line
+	11150 7050 11325 7050
+Connection ~ 10975 7275
+Wire Wire Line
+	10975 7275 10900 7275
+Text Label 7650 5200 2    50   ~ 0
+PUSH_SW1
+$Comp
+L LED:WS2812B D5
+U 1 1 5E7C5A74
+P 9650 8700
+F 0 "D5" H 9800 8400 50  0000 L CNN
+F 1 "WS2812B" H 9800 8300 50  0000 L CNN
+F 2 "LED_SMD:LED_WS2812B_PLCC4_5.0x5.0mm_P3.2mm" H 9700 8400 50  0001 L TNN
+F 3 "https://cdn-shop.adafruit.com/datasheets/WS2812B.pdf" H 9750 8325 50  0001 L TNN
+	1    9650 8700
+	-1   0    0    1
+$EndComp
+Text Label 9650 8400 1    50   ~ 0
+GND
+$Comp
+L Device:C C12
+U 1 1 5E7C5A7B
+P 9900 9400
+F 0 "C12" H 10015 9446 50  0000 L CNN
+F 1 "0.1uF" H 10015 9355 50  0000 L CNN
+F 2 "Capacitor_SMD:C_1206_3216Metric_Pad1.42x1.75mm_HandSolder" H 9938 9250 50  0001 C CNN
+F 3 "~" H 9900 9400 50  0001 C CNN
+	1    9900 9400
+	1    0    0    -1
+$EndComp
+Text Label 9650 9350 3    50   ~ 0
+5v
+Wire Wire Line
+	9650 9000 9650 9250
+Wire Wire Line
+	9900 9250 9650 9250
+Connection ~ 9650 9250
+Wire Wire Line
+	9650 9250 9650 9350
+Wire Wire Line
+	10150 8700 9950 8700
+Text Label 9900 9550 3    50   ~ 0
+GND
+$Comp
+L LED:WS2812B D4
+U 1 1 5E7CAC28
+P 8850 8700
+F 0 "D4" H 9000 8400 50  0000 L CNN
+F 1 "WS2812B" H 9000 8300 50  0000 L CNN
+F 2 "LED_SMD:LED_WS2812B_PLCC4_5.0x5.0mm_P3.2mm" H 8900 8400 50  0001 L TNN
+F 3 "https://cdn-shop.adafruit.com/datasheets/WS2812B.pdf" H 8950 8325 50  0001 L TNN
+	1    8850 8700
+	-1   0    0    1
+$EndComp
+Text Label 8850 8400 1    50   ~ 0
+GND
+$Comp
+L Device:C C11
+U 1 1 5E7CAC2F
+P 9100 9400
+F 0 "C11" H 9215 9446 50  0000 L CNN
+F 1 "0.1uF" H 9215 9355 50  0000 L CNN
+F 2 "Capacitor_SMD:C_1206_3216Metric_Pad1.42x1.75mm_HandSolder" H 9138 9250 50  0001 C CNN
+F 3 "~" H 9100 9400 50  0001 C CNN
+	1    9100 9400
+	1    0    0    -1
+$EndComp
+Text Label 8850 9350 3    50   ~ 0
+5v
+Wire Wire Line
+	8850 9000 8850 9250
+Wire Wire Line
+	9100 9250 8850 9250
+Connection ~ 8850 9250
+Wire Wire Line
+	8850 9250 8850 9350
+Wire Wire Line
+	9350 8700 9150 8700
+Text Label 9100 9550 3    50   ~ 0
+GND
 $EndSCHEMATC

Commit message: finished schematic
Parts:
- removed SW1, SW2: SW_Push, keyswitches:MX, symbol Switch:SW_Push
- added SW1, SW2: TL3315NF160Q, misc:KSC_SW, symbol dk_Tactile-Switches:TL3315NF160Q
- MH1, MH2, MH3, MH4: footprint MountingHole:MountingHole_4.3mm_M4 -> MountingHole:MountingHole_3.2mm_M3
- R17, R19: value R -> R_PULL_UP; footprint Resistor_THT:R_Axial_DIN0309_L9.0mm_D3.2mm_P12.70mm_Horizontal -> Resistor_SMD:R_1206_3216Metric_Pad1.42x1.75mm_HandSolder
- R20: value R -> R_BZ
Connections:
- wire segments 151 -> 163
- no-connect marks 28 -> 32
Changed lines of the file:
@@
 P 15200 7050
 F 0 "R20" V 14993 7050 50  0000 C CNN
-F 1 "R" V 15084 7050 50  0000 C CNN
+F 1 "R_BZ" V 15084 7050 50  0000 C CNN
 F 2 "Resistor_SMD:R_1206_3216Metric_Pad1.42x1.75mm_HandSolder" V 15130 7050 50  0001 C CNN
 F 3 "~" H 15200 7050 50  0001 C CNN
@@
 P 12575 7450
 F 0 "R17" H 12645 7496 50  0000 L CNN
-F 1 "R" H 12645 7405 50  0000 L CNN
-F 2 "Resistor_THT:R_Axial_DIN0309_L9.0mm_D3.2mm_P12.70mm_Horizontal" V 12505 7450 50  0001 C CNN
+F 1 "R_PULL_UP" H 12645 7405 50  0000 L CNN
+F 2 "Resistor_SMD:R_1206_3216Metric_Pad1.42x1.75mm_HandSolder" V 12505 7450 50  0001 C CNN
 F 3 "~" H 12575 7450 50  0001 C CNN
 	1    12575 7450
@@
 Text Label 12800 7075 0    50   ~ 0
 PUSH_SW
-$Comp
-L Switch:SW_Push SW1
-U 1 1 5D2BB906
-P 12175 7300
-F 0 "SW1" H 12175 7585 50  0000 C CNN
-F 1 "SW_Push" H 12175 7494 50  0000 C CNN
-F 2 "keyswitches:MX" H 12175 7500 50  0001 C CNN
-F 3 "~" H 12175 7500 50  0001 C CNN
-	1    12175 7300
-	1    0    0    -1
-$EndComp
 Wire Wire Line
 	12575 7300 12450 7300
@@
 U 1 1 5E798BF8
 P 13700 6900
-F 0 "R18" H 13525 6950 50  0000 L CNN
+F 0 "R18" H 13475 6950 50  0000 L CNN
 F 1 "4.7k" H 13475 6850 50  0000 L CNN
 F 2 "Resistor_SMD:R_1206_3216Metric_Pad1.42x1.75mm_HandSolder" V 13630 6900 50  0001 C CNN
@@
 F 0 "MH4" H 14900 5921 50  0000 L CNN
 F 1 "M4" H 14900 5830 50  0000 L CNN
-F 2 "MountingHole:MountingHole_4.3mm_M4" H 14800 5875 50  0001 C CNN
+F 2 "MountingHole:MountingHole_3.2mm_M3" H 14800 5875 50  0001 C CNN
 F 3 "~" H 14800 5875 50  0001 C CNN
 	1    14800 5875
@@
 F 0 "MH2" H 14075 5946 50  0000 L CNN
 F 1 "M4" H 14075 5855 50  0000 L CNN
-F 2 "MountingHole:MountingHole_4.3mm_M4" H 13975 5900 50  0001 C CNN
+F 2 "MountingHole:MountingHole_3.2mm_M3" H 13975 5900 50  0001 C CNN
 F 3 "~" H 13975 5900 50  0001 C CNN
 	1    13975 5900
@@
 F 0 "MH1" H 14075 5546 50  0000 L CNN
 F 1 "M4" H 14075 5455 50  0000 L CNN
-F 2 "MountingHole:MountingHole_4.3mm_M4" H 13975 5500 50  0001 C CNN
+F 2 "MountingHole:MountingHole_3.2mm_M3" H 13975 5500 50  0001 C CNN
 F 3 "~" H 13975 5500 50  0001 C CNN
 	1    13975 5500
@@
 F 0 "MH3" H 14900 5546 50  0000 L CNN
 F 1 "M4" H 14900 5455 50  0000 L CNN
-F 2 "MountingHole:MountingHole_4.3mm_M4" H 14800 5500 50  0001 C CNN
+F 2 "MountingHole:MountingHole_3.2mm_M3" H 14800 5500 50  0001 C CNN
 F 3 "~" H 14800 5500 50  0001 C CNN
 	1    14800 5500
@@
 Text Label 12425 3675 2    50   ~ 0
 vBatt
-Text Label 11100 7575 3    50   ~ 0
+Text Label 12550 6575 3    50   ~ 0
 3.3v
 $Comp
 L Device:R R19
 U 1 1 5E7B1BAC
-P 11100 7425
-F 0 "R19" H 11170 7471 50  0000 L CNN
-F 1 "R" H 11170 7380 50  0000 L CNN
-F 2 "Resistor_THT:R_Axial_DIN0309_L9.0mm_D3.2mm_P12.70mm_Horizontal" V 11030 7425 50  0001 C CNN
-F 3 "~" H 11100 7425 50  0001 C CNN
-	1    11100 7425
-	1    0    0    -1
-$EndComp
-Text Label 10500 7275 2    50   ~ 0
-GND
-Text Label 11325 7050 0    50   ~ 0
+P 12550 6425
+F 0 "R19" H 12620 6471 50  0000 L CNN
+F 1 "R_PULL_UP" H 12620 6380 50  0000 L CNN
+F 2 "Resistor_SMD:R_1206_3216Metric_Pad1.42x1.75mm_HandSolder" V 12480 6425 50  0001 C CNN
+F 3 "~" H 12550 6425 50  0001 C CNN
+	1    12550 6425
+	1    0    0    -1
+$EndComp
+Text Label 11950 6275 2    50   ~ 0
+GND
+Text Label 12775 6050 0    50   ~ 0
 PUSH_SW1
-$Comp
-L Switch:SW_Push SW2
-U 1 1 5E7B1BB4
-P 10700 7275
-F 0 "SW2" H 10700 7560 50  0000 C CNN
-F 1 "SW_Push" H 10700 7469 50  0000 C CNN
-F 2 "keyswitches:MX" H 10700 7475 50  0001 C CNN
-F 3 "~" H 10700 7475 50  0001 C CNN
-	1    10700 7275
-	1    0    0    -1
-$EndComp
-Wire Wire Line
-	11100 7275 10975 7275
-Wire Wire Line
-	10975 7275 10975 7150
-Wire Wire Line
-	10975 7150 11150 7150
-Wire Wire Line
-	11150 7150 11150 7050
-Wire Wire Line
-	11150 7050 11325 7050
-Connection ~ 10975 7275
-Wire Wire Line
-	10975 7275 10900 7275
+Wire Wire Line
+	12550 6275 12425 6275
+Wire Wire Line
+	12425 6275 12425 6150
+Wire Wire Line
+	12425 6150 12600 6150
+Wire Wire Line
+	12600 6150 12600 6050
+Wire Wire Line
+	12600 6050 12775 6050
+Connection ~ 12425 6275
+Wire Wire Line
+	12425 6275 12350 6275
 Text Label 7650 5200 2    50   ~ 0
 PUSH_SW1
@@
 Text Label 9100 9550 3    50   ~ 0
 GND
+Wire Wire Line
+	13900 6700 13900 6475
+Wire Wire Line
+	13900 6475 14125 6475
+Wire Wire Line
+	14125 6325 14400 6325
+Wire Wire Line
+	14125 6575 14400 6575
+Wire Wire Line
+	14125 6325 14125 6475
+Connection ~ 14125 6475
+Wire Wire Line
+	14125 6475 14125 6575
+Wire Wire Line
+	13700 6750 13700 6525
+Wire Wire Line
+	13700 6525 13500 6525
+Wire Wire Line
+	13500 6525 13500 6350
+Wire Wire Line
+	13500 6350 13300 6350
+Wire Wire Line
+	13500 6525 13500 6675
+Wire Wire Line
+	13500 6675 13325 6675
+Connection ~ 13500 6525
+Text Label 14400 6325 0    50   ~ 0
+5v
+Text Label 13300 6350 2    50   ~ 0
+5v
+Text Label 13325 6675 2    50   ~ 0
+3.3v
+Text Label 14400 6575 0    50   ~ 0
+3.3v
+$Comp
+L dk_Tactile-Switches:TL3315NF160Q SW2
+U 1 1 5E82A741
+P 12150 6175
+F 0 "SW2" H 12150 6522 60  0000 C CNN
+F 1 "TL3315NF160Q" H 12150 6416 60  0000 C CNN
+F 2 "misc:KSC_SW" H 12350 6375 60  0001 L CNN
+F 3 "http://spec_sheets.e-switch.com/specs/P010337.pdf" H 12350 6475 60  0001 L CNN
+F 4 "EG4621CT-ND" H 12350 6575 60  0001 L CNN "Digi-Key_PN"
+F 5 "TL3315NF160Q" H 12350 6675 60  0001 L CNN "MPN"
+F 6 "Switches" H 12350 6775 60  0001 L CNN "Category"
+F 7 "Tactile Switches" H 12350 6875 60  0001 L CNN "Family"
+F 8 "http://spec_sheets.e-switch.com/specs/P010337.pdf" H 12350 6975 60  0001 L CNN "DK_Datasheet_Link"
+F 9 "/product-detail/en/e-switch/TL3315NF160Q/EG4621CT-ND/1870401" H 12350 7075 60  0001 L CNN "DK_Detail_Page"
+F 10 "SWITCH TACTILE SPST-NO 0.05A 15V" H 12350 7175 60  0001 L CNN "Description"
+F 11 "E-Switch" H 12350 7275 60  0001 L CNN "Manufacturer"
+F 12 "Active" H 12350 7375 60  0001 L CNN "Status"
+	1    12150 6175
+	1    0    0    -1
+$EndComp
+$Comp
+L dk_Tactile-Switches:TL3315NF160Q SW1
+U 1 1 5E82ABEF
+P 12175 7200
+F 0 "SW1" H 12175 7547 60  0000 C CNN
+F 1 "TL3315NF160Q" H 12175 7441 60  0000 C CNN
+F 2 "misc:KSC_SW" H 12375 7400 60  0001 L CNN
+F 3 "http://spec_sheets.e-switch.com/specs/P010337.pdf" H 12375 7500 60  0001 L CNN
+F 4 "EG4621CT-ND" H 12375 7600 60  0001 L CNN "Digi-Key_PN"
+F 5 "TL3315NF160Q" H 12375 7700 60  0001 L CNN "MPN"
+F 6 "Switches" H 12375 7800 60  0001 L CNN "Category"
+F 7 "Tactile Switches" H 12375 7900 60  0001 L CNN "Family"
+F 8 "http://spec_sheets.e-switch.com/specs/P010337.pdf" H 12375 8000 60  0001 L CNN "DK_Datasheet_Link"
+F 9 "/product-detail/en/e-switch/TL3315NF160Q/EG4621CT-ND/1870401" H 12375 8100 60  0001 L CNN "DK_Detail_Page"
+F 10 "SWITCH TACTILE SPST-NO 0.05A 15V" H 12375 8200 60  0001 L CNN "Description"
+F 11 "E-Switch" H 12375 8300 60  0001 L CNN "Manufacturer"
+F 12 "Active" H 12375 8400 60  0001 L CNN "Status"
+	1    12175 7200
+	1    0    0    -1
+$EndComp
+NoConn ~ 11950 6075
+NoConn ~ 11975 7100
+NoConn ~ 12375 7100
+NoConn ~ 12350 6075
 $EndSCHEMATC

Commit message: fixed drc errors on schematic
Connections:
- no-connect marks 32 -> 34
Changed lines of the file:
@@
 NoConn ~ 12375 7100
 NoConn ~ 12350 6075
+NoConn ~ 13075 3625
+Text Label 14325 3725 3    50   ~ 0
+GND
+NoConn ~ 8550 8700
 $EndSCHEMATC
