File: pcb_files/mouse/mouse.sch (KiCad schematic (older format))
At the start: 72 parts, among them J2 BT_Conn, J4 I2C_Conn, M1 Motor_DC, M2 Motor_DC, M3 CASTER_BALL, Q0 Q_Photo_NPN, Q1 Q_Photo_NPN, Q2 Q_Photo_NPN, Q3 Q_Photo_NPN, SW1 TL3315NF160Q, SW2 TL3315NF160Q, T0 Q_NMOS_DGS, T1 Q_NMOS_DGS, T2 Q_NMOS_DGS, T3 Q_NMOS_DGS, U1 Teensy3.2, U2 SN754410NE, U3 LM1084-5.0, U4 Encoder_3081, U5 Encoder_3081

Commit message: reworked mouse shape
Parts:
- MH1, MH2, MH3, MH4: value M4 -> M3
Changed lines of the file:
@@
 P 14800 5875
 F 0 "MH4" H 14900 5921 50  0000 L CNN
-F 1 "M4" H 14900 5830 50  0000 L CNN
+F 1 "M3" H 14900 5830 50  0000 L CNN
 F 2 "MountingHole:MountingHole_3.2mm_M3" H 14800 5875 50  0001 C CNN
 F 3 "~" H 14800 5875 50  0001 C CNN
@@
 P 13975 5900
 F 0 "MH2" H 14075 5946 50  0000 L CNN
-F 1 "M4" H 14075 5855 50  0000 L CNN
+F 1 "M3" H 14075 5855 50  0000 L CNN
 F 2 "MountingHole:MountingHole_3.2mm_M3" H 13975 5900 50  0001 C CNN
 F 3 "~" H 13975 5900 50  0001 C CNN
@@
 P 13975 5500
 F 0 "MH1" H 14075 5546 50  0000 L CNN
-F 1 "M4" H 14075 5455 50  0000 L CNN
+F 1 "M3" H 14075 5455 50  0000 L CNN
 F 2 "MountingHole:MountingHole_3.2mm_M3" H 13975 5500 50  0001 C CNN
 F 3 "~" H 13975 5500 50  0001 C CNN
@@
 P 14800 5500
 F 0 "MH3" H 14900 5546 50  0000 L CNN
-F 1 "M4" H 14900 5455 50  0000 L CNN
+F 1 "M3" H 14900 5455 50  0000 L CNN
 F 2 "MountingHole:MountingHole_3.2mm_M3" H 14800 5500 50  0001 C CNN
 F 3 "~" H 14800 5500 50  0001 C CNN
