File: pcb_files/mouse/mouse.kicad_pcb (KiCad board)
At the start: 2 copper layers, 23 parts, among them Q0 Q_Photo_NPN, Q1 Q_Photo_NPN, Q2 Q_Photo_NPN, Q3 Q_Photo_NPN, U1 Teensy3.2, U2 SN754410NE, U3 LM1084-5.0, U4 Encoder_3081, U5 Encoder_3081, U6 NRF24L01_Breakout

Commit message: caster ball footprint
Parts:
- added M1: Motor_DC, misc:Motor_mouse, F.Cu at (172.7, 77.4)
- added M2: Motor_DC, misc:Motor_mouse, F.Cu at (219.1, 77.4)
- added M3: Motor_DC, misc:Mouse_caster, F.Cu at (221.8, 50.7)
Changed lines of the file:
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@@
     (tracks 0)
     (zones 0)
-    (modules 23)
+    (modules 26)
     (nets 74)
   )
@@
     )
   )
+  (module misc:Motor_mouse (layer F.Cu)
+    (at 172.744801 77.435301)
+    (fp_text reference M1 (at 0 3) (layer F.SilkS)
+      (effects (font (size 1 1) (thickness 0.15)))
+    )
+    (fp_text value Motor_DC (at 0 1.5) (layer F.Fab)
+      (effects (font (size 1 1) (thickness 0.15)))
+    )
+    (fp_line (start 0 0) (end 0 6) (layer F.SilkS) (width 0.15))
+    (fp_line (start 0 0) (end 0 -6) (layer F.SilkS) (width 0.15))
+    (fp_line (start 0 -6) (end -31 -6) (layer F.SilkS) (width 0.15))
+    (fp_line (start 0 6) (end -31 6) (layer F.SilkS) (width 0.15))
+    (fp_line (start -31 -6) (end -31 -1.5) (layer F.SilkS) (width 0.15))
+    (fp_line (start -31 6) (end -31 1.5) (layer F.SilkS) (width 0.15))
+    (fp_line (start -31 -1.5) (end -41 -1.5) (layer F.SilkS) (width 0.15))
+    (fp_line (start -31 1.5) (end -41 1.5) (layer F.SilkS) (width 0.15))
+    (fp_line (start -41 -1.5) (end -41 1.5) (layer F.SilkS) (width 0.15))
+    (fp_line (start -32.2 0) (end -32.2 -14) (layer F.SilkS) (width 0.15))
+    (fp_line (start -32.2 0) (end -32.2 14) (layer F.SilkS) (width 0.15))
+    (fp_line (start -32.2 -14) (end -46 -14) (layer F.SilkS) (width 0.15))
+    (fp_line (start -32.2 14) (end -46 14) (layer F.SilkS) (width 0.15))
+    (fp_line (start -46 -14) (end -46 14) (layer F.SilkS) (width 0.15))
+    (fp_line (start -22.5 6) (end -22.5 13.3) (layer F.SilkS) (width 0.15))
+    (fp_line (start -22.5 -6) (end -22.5 -13.3) (layer F.SilkS) (width 0.15))
+    (fp_line (start -31 0) (end -31 13.3) (layer F.SilkS) (width 0.15))
+    (fp_line (start -31 0) (end -31 -13.3) (layer F.SilkS) (width 0.15))
+    (fp_line (start -31 -13.3) (end -22.5 -13.3) (layer F.SilkS) (width 0.15))
+    (fp_line (start -31 13.3) (end -22.5 13.3) (layer F.SilkS) (width 0.15))
+    (fp_line (start -19.5 0) (end -19.5 7.5) (layer F.SilkS) (width 0.15))
+    (fp_line (start -19.5 0) (end -19.5 -7.5) (layer F.SilkS) (width 0.15))
+    (fp_line (start -31 -7.5) (end -19.5 -7.5) (layer F.SilkS) (width 0.15))
+    (fp_line (start -31 7.5) (end -19.5 7.5) (layer F.SilkS) (width 0.15))
+    (pad "" np_thru_hole circle (at -26.75 -9) (size 2.1844 2.1844) (drill 2.1844) (layers *.Cu *.Mask))
+    (pad "" np_thru_hole circle (at -26.75 9) (size 2.1844 2.1844) (drill 2.1844) (layers *.Cu *.Mask))
+  )
+  (module misc:Motor_mouse (layer F.Cu)
+    (at 219.064801 77.435301)
+    (fp_text reference M2 (at 3.464599 4.212999) (layer F.SilkS)
+      (effects (font (size 1 1) (thickness 0.15)))
+    )
+    (fp_text value Motor_DC (at 0 1.5) (layer F.Fab)
+      (effects (font (size 1 1) (thickness 0.15)))
+    )
+    (fp_line (start -31 7.5) (end -19.5 7.5) (layer F.SilkS) (width 0.15))
+    (fp_line (start -31 -7.5) (end -19.5 -7.5) (layer F.SilkS) (width 0.15))
+    (fp_line (start -19.5 0) (end -19.5 -7.5) (layer F.SilkS) (width 0.15))
+    (fp_line (start -19.5 0) (end -19.5 7.5) (layer F.SilkS) (width 0.15))
+    (fp_line (start -31 13.3) (end -22.5 13.3) (layer F.SilkS) (width 0.15))
+    (fp_line (start -31 -13.3) (end -22.5 -13.3) (layer F.SilkS) (width 0.15))
+    (fp_line (start -31 0) (end -31 -13.3) (layer F.SilkS) (width 0.15))
+    (fp_line (start -31 0) (end -31 13.3) (layer F.SilkS) (width 0.15))
+    (fp_line (start -22.5 -6) (end -22.5 -13.3) (layer F.SilkS) (width 0.15))
+    (fp_line (start -22.5 6) (end -22.5 13.3) (layer F.SilkS) (width 0.15))
+    (fp_line (start -46 -14) (end -46 14) (layer F.SilkS) (width 0.15))
+    (fp_line (start -32.2 14) (end -46 14) (layer F.SilkS) (width 0.15))
+    (fp_line (start -32.2 -14) (end -46 -14) (layer F.SilkS) (width 0.15))
+    (fp_line (start -32.2 0) (end -32.2 14) (layer F.SilkS) (width 0.15))
+    (fp_line (start -32.2 0) (end -32.2 -14) (layer F.SilkS) (width 0.15))
+    (fp_line (start -41 -1.5) (end -41 1.5) (layer F.SilkS) (width 0.15))
+    (fp_line (start -31 1.5) (end -41 1.5) (layer F.SilkS) (width 0.15))
+    (fp_line (start -31 -1.5) (end -41 -1.5) (layer F.SilkS) (width 0.15))
+    (fp_line (start -31 6) (end -31 1.5) (layer F.SilkS) (width 0.15))
+    (fp_line (start -31 -6) (end -31 -1.5) (layer F.SilkS) (width 0.15))
+    (fp_line (start 0 6) (end -31 6) (layer F.SilkS) (width 0.15))
+    (fp_line (start 0 -6) (end -31 -6) (layer F.SilkS) (width 0.15))
+    (fp_line (start 0 0) (end 0 -6) (layer F.SilkS) (width 0.15))
+    (fp_line (start 0 0) (end 0 6) (layer F.SilkS) (width 0.15))
+    (pad "" np_thru_hole circle (at -26.75 9) (size 2.1844 2.1844) (drill 2.1844) (layers *.Cu *.Mask))
+    (pad "" np_thru_hole circle (at -26.75 -9) (size 2.1844 2.1844) (drill 2.1844) (layers *.Cu *.Mask))
+  )
+  (module misc:Mouse_caster (layer F.Cu)
+    (at 221.8309 50.6857)
+    (fp_text reference M3 (at 0 7.8) (layer F.SilkS)
+      (effects (font (size 1 1) (thickness 0.15)))
+    )
+    (fp_text value Motor_DC (at 0.1 9.5) (layer F.Fab)
+      (effects (font (size 1 1) (thickness 0.15)))
+    )
+    (fp_line (start 0 0) (end 6.75 0) (layer F.SilkS) (width 0.15))
+    (fp_line (start 0 0) (end -6.75 0) (layer F.SilkS) (width 0.15))
+    (fp_line (start 0 0) (end 0 -6.1) (layer F.SilkS) (width 0.15))
+    (fp_line (start 0 0) (end 0 6.1) (layer F.SilkS) (width 0.15))
+    (fp_line (start 0 -6.1) (end -9.6 -6.1) (layer F.SilkS) (width 0.15))
+    (fp_line (start 0 -6.1) (end 9.6 -6.1) (layer F.SilkS) (width 0.15))
+    (fp_line (start 0 6.1) (end 9.6 6.1) (layer F.SilkS) (width 0.15))
+    (fp_line (start 0 6.1) (end -9.6 6.1) (layer F.SilkS) (width 0.15))
+    (fp_line (start 9.6 6.1) (end 9.6 -6.1) (layer F.SilkS) (width 0.15))
+    (fp_line (start -9.6 6.1) (end -9.6 -6.1) (layer F.SilkS) (width 0.15))
+    (pad "" np_thru_hole circle (at 6.75 0) (size 2.1844 2.1844) (drill 2.1844) (layers *.Cu *.Mask))
+    (pad "" np_thru_hole circle (at -6.75 0) (size 2.1844 2.1844) (drill 2.1844) (layers *.Cu *.Mask))
+  )
 )

Commit message: started basic layout
Parts:
- moved M3 111.0 mm to (159.0, 142.2)
- moved D0 67.8 mm to (202.9, 115.0), turned to 90 degrees
- moved U4 65.7 mm to (163.1, 61.2), turned to 270 degrees
- moved R0 63.5 mm to (197.8, 112.5), turned to 270 degrees
- moved U5 62.2 mm to (153.1, 59.2), turned to 90 degrees
- moved M2 59.5 mm to (160.0, 69.7), turned to 180 degrees
- moved U6 59.4 mm to (185.5, 87.7)
- moved R1 56.5 mm to (184.7, 135.1), turned to 180 degrees
- moved Q2 56.3 mm to (119.4, 107.9), turned to 270 degrees
- moved D1 45.2 mm to (182.5, 138.3)
- moved R7 45.1 mm to (134.5, 135.7)
- moved U3 43.5 mm to (134.6, 89.6)
- moved BT1 42.4 mm to (128.5, 88.0)
- moved R6 39.6 mm to (122.6, 110.2), turned to 90 degrees
- moved U2 39.5 mm to (166.4, 73.2), turned to 90 degrees
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Other:
- board outline added: 94.7 x 93.9 mm

Commit message: update
Parts:
- moved U2 7.76 mm to (166.4, 65.4)
Changed lines of the file:
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@@
   (general
     (thickness 1.6)
-    (drawings 10)
+    (drawings 12)
     (tracks 0)
     (zones 0)
@@
   )
   (module SN754410NE.kicad_mod:DIP254P762X508-16 (layer F.Cu)
-    (at 166.3573 73.1647 90)
+    (at 166.37 65.405 90)
     (fp_text reference U2 (at -4.57256 -20.297 90) (layer F.SilkS)
       (effects (font (size 1.6402 1.6402) (thickness 0.05)))
@@
     (pad "" np_thru_hole circle (at -6.75 0) (size 2.1844 2.1844) (drill 2.1844) (layers *.Cu *.Mask))
   )
+  (dimension 99.579663 (width 0.3) (layer Dwgs.User)
+    (gr_text "99.580 mm" (at 246.925839 105.237574 89.12309226) (layer Dwgs.User)
+      (effects (font (size 1.5 1.5) (thickness 0.3)))
+    )
+    (feature1 (pts (xy 157.861 153.67) (xy 244.650437 154.99841)))
+    (feature2 (pts (xy 159.385 54.102) (xy 246.174437 55.43041)))
+    (crossbar (pts (xy 245.588085 55.421435) (xy 244.064085 154.989435)))
+    (arrow1a (pts (xy 244.064085 154.989435) (xy 243.494973 153.854088)))
+    (arrow1b (pts (xy 244.064085 154.989435) (xy 244.667677 153.872038)))
+    (arrow2a (pts (xy 245.588085 55.421435) (xy 244.984493 56.538832)))
+    (arrow2b (pts (xy 245.588085 55.421435) (xy 246.157197 56.556782)))
+  )
+  (dimension 100.965319 (width 0.3) (layer Dwgs.User)
+    (gr_text "100.965 mm" (at 157.245557 41.714466 0.1441400217) (layer Dwgs.User)
+      (effects (font (size 1.5 1.5) (thickness 0.3)))
+    )
+    (feature1 (pts (xy 106.807 59.309) (xy 106.766864 43.35504)))
+    (feature2 (pts (xy 207.772 59.055) (xy 207.731864 43.10104)))
+    (crossbar (pts (xy 207.73334 43.687459) (xy 106.76834 43.941459)))
+    (arrow1a (pts (xy 106.76834 43.941459) (xy 107.893365 43.352206)))
+    (arrow1b (pts (xy 106.76834 43.941459) (xy 107.896315 44.525044)))
+    (arrow2a (pts (xy 207.73334 43.687459) (xy 206.605365 43.103874)))
+    (arrow2b (pts (xy 207.73334 43.687459) (xy 206.608315 44.276712)))
+  )
   (gr_line (start 124.448629 100.019819) (end 194.298629 100.019819) (layer Edge.Cuts) (width 0.15))

Commit message: removed wirless module
Changed lines of the file:
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@@
-(kicad_pcb (version 20171130) (host pcbnew "(5.0.0-3-g5ebb6b6)")
+(kicad_pcb (version 20171130) (host pcbnew "(5.1.2)-2")
   (general
     (thickness 1.6)
@@
     (zone_45_only no)
     (trace_min 0.2)
-    (segment_width 0.2)
-    (edge_width 0.15)
     (via_size 0.8)
     (via_drill 0.4)
@@
     (uvia_min_size 0.2)
     (uvia_min_drill 0.1)
+    (edge_width 0.15)
+    (segment_width 0.2)
     (pcb_text_width 0.3)
     (pcb_text_size 1.5 1.5)
@@
     (pad_to_mask_clearance 0.2)
     (aux_axis_origin 0 0)
-    (visible_elements FFFFFF7F)
+    (visible_elements 7FFFFFFF)
     (pcbplotparams
       (layerselection 0x010fc_ffffffff)
@@
     (fp_line (start -3.5052 -18.7452) (end -4.1148 -18.7452) (layer F.SilkS) (width 0.1524))
     (fp_line (start -4.1148 -18.7452) (end -6.2992 -18.7452) (layer F.SilkS) (width 0.1524))
-    (fp_arc (start -3.81 -18.7452) (end -4.1148 -18.7452) (angle -180) (layer F.SilkS) (width 0))
+    (fp_arc (start -3.81 -18.7452) (end -4.1148 -18.7452) (angle -180) (layer F.SilkS) (width 0.1))
     (fp_line (start -7.112 -17.2212) (end -7.112 -18.3388) (layer Eco2.User) (width 0.1524))
     (fp_line (start -7.112 -18.3388) (end -8.1788 -18.3388) (layer Eco2.User) (width 0.1524))
@@
     (fp_line (start -4.1148 -18.7452) (end -7.112 -18.7452) (layer Eco2.User) (width 0.1524))
     (fp_line (start -7.112 -18.7452) (end -7.112 0.9652) (layer Eco2.User) (width 0.1524))
-    (fp_arc (start -3.81 -18.7452) (end -4.1148 -18.7452) (angle -180) (layer Eco2.User) (width 0))
+    (fp_arc (start -3.81 -18.7452) (end -4.1148 -18.7452) (angle -180) (layer Eco2.User) (width 0.1))
     (pad 1 thru_hole rect (at -7.62 -17.78 90) (size 1.6764 1.6764) (drill 1.1176) (layers *.Cu *.Mask)
       (net 24 /M1_speed))

Commit message: update
Parts:
- removed U6: NRF24L01_Breakout, Connector_PinSocket_2.54mm:PinSocket_2x04_P2.54mm_Vertical
- added BZ1: Buzzer, misc:9x5.5mm Buzzer, F.Cu at (174.5, 69.2)
- added D4: STATUS_0, misc:3528_SMD_LED, F.Cu at (203.7, 88.4)
- added D5: STATUS_1, misc:3528_SMD_LED, F.Cu at (203.8, 95.5)
- added MH_GND1: MountingHole_Pad, Connector_PinHeader_2.54mm:PinHeader_1x01_P2.54mm_Vertical, F.Cu at (115.7, 103.8)
- added MH_SCL1: MountingHole_Pad, Connector_PinHeader_2.54mm:PinHeader_1x01_P2.54mm_Vertical, F.Cu at (118.6, 102.2)
- added MH_SDA1: MountingHole_Pad, Connector_PinHeader_2.54mm:PinHeader_1x01_P2.54mm_Vertical, F.Cu at (121.7, 102.9)
- added MH_vBatt1: MountingHole_Pad, Connector_PinHeader_2.54mm:PinHeader_1x01_P2.54mm_Vertical, F.Cu at (113.2, 103.5)
- added R10: R, Resistor_THT:R_Axial_DIN0207_L6.3mm_D2.5mm_P2.54mm_Vertical, F.Cu at (183.6, 85.9)
- added R11: R, Resistor_THT:R_Axial_DIN0207_L6.3mm_D2.5mm_P2.54mm_Vertical, F.Cu at (183.8, 89.2)
- added R8: R, Resistor_THT:R_Axial_DIN0207_L6.3mm_D2.5mm_P2.54mm_Vertical, F.Cu at (181.7, 92.3)
- added R9: R, Resistor_THT:R_Axial_DIN0207_L6.3mm_D2.5mm_P2.54mm_Vertical, F.Cu at (201.7, 102.2)
- added SW1: SW_Push, keyswitches:MX, F.Cu at (193.9, 92.3)
- M3: value Motor_DC -> CASTER_BALL
- moved U2 39.6 mm to (133.6, 87.6)
- moved U3 33.4 mm to (149.1, 59.6), turned to 270 degrees
- moved BT1 31.5 mm to (137.8, 57.9)
- moved U5 16.2 mm to (169.3, 59.9)
- moved U1 2.44 mm to (158.5, 85.5)
- moved U4 1.91 mm to (164.2, 59.6)
Connections:
- R2 pad 2: /Emiter_2 -> /Emitter_2
- U1 pad 10: Net-(U1-Pad10) -> /M1_backward
- U1 pad 11: /u1_CE -> /M2_forward
- U1 pad 12: /u1_CS -> /M2_backward
- U1 pad 13: /u1_MOSI -> /Emitter_0
- U1 pad 14: /u1_MISO -> /Emitter_1
- U1 pad 20: /u1_SCK -> Net-(U1-Pad20)
- U1 pad 25: /Emitter_0 -> /i2c_SDA
- U1 pad 26: /Emitter_1 -> /i2c_SCL
- U1 pad 5: Net-(U1-Pad5) -> /STATUS_LED_0
- U1 pad 6: Net-(U1-Pad6) -> /STATUS_LED_1
- U1 pad 7: Net-(U1-Pad7) -> /Buzzer
- U1 pad 9: Net-(U1-Pad9) -> /M1_forward
- U2 pad 16: Net-(U2-Pad16) -> /5v

Commit message: update
Parts:
- U4, U5: footprint Connector_PinHeader_2.00mm:PinHeader_1x06_P2.00mm_Vertical -> Connector_PinSocket_2.54mm:PinSocket_1x06_P2.54mm_Vertical
- moved BT1 18.8 mm to (156.6, 57.8), turned to 90 degrees
- moved U4 14.2 mm to (150.0, 59.6)
- moved U3 11.9 mm to (160.8, 61.7)
- moved U5 1.49 mm to (167.9, 59.4)
- moved MH_vBatt1 0.65 mm to (112.5, 103.4)

Commit message: traces
Parts:
- BZ1, D4, D5, M3, R10, R11, R8, R9, SW1: moved to B.Cu
- moved D5 90.5 mm to (113.7, 102.7), turned to 0 degrees
- moved R9 86.9 mm to (114.8, 98.8), turned to 180 degrees
- moved SW1 74.8 mm to (119.1, 93.0), turned to 180 degrees
- moved R11 70.9 mm to (112.9, 86.6), turned to 270 degrees
- moved MH_GND1 53.8 mm to (169.5, 103.8)
- moved U2 52.3 mm to (185.4, 95.0), turned to 270 degrees
- moved MH_SCL1 42.9 mm to (161.5, 103.3)
- moved MH_vBatt1 37.7 mm to (150.2, 101.9)
- moved MH_SDA1 36.4 mm to (158.1, 102.9)
- moved BT1 33.7 mm to (139.2, 86.6), turned to 0 degrees
- moved R10 33.6 mm to (159.8, 62.2)
- moved U5 31.2 mm to (136.7, 58.9)
- moved R8 23.7 mm to (204.5, 99.1), turned to 180 degrees
- moved U4 17.9 mm to (167.9, 58.9), turned to 90 degrees
- moved BZ1 16.0 mm to (158.5, 68.3)
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Connections:
- R11 pad 1: Net-(R11-Pad1) -> /PUSH_SW
- SW1 pad 2: Net-(R11-Pad1) -> /PUSH_SW
- U1 pad 1: Net-(U1-Pad1) -> /GND
- U1 pad 10: /M1_backward -> /M1_encoder_A
- U1 pad 11: /M2_forward -> /M1_encoder_B
- U1 pad 12: /M2_backward -> /STATUS_LED_0
- U1 pad 13: /Emitter_0 -> /STATUS_LED_1
- U1 pad 14: /Emitter_1 -> /PUSH_SW
- U1 pad 17: Net-(U1-Pad17) -> /GND
- U1 pad 2: Net-(U1-Pad2) -> /M1_backward
- U1 pad 20: Net-(U1-Pad20) -> /Reciever_2
- U1 pad 21: /Reciever_0 -> /Reciever_3
- U1 pad 23: /Reciever_2 -> /Reciever_0
- U1 pad 24: /Reciever_3 -> /Buzzer
- U1 pad 29: /M2_speed -> /Emitter_1
- U1 pad 3: Net-(U1-Pad3) -> /M1_forward
- U1 pad 30: /M1_speed -> /Emitter_0
- U1 pad 4: Net-(R11-Pad1) -> /M2_forward
- U1 pad 5: /STATUS_LED_0 -> /M2_backward
- U1 pad 6: /STATUS_LED_1 -> /M1_speed
- U1 pad 7: /Buzzer -> /M2_speed
- U1 pad 8: Net-(U1-Pad8) -> /M2_encoder_A
- U1 pad 9: /M1_forward -> /M2_encoder_B
- U4 pad 5: /OUT4 -> /OUT3
- U4 pad 6: /OUT3 -> /OUT4
- U5 pad 5: /OUT2 -> /OUT1
- U5 pad 6: /OUT1 -> /OUT2
Routing:
- net /5v: track 0.00 -> 101.7 mm, vias 0 -> 1
- net /STATUS_LED_0: track 0.00 -> 83.5 mm, vias 0 -> 2
- net /OUT1: track 0.00 -> 82.7 mm
- net /OUT2: track 0.00 -> 70.8 mm
- net /STATUS_LED_1: track 0.00 -> 51.8 mm
- net /OUT4: track 0.00 -> 51.4 mm, vias 0 -> 1
- net /M1_speed: track 0.00 -> 46.5 mm
- net /OUT3: track 0.00 -> 45.0 mm
- net /M2_backward: track 0.00 -> 44.5 mm
- net /Emitter_2: track 0.00 -> 41.2 mm
- net /Emitter_3: track 0.00 -> 39.0 mm
- net /PUSH_SW: track 0.00 -> 38.3 mm
- net /Emitter_1: track 0.00 -> 36.2 mm
- net /M1_forward: track 0.00 -> 35.2 mm
- net /M2_speed: track 0.00 -> 35.0 mm
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Other:
- board size 94.7 x 93.9 mm -> 94.7 x 94.9 mm

Commit message: placed ir sensors
Parts:
- R10: moved to F.Cu
- moved R5 19.8 mm to (194.2, 125.9), turned to 65 degrees
- moved D1 18.6 mm to (163.3, 140.5), turned to 63.5 degrees
- moved Q3 18.3 mm to (152.5, 138.3), turned to 296.5 degrees
- moved D3 11.5 mm to (150.3, 133.8), turned to 296.5 degrees
- moved Q1 11.0 mm to (165.5, 136.0), turned to 63.5 degrees
- moved BT1 10.3 mm to (129.0, 88.1)
- moved R2 8.63 mm to (121.3, 107.0), turned to 180 degrees
- moved D0 7.78 mm to (196.3, 110.0), turned to 0 degrees
- moved R6 7.35 mm to (116.0, 107.0), turned to 180 degrees
- moved Q2 6.14 mm to (113.7, 110.2), turned to 0 degrees
- moved R0 5.55 mm to (198.6, 106.2), turned to 180 degrees
- moved R4 3.50 mm to (201.7, 106.2), turned to 0 degrees
- moved D2 3.07 mm to (119.0, 110.1), turned to 0 degrees
- moved M3 2.85 mm to (158.6, 143.8)
- moved Q0 1.83 mm to (201.7, 110.0), turned to 0 degrees
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Routing:
- net /vBatt: track 0.00 -> 62.9 mm, vias 0 -> 1
- net /3.3v: track 0.00 -> 41.5 mm
- net /GND: track 20.3 -> 0.00 mm
- net /5v: track 101.7 -> 117.4 mm
- added copper zone on F.Cu, net /GND
Other:
- outline, holes or cut-outs redrawn
