File: pcb_files/mouse/mouse.kicad_pcb (KiCad board)
At the start: 2 copper layers, 94.7 x 94.9 mm, 37 parts, among them M1 Motor_DC, M2 Motor_DC, M3 CASTER_BALL, Q0 Q_Photo_NPN, Q1 Q_Photo_NPN, Q2 Q_Photo_NPN, Q3 Q_Photo_NPN, SW1 SW_Push, U1 Teensy3.2, U2 SN754410NE, U3 LM1084-5.0, U4 Encoder_3081, U5 Encoder_3081

Commit message: traces finished
Parts:
- moved MH_GND1 39.9 mm to (131.9, 90.6)
- moved R5 34.9 mm to (160.3, 133.8), turned to 270 degrees
- moved R1 25.3 mm to (160.5, 142.7), turned to 270 degrees
- moved MH_vBatt1 22.8 mm to (132.0, 88.1)
- moved R7 22.4 mm to (156.8, 133.8), turned to 270 degrees
- moved R3 15.4 mm to (156.5, 142.7), turned to 270 degrees
- moved D3 5.04 mm to (152.5, 138.3)
- moved Q3 5.01 mm to (150.3, 133.8)
- moved MH_SCL1 4.73 mm to (158.0, 100.1)
- moved MH_SDA1 3.90 mm to (155.4, 100.1)
- moved R6 3.24 mm to (112.9, 105.9), turned to 0 degrees
- moved R2 1.73 mm to (119.6, 106.7), turned to 90 degrees
- moved R0 1.30 mm to (197.4, 106.7), turned to 90 degrees
- moved D2 0.86 mm to (118.4, 109.5)
- moved Q2 0.71 mm to (113.3, 109.5)
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Routing:
- net /3.3v: track 41.5 -> 290.2 mm, vias 0 -> 3
- net /Reciever_0: track 32.6 -> 152.9 mm, vias 0 -> 2
- net /Emitter_2: track 41.2 -> 155.2 mm
- net /Reciever_1: track 30.6 -> 107.2 mm
- net /Emitter_3: track 39.0 -> 107.9 mm
- net /Emitter_1: track 36.2 -> 104.4 mm
- net /Reciever_3: track 28.1 -> 93.7 mm
- net /Buzzer: track 0.00 -> 33.5 mm, vias 0 -> 2
- net /Reciever_2: track 25.5 -> 41.1 mm
- net Net-(D1-Pad2): track 0.00 -> 6.94 mm
- net /i2c_SDA: track 0.00 -> 6.12 mm
- net /i2c_SCL: track 0.00 -> 6.12 mm
- net Net-(D3-Pad2): track 0.00 -> 3.74 mm
- net Net-(D0-Pad2): track 0.00 -> 3.41 mm
- net Net-(D2-Pad2): track 0.00 -> 3.35 mm
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- added copper zone on B.Cu, net /GND
Other:
- outline, holes or cut-outs redrawn

Commit message: cleaned up labels
Parts:
- moved GND 0.18 mm to (132.0, 90.7)
- renumbered MH_vBatt1 to BT, MH_GND1 to GND, MH_SCL1 to SCL, MH_SDA1 to SDA
Other:
- board text added: "GND"

Commit message: LED polarity markings
Parts:
- moved R8 0.76 mm to (204.5, 98.3)
Routing:
- net /3.3v: track 290.2 -> 288.6 mm
- net Net-(D4-Pad2): track 2.89 -> 3.65 mm
Other:
- board text added: "+"
- board text added: "-"
- board text added: "D18"
- board text added: "D19"

Commit message: ldo regulator labels
Other:
- board text added: "IN"
- board text added: "OUT"
Changed lines of the file:
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@@
   (general
     (thickness 1.6)
-    (drawings 45)
+    (drawings 48)
     (tracks 446)
     (zones 0)
@@
     (descr "Through hole straight pin header, 1x03, 2.54mm pitch, single row")
     (tags "Through hole pin header THT 1x03 2.54mm single row")
-    (fp_text reference U3 (at -2.3876 2.5908) (layer F.SilkS)
+    (fp_text reference U3 (at -3.175 2.5908) (layer F.SilkS)
       (effects (font (size 1 1) (thickness 0.15)))
     )
@@
     (descr "Through hole straight socket strip, 1x06, 2.54mm pitch, single row (from Kicad 4.0.7), script generated")
     (tags "Through hole socket strip THT 1x06 2.54mm single row")
-    (fp_text reference U4 (at 2.1844 6.4516 180) (layer F.SilkS)
+    (fp_text reference U4 (at 2.54 6.4516 180) (layer F.SilkS)
       (effects (font (size 1 1) (thickness 0.15)))
     )
@@
     )
   )
+  (gr_text IN (at 155.956 57.15) (layer F.SilkS)
+    (effects (font (size 0.7 0.7) (thickness 0.1)))
+  )
+  (gr_text OUT (at 158.496 57.15) (layer F.SilkS)
+    (effects (font (size 0.7 0.7) (thickness 0.1)))
+  )
+  (gr_text GND (at 161.036 57.15) (layer F.SilkS)
+    (effects (font (size 0.7 0.7) (thickness 0.1)))
+  )
   (gr_text + (at 204.47 100.076) (layer B.SilkS)

Commit message: shifted motors back 3mm
Parts:
- R10: moved to B.Cu
- moved M1 1.02 mm to (157.1, 68.7)
- moved M2 1.02 mm to (160.0, 68.7)
Changed lines of the file:
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@@
   )
   (module misc:Motor_mouse (layer F.Cu)
-    (at 157.1117 69.723)
+    (at 157.099 68.707)
     (fp_text reference M1 (at -11.9253 -7.1882) (layer F.SilkS)
       (effects (font (size 1 1) (thickness 0.15)))
@@
       (effects (font (size 1 1) (thickness 0.15)))
     )
+    (fp_line (start -31 7.5) (end -19.5 7.5) (layer F.SilkS) (width 0.15))
+    (fp_line (start -31 -7.5) (end -19.5 -7.5) (layer F.SilkS) (width 0.15))
+    (fp_line (start -19.5 0) (end -19.5 -7.5) (layer F.SilkS) (width 0.15))
+    (fp_line (start -19.5 0) (end -19.5 7.5) (layer F.SilkS) (width 0.15))
+    (fp_line (start -31 13.3) (end -22.5 13.3) (layer F.SilkS) (width 0.15))
+    (fp_line (start -31 -13.3) (end -22.5 -13.3) (layer F.SilkS) (width 0.15))
+    (fp_line (start -31 0) (end -31 -13.3) (layer F.SilkS) (width 0.15))
+    (fp_line (start -31 0) (end -31 13.3) (layer F.SilkS) (width 0.15))
+    (fp_line (start -22.5 -6) (end -22.5 -13.3) (layer F.SilkS) (width 0.15))
+    (fp_line (start -22.5 6) (end -22.5 13.3) (layer F.SilkS) (width 0.15))
+    (fp_line (start -46 -14) (end -46 14) (layer F.SilkS) (width 0.15))
+    (fp_line (start -32.2 14) (end -46 14) (layer F.SilkS) (width 0.15))
+    (fp_line (start -32.2 -14) (end -46 -14) (layer F.SilkS) (width 0.15))
+    (fp_line (start -32.2 0) (end -32.2 14) (layer F.SilkS) (width 0.15))
+    (fp_line (start -32.2 0) (end -32.2 -14) (layer F.SilkS) (width 0.15))
+    (fp_line (start -41 -1.5) (end -41 1.5) (layer F.SilkS) (width 0.15))
+    (fp_line (start -31 1.5) (end -41 1.5) (layer F.SilkS) (width 0.15))
+    (fp_line (start -31 -1.5) (end -41 -1.5) (layer F.SilkS) (width 0.15))
+    (fp_line (start -31 6) (end -31 1.5) (layer F.SilkS) (width 0.15))
+    (fp_line (start -31 -6) (end -31 -1.5) (layer F.SilkS) (width 0.15))
+    (fp_line (start 0 6) (end -31 6) (layer F.SilkS) (width 0.15))
+    (fp_line (start 0 -6) (end -31 -6) (layer F.SilkS) (width 0.15))
+    (fp_line (start 0 0) (end 0 -6) (layer F.SilkS) (width 0.15))
     (fp_line (start 0 0) (end 0 6) (layer F.SilkS) (width 0.15))
-    (fp_line (start 0 0) (end 0 -6) (layer F.SilkS) (width 0.15))
-    (fp_line (start 0 -6) (end -31 -6) (layer F.SilkS) (width 0.15))
-    (fp_line (start 0 6) (end -31 6) (layer F.SilkS) (width 0.15))
-    (fp_line (start -31 -6) (end -31 -1.5) (layer F.SilkS) (width 0.15))
-    (fp_line (start -31 6) (end -31 1.5) (layer F.SilkS) (width 0.15))
-    (fp_line (start -31 -1.5) (end -41 -1.5) (layer F.SilkS) (width 0.15))
-    (fp_line (start -31 1.5) (end -41 1.5) (layer F.SilkS) (width 0.15))
-    (fp_line (start -41 -1.5) (end -41 1.5) (layer F.SilkS) (width 0.15))
-    (fp_line (start -32.2 0) (end -32.2 -14) (layer F.SilkS) (width 0.15))
-    (fp_line (start -32.2 0) (end -32.2 14) (layer F.SilkS) (width 0.15))
-    (fp_line (start -32.2 -14) (end -46 -14) (layer F.SilkS) (width 0.15))
-    (fp_line (start -32.2 14) (end -46 14) (layer F.SilkS) (width 0.15))
-    (fp_line (start -46 -14) (end -46 14) (layer F.SilkS) (width 0.15))
-    (fp_line (start -22.5 6) (end -22.5 13.3) (layer F.SilkS) (width 0.15))
-    (fp_line (start -22.5 -6) (end -22.5 -13.3) (layer F.SilkS) (width 0.15))
-    (fp_line (start -31 0) (end -31 13.3) (layer F.SilkS) (width 0.15))
-    (fp_line (start -31 0) (end -31 -13.3) (layer F.SilkS) (width 0.15))
-    (fp_line (start -31 -13.3) (end -22.5 -13.3) (layer F.SilkS) (width 0.15))
-    (fp_line (start -31 13.3) (end -22.5 13.3) (layer F.SilkS) (width 0.15))
-    (fp_line (start -19.5 0) (end -19.5 7.5) (layer F.SilkS) (width 0.15))
-    (fp_line (start -19.5 0) (end -19.5 -7.5) (layer F.SilkS) (width 0.15))
-    (fp_line (start -31 -7.5) (end -19.5 -7.5) (layer F.SilkS) (width 0.15))
-    (fp_line (start -31 7.5) (end -19.5 7.5) (layer F.SilkS) (width 0.15))
+    (pad "" np_thru_hole circle (at -26.75 9) (size 2.1844 2.1844) (drill 2.1844) (layers *.Cu *.Mask))
     (pad "" np_thru_hole circle (at -26.75 -9) (size 2.1844 2.1844) (drill 2.1844) (layers *.Cu *.Mask))
-    (pad "" np_thru_hole circle (at -26.75 9) (size 2.1844 2.1844) (drill 2.1844) (layers *.Cu *.Mask))
   )
   (module misc:Motor_mouse (layer F.Cu)
-    (at 160.02 69.723 180)
+    (at 160.02 68.707 180)
     (fp_text reference M2 (at -12.2428 7.4422 180) (layer F.SilkS)
       (effects (font (size 1 1) (thickness 0.15)))
@@
     )
   )
-  (module Resistor_THT:R_Axial_DIN0207_L6.3mm_D2.5mm_P2.54mm_Vertical (layer F.Cu)
+  (module Resistor_THT:R_Axial_DIN0207_L6.3mm_D2.5mm_P2.54mm_Vertical (layer B.Cu)
     (at 159.766 62.23 180)
     (descr "Resistor, Axial_DIN0207 series, Axial, Vertical, pin pitch=2.54mm, 0.25W = 1/4W, length*diameter=6.3*2.5mm^2, http://cdn-reichelt.de/documents/datenblatt/B400/1_4W%23YAG.pdf")
     (tags "Resistor Axial_DIN0207 series Axial Vertical pin pitch 2.54mm 0.25W = 1/4W length 6.3mm diameter 2.5mm")
-    (fp_text reference R10 (at -3.302 0 180) (layer F.SilkS)
-      (effects (font (size 1 1) (thickness 0.15)))
-    )
-    (fp_text value R (at 1.27 2.37 180) (layer F.Fab)
-      (effects (font (size 1 1) (thickness 0.15)))
-    )
-    (fp_text user %R (at 1.27 -2.37 180) (layer F.Fab)
-      (effects (font (size 1 1) (thickness 0.15)))
-    )
-    (fp_line (start 3.59 -1.5) (end -1.5 -1.5) (layer F.CrtYd) (width 0.05))
-    (fp_line (start 3.59 1.5) (end 3.59 -1.5) (layer F.CrtYd) (width 0.05))
-    (fp_line (start -1.5 1.5) (end 3.59 1.5) (layer F.CrtYd) (width 0.05))
-    (fp_line (start -1.5 -1.5) (end -1.5 1.5) (layer F.CrtYd) (width 0.05))
-    (fp_line (start 1.37 0) (end 1.44 0) (layer F.SilkS) (width 0.12))
-    (fp_line (start 0 0) (end 2.54 0) (layer F.Fab) (width 0.1))
-    (fp_circle (center 0 0) (end 1.37 0) (layer F.SilkS) (width 0.12))
-    (fp_circle (center 0 0) (end 1.25 0) (layer F.Fab) (width 0.1))
+    (fp_text reference R10 (at -3.302 0 180) (layer B.SilkS)
+      (effects (font (size 1 1) (thickness 0.15)) (justify mirror))
+    )
+    (fp_text value R (at 1.27 -2.37 180) (layer B.Fab)
+      (effects (font (size 1 1) (thickness 0.15)) (justify mirror))
+    )
+    (fp_text user %R (at 1.27 2.37 180) (layer B.Fab)
+      (effects (font (size 1 1) (thickness 0.15)) (justify mirror))
+    )
+    (fp_line (start 3.59 1.5) (end -1.5 1.5) (layer B.CrtYd) (width 0.05))
+    (fp_line (start 3.59 -1.5) (end 3.59 1.5) (layer B.CrtYd) (width 0.05))
+    (fp_line (start -1.5 -1.5) (end 3.59 -1.5) (layer B.CrtYd) (width 0.05))
+    (fp_line (start -1.5 1.5) (end -1.5 -1.5) (layer B.CrtYd) (width 0.05))
+    (fp_line (start 1.37 0) (end 1.44 0) (layer B.SilkS) (width 0.12))
+    (fp_line (start 0 0) (end 2.54 0) (layer B.Fab) (width 0.1))
+    (fp_circle (center 0 0) (end 1.37 0) (layer B.SilkS) (width 0.12))
+    (fp_circle (center 0 0) (end 1.25 0) (layer B.Fab) (width 0.1))
     (pad 2 thru_hole oval (at 2.54 0 180) (size 1.6 1.6) (drill 0.8) (layers *.Cu *.Mask)
       (net 62 /Buzzer))

Commit message: fixed switch
Parts:
- removed BT, SCL, SDA: MountingHole_Pad, Connector_PinHeader_2.54mm:PinHeader_1x01_P2.54mm_Vertical
- added BAT: MountingHole_Pad, Connector_PinHeader_2.54mm:PinHeader_1x01_P2.54mm_Vertical, F.Cu at (132.6, 88.1)
- added MH_SCL1: MountingHole_Pad, Connector_PinHeader_2.54mm:PinHeader_1x01_P2.54mm_Vertical, F.Cu at (158.0, 100.2)
- added MH_SDA1: MountingHole_Pad, Connector_PinHeader_2.54mm:PinHeader_1x01_P2.54mm_Vertical, F.Cu at (155.6, 100.2)
- moved GND 0.56 mm to (132.6, 90.7)
Connections:
- R11 pad 2: /GND -> /3.3v
- SW1 pad 1: /3.3v -> /GND
Routing:
- net /3.3v: track 288.6 -> 297.3 mm
- net /vBatt: track 65.9 -> 66.5 mm

Commit message: added version label
Parts:
- renumbered MH_SCL1 to SCL, MH_SDA1 to SDA
Other:
- board text added: "version 1.0"
Changed lines of the file:
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@@
   (general
     (thickness 1.6)
-    (drawings 48)
+    (drawings 49)
     (tracks 452)
     (zones 0)
@@
     (descr "Through hole straight pin header, 1x01, 2.54mm pitch, single row")
     (tags "Through hole pin header THT 1x01 2.54mm single row")
-    (fp_text reference MH_SCL1 (at 0 -2.33) (layer F.SilkS)
+    (fp_text reference SCL (at 3.175 0) (layer F.SilkS)
       (effects (font (size 1 1) (thickness 0.15)))
     )
@@
     (descr "Through hole straight pin header, 1x01, 2.54mm pitch, single row")
     (tags "Through hole pin header THT 1x01 2.54mm single row")
-    (fp_text reference MH_SDA1 (at 0 -2.33) (layer F.SilkS)
+    (fp_text reference SDA (at -3.556 -0.127) (layer F.SilkS)
       (effects (font (size 1 1) (thickness 0.15)))
     )
@@
     )
   )
+  (gr_text "version 1.0" (at 127.254 135.382 135) (layer F.SilkS)
+    (effects (font (size 1.5 1.5) (thickness 0.3)))
+  )
   (gr_text IN (at 155.956 57.15) (layer F.SilkS)
