File: pcb_files/mouse/_autosave-mouse_v2.kicad_pcb (KiCad board)
At the start: 2 copper layers, 94.7 x 94.9 mm, 70 parts, among them J2 BT_Conn, J4 I2C_Conn, M1 Motor_DC, M2 Motor_DC, M3 CASTER_BALL, Q0 Q_Photo_NPN, Q1 Q_Photo_NPN, Q2 Q_Photo_NPN, Q3 Q_Photo_NPN, SW1 SW_Push, T0 Q_NMOS_DGS, T1 Q_NMOS_DGS, T2 Q_NMOS_DGS, T3 Q_NMOS_DGS, U1 Teensy3.2, U2 SN754410NE, U4 Encoder_3081, U5 Encoder_3081, U6 LM2596S-5

Commit message: finished schematic
Parts:
- removed D12: 1n5824, Diode_THT:D_DO-201AD_P12.70mm_Horizontal
- removed L1: 22uH, misc:PE-53933SNL
- removed U6: LM2596S-5, Package_TO_SOT_SMD:TO-263-5_TabPin3
- added C11: 0.1uF, Capacitor_SMD:C_1206_3216Metric_Pad1.42x1.75mm_HandSolder, F.Cu at (113.2, 30.1)
- added C12: 0.1uF, Capacitor_SMD:C_1206_3216Metric_Pad1.42x1.75mm_HandSolder, F.Cu at (113.2, 33.9)
- added D4: WS2812B, LED_SMD:LED_WS2812B_PLCC4_5.0x5.0mm_P3.2mm, F.Cu at (119.4, 32.2)
- added SW2: SW_Push, keyswitches:MX, F.Cu at (98.8, 38.8)
- added U3: LM1084-5.0, Package_TO_SOT_SMD:TO-263-3_TabPin2, F.Cu at (158.3, 60.7)
- C10: value 220uF -> 10uF(Tantalum); footprint Capacitor_Tantalum_SMD:CP_EIA-7343-15_Kemet-W_Pad2.25x2.55mm_HandSolder -> Capacitor_SMD:C_1206_3216Metric_Pad1.42x1.75mm_HandSolder
- C9: value 680uF -> 10uF; footprint Capacitor_THT:CP_Radial_D10.0mm_P5.00mm -> Capacitor_SMD:C_1206_3216Metric_Pad1.42x1.75mm_HandSolder
- D5: value STATUS_1 -> WS2812B; footprint misc:3528_SMD_LED -> LED_SMD:LED_WS2812B_PLCC4_5.0x5.0mm_P3.2mm
- R19: footprint Resistor_THT:R_Axial_DIN0309_L9.0mm_D3.2mm_P15.24mm_Horizontal -> Resistor_THT:R_Axial_DIN0309_L9.0mm_D3.2mm_P12.70mm_Horizontal
- R20: footprint Resistor_THT:R_Axial_DIN0309_L9.0mm_D3.2mm_P15.24mm_Horizontal -> Resistor_SMD:R_1206_3216Metric_Pad1.42x1.75mm_HandSolder
- moved D6 11.9 mm to (187.2, 40.2)
Connections:
- C10 pad 2: /GND -> Net-(C10-Pad2)
- D5 pad 1: /GND -> /5v
- D5 pad 2: Net-(D5-Pad2) -> Net-(D4-Pad4)
- D6 pad 2: Net-(D6-Pad2) -> Net-(D5-Pad4)
- R19 pad 1: Net-(D5-Pad2) -> /PUSH_SW1
- R19 pad 2: /STATUS_LED_1 -> /3.3v
- S1 pad 1: Net-(S1-Pad1) -> Net-(C9-Pad1)
- S1 pad 3: Net-(C9-Pad1) -> Net-(S1-Pad3)
- U1 pad 13: /STATUS_LED_1 -> /PUSH_SW1
Routing:
- net /STATUS_LED_0: track 81.7 -> 0.00 mm
- net Net-(BZ1-Pad1): track 69.6 -> 151.3 mm
- net Net-(S1-Pad3): track 0.00 -> 63.2 mm, vias 0 -> 1
- net Net-(C9-Pad1): track 63.2 -> 0.00 mm, vias 1 -> 0
- net Net-(D5-Pad2): track 13.6 -> 0.00 mm, vias 1 -> 0
- net /PUSH_SW1: track 0.00 -> 13.6 mm, vias 0 -> 1

Commit message: fixed drc errors on schematic
Parts:
- moved D4 11.8 mm to (131.0, 30.3)
Changed lines of the file:
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@@
   )
   (module LED_SMD:LED_WS2812B_PLCC4_5.0x5.0mm_P3.2mm (layer F.Cu)
-    (at 119.352999 32.245799 180)
+    (at 130.9624 30.2514 180)
     (descr https://cdn-shop.adafruit.com/datasheets/WS2812B.pdf)
     (tags "LED RGB NeoPixel")
