File: pcb_files/mouse/mouse_v2.kicad_pcb (KiCad board)
At the start: 2 copper layers, 94.7 x 94.9 mm, 53 parts, among them M1 Motor_DC, M2 Motor_DC, M3 CASTER_BALL, Q0 Q_Photo_NPN, Q1 Q_Photo_NPN, Q2 Q_Photo_NPN, Q3 Q_Photo_NPN, SW1 SW_Push, T0 Q_NMOS_DGS, T1 Q_NMOS_DGS, T2 Q_NMOS_DGS, T3 Q_NMOS_DGS, U1 Teensy3.2, U2 SN754410NE, U3 LM1084-5.0, U4 Encoder_3081, U5 Encoder_3081

Commit message: started new design
Parts:
- removed BT, GND, MH_SCL1, MH_SDA1: MountingHole_Pad, Connector_PinHeader_2.54mm:PinHeader_1x01_P2.54mm_Vertical
- removed G***: LOGO, pika:pika3
- added J2: BT_Conn, Connector_PinSocket_2.54mm:PinSocket_1x02_P2.54mm_Vertical, F.Cu at (158.0, 100.0)
- added J4: I2C_Conn, Connector_PinSocket_2.54mm:PinSocket_1x02_P2.54mm_Vertical, F.Cu at (134.3, 96.1)
- added S1: EG1218, misc:Switch_amazon, F.Cu at (134.2, 88.2)
- CP1: footprint Capacitor_SMD:C_1206_3216Metric_Pad1.42x1.75mm_HandSolder -> Capacitor_SMD:C_0603_1608Metric_Pad1.05x0.95mm_HandSolder
- moved BT1 12.1 mm to (137.8, 98.6), turned to 180 degrees
Connections:
- U3 pad 3: /vBatt -> Net-(S1-Pad3)
Routing:
- net Net-(S1-Pad3): track 0.00 -> 63.2 mm, vias 0 -> 1
- net /vBatt: track 69.4 -> 17.7 mm, vias 1 -> 0
- net /i2c_SDA: track 5.05 -> 6.14 mm
- net /i2c_SCL: track 5.04 -> 6.10 mm

Commit message: modified battery layout
Parts:
- moved J2 6.89 mm to (159.8, 106.7)
- moved U1 4.92 mm to (159.7, 91.3)
Routing:
- net Net-(U1-Pad49): track 0.00 -> 6.14 mm
- net /i2c_SDA: track 6.14 -> 0.00 mm
- net Net-(U1-Pad50): track 0.00 -> 6.10 mm
- net /i2c_SCL: track 6.10 -> 0.00 mm
Changed lines of the file:
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@@
   (general
     (thickness 1.6)
-    (drawings 39)
+    (drawings 41)
     (tracks 456)
     (zones 0)
@@
   )
   (module teensy:Teensy30_31_32_LC (layer F.Cu)
-    (at 159.258 86.36 180)
+    (at 159.7152 91.2622 180)
     (fp_text reference U1 (at 0 -10.16 180) (layer F.SilkS)
       (effects (font (size 1 1) (thickness 0.15)))
@@
   )
   (module Connector_PinSocket_2.54mm:PinSocket_1x02_P2.54mm_Vertical (layer F.Cu)
-    (at 158.0388 100.0252 270)
+    (at 159.8422 106.68 270)
     (descr "Through hole straight socket strip, 1x02, 2.54mm pitch, single row (from Kicad 4.0.7), script generated")
     (tags "Through hole socket strip THT 1x02 2.54mm single row")
@@
     )
   )
+  (dimension 26.823855 (width 0.3) (layer F.SilkS)
+    (gr_text "26.824 mm" (at 126.782163 118.257865 359.4031905) (layer F.SilkS)
+      (effects (font (size 1.5 1.5) (thickness 0.3)))
+    )
+    (feature1 (pts (xy 140.5382 85.2932) (xy 140.209128 116.884068)))
+    (feature2 (pts (xy 113.7158 85.0138) (xy 113.386728 116.604668)))
+    (crossbar (pts (xy 113.392837 116.018279) (xy 140.215237 116.297679)))
+    (arrow1a (pts (xy 140.215237 116.297679) (xy 139.082686 116.872334)))
+    (arrow1b (pts (xy 140.215237 116.297679) (xy 139.094903 115.699556)))
+    (arrow2a (pts (xy 113.392837 116.018279) (xy 114.513171 116.616402)))
+    (arrow2b (pts (xy 113.392837 116.018279) (xy 114.525388 115.443624)))
+  )
+  (dimension 27.864089 (width 0.3) (layer F.SilkS)
+    (gr_text "27.864 mm" (at 93.892098 98.880225 89.73885423) (layer F.SilkS)
+      (effects (font (size 1.5 1.5) (thickness 0.3)))
+    )
+    (feature1 (pts (xy 113.7666 112.903) (xy 95.342162 112.819024)))
+    (feature2 (pts (xy 113.8936 85.0392) (xy 95.469162 84.955224)))
+    (crossbar (pts (xy 96.055576 84.957896) (xy 95.928576 112.821696)))
+    (arrow1a (pts (xy 95.928576 112.821696) (xy 95.347296 111.692531)))
+    (arrow1b (pts (xy 95.928576 112.821696) (xy 96.520125 111.697877)))
+    (arrow2a (pts (xy 96.055576 84.957896) (xy 95.464027 86.081715)))
+    (arrow2b (pts (xy 96.055576 84.957896) (xy 96.636856 86.087061)))
+  )
   (gr_text v2.0 (at 180.721 56.1086 180) (layer B.SilkS)
     (effects (font (size 1.5 1.5) (thickness 0.3)) (justify mirror))
@@
   (segment (start 134.3914 98.6282) (end 134.3406 98.679) (width 0.75) (layer B.Cu) (net 1))
   (segment (start 137.8458 98.6282) (end 134.3914 98.6282) (width 0.75) (layer B.Cu) (net 1))
-  (segment (start 155.956 57.725919) (end 153.856081 55.626) (width 0.75) (layer F.Cu) (net 73))
-  (segment (start 155.956 58.928) (end 155.956 57.725919) (width 0.75) (layer F.Cu) (net 73))
-  (segment (start 153.856081 55.626) (end 128.778 55.626) (width 0.75) (layer F.Cu) (net 73))
-  (segment (start 127.508 56.896) (end 128.778 55.626) (width 0.75) (layer F.Cu) (net 73))
-  (via (at 127.508 78.232) (size 1.6) (drill 0.8) (layers F.Cu B.Cu) (net 73))
-  (segment (start 127.508 78.232) (end 127.508 56.896) (width 0.75) (layer F.Cu) (net 73))
   (via (at 112.5728 102.616) (size 0.8) (drill 0.4) (layers F.Cu B.Cu) (net 2))
   (via (at 191.7954 93.3704) (size 0.8) (drill 0.4) (layers F.Cu B.Cu) (net 2))
@@
   (segment (start 114.765 105.6972) (end 114.765 102.743) (width 0.25) (layer F.Cu) (net 53))
   (segment (start 115.4557 106.3879) (end 114.765 105.6972) (width 0.25) (layer F.Cu) (net 53))
-  (segment (start 158.0134 94.0054) (end 157.988 93.98) (width 0.25) (layer F.Cu) (net 54))
-  (segment (start 158.0388 94.0308) (end 157.988 93.98) (width 0.25) (layer F.Cu) (net 54))
-  (segment (start 158.0388 100.0252) (end 158.0388 94.0308) (width 0.25) (layer F.Cu) (net 54))
-  (segment (start 155.4988 94.0308) (end 155.448 93.98) (width 0.25) (layer F.Cu) (net 55))
-  (segment (start 155.448 99.9744) (end 155.4988 100.0252) (width 0.25) (layer F.Cu) (net 55))
-  (segment (start 155.448 93.98) (end 155.448 99.9744) (width 0.25) (layer F.Cu) (net 55))
+  (segment (start 158.0134 94.0054) (end 157.988 93.98) (width 0.25) (layer F.Cu) (net 36))
+  (segment (start 158.0388 94.0308) (end 157.988 93.98) (width 0.25) (layer F.Cu) (net 36))
+  (segment (start 158.0388 100.0252) (end 158.0388 94.0308) (width 0.25) (layer F.Cu) (net 36))
+  (segment (start 155.4988 94.0308) (end 155.448 93.98) (width 0.25) (layer F.Cu) (net 35))
+  (segment (start 155.448 99.9744) (end 155.4988 100.0252) (width 0.25) (layer F.Cu) (net 35))
+  (segment (start 155.448 93.98) (end 155.448 99.9744) (width 0.25) (layer F.Cu) (net 35))
   (segment (start 179.2351 108.9406) (end 176.8094 106.5149) (width 0.25) (layer F.Cu) (net 56))
   (segment (start 189.4078 107.823) (end 188.2902 108.9406) (width 0.25) (layer F.Cu) (net 56))
@@
   (segment (start 154.8384 113.69147) (end 154.8384 112.5601) (width 0.25) (layer F.Cu) (net 71))
   (segment (start 147.3835 121.5263) (end 148.51487 121.5263) (width 0.25) (layer F.Cu) (net 71))
+  (segment (start 155.956 57.725919) (end 153.856081 55.626) (width 0.75) (layer F.Cu) (net 73))
+  (segment (start 155.956 58.928) (end 155.956 57.725919) (width 0.75) (layer F.Cu) (net 73))
+  (segment (start 153.856081 55.626) (end 128.778 55.626) (width 0.75) (layer F.Cu) (net 73))
+  (segment (start 127.508 56.896) (end 128.778 55.626) (width 0.75) (layer F.Cu) (net 73))
+  (via (at 127.508 78.232) (size 1.6) (drill 0.8) (layers F.Cu B.Cu) (net 73))
+  (segment (start 127.508 78.232) (end 127.508 56.896) (width 0.75) (layer F.Cu) (net 73))
   (segment (start 127.508 86.2586) (end 129.4636 88.2142) (width 0.75) (layer B.Cu) (net 73))
   (segment (start 127.508 78.232) (end 127.508 86.2586) (width 0.75) (layer B.Cu) (net 73))

Commit message: added rgb led to schematic
Parts:
- moved U1 6.11 mm to (158.9, 97.3)
- moved R8 5.94 mm to (151.1, 131.6)
- moved R14 5.94 mm to (166.0, 131.7)
- moved R6 5.94 mm to (162.3, 133.8)
- moved T3 5.94 mm to (153.3, 112.6)
- moved J2 5.94 mm to (159.8, 112.6)
- moved R10 5.94 mm to (169.7, 127.5)
- moved R12 5.94 mm to (147.4, 127.5)
- moved R16 5.94 mm to (154.8, 133.7)
- moved R2 5.94 mm to (173.5, 125.4)
- moved R4 5.94 mm to (143.7, 125.4)
- moved T1 5.94 mm to (166.4, 112.7)
Routing:
- net /Emitter_0: track 48.8 -> 0.00 mm
- net /Reciever_0: track 55.5 -> 14.5 mm
- net /Buzzer: track 38.4 -> 0.00 mm
- net /Reciever_2: track 45.5 -> 12.4 mm
- net /Reciever_1: track 53.1 -> 32.5 mm
- net Net-(R12-Pad1): track 19.2 -> 0.00 mm
- net /Emitter_2: track 31.0 -> 12.3 mm
- net /Emitter_1: track 18.1 -> 0.00 mm
- net /Emitter_3: track 15.1 -> 0.00 mm
- net /Reciever_3: track 58.3 -> 44.3 mm
- net Net-(U1-Pad50): track 6.10 -> 0.00 mm
- net Net-(U1-Pad49): track 6.14 -> 0.07 mm

Commit message: updates
Parts:
- removed CP1: 10uF (Tantalum), Capacitor_SMD:C_0603_1608Metric_Pad1.05x0.95mm_HandSolder
- removed U3: LM1084-5.0, Connector_PinHeader_2.54mm:PinHeader_1x03_P2.54mm_Vertical
- added D10: WS2812B, LED_SMD:LED_WS2812B_PLCC4_5.0x5.0mm_P3.2mm, F.Cu at (197.5, 51.2)
- added D11: WS2812B, LED_SMD:LED_WS2812B_PLCC4_5.0x5.0mm_P3.2mm, F.Cu at (219.5, 56.3)
- added D6: WS2812B, LED_SMD:LED_WS2812B_PLCC4_5.0x5.0mm_P3.2mm, F.Cu at (182.7, 51.2)
- added D7: WS2812B, LED_SMD:LED_WS2812B_PLCC4_5.0x5.0mm_P3.2mm, F.Cu at (199.3, 39.9)
- added D8: WS2812B, LED_SMD:LED_WS2812B_PLCC4_5.0x5.0mm_P3.2mm, F.Cu at (190.1, 51.2)
- added D9: WS2812B, LED_SMD:LED_WS2812B_PLCC4_5.0x5.0mm_P3.2mm, F.Cu at (199.3, 45.5)
- added U6: LM2596S-5, Package_TO_SOT_SMD:TO-263-5_TabPin3, F.Cu at (158.4, 64.2)
- U4, U5: footprint Connector_PinSocket_2.54mm:PinSocket_1x06_P2.54mm_Vertical -> Connector_PinSocket_2.00mm:PinSocket_1x06_P2.00mm_Vertical
Routing:
- net /OUT1: track 82.7 -> 98.4 mm
- net /5v: track 266.0 -> 250.3 mm

Commit message: finished schematic
Parts:
- removed U6: LM2596S-5, Package_TO_SOT_SMD:TO-263-5_TabPin3
- added C1: 0.1uF, Capacitor_SMD:C_1206_3216Metric_Pad1.42x1.75mm_HandSolder, F.Cu at (243.9, 112.0)
- added C10: 10uF(Tantalum), Capacitor_SMD:C_1206_3216Metric_Pad1.42x1.75mm_HandSolder, F.Cu at (236.9, 113.2)
- added C11: 0.1uF, Capacitor_SMD:C_1206_3216Metric_Pad1.42x1.75mm_HandSolder, F.Cu at (113.2, 30.1)
- added C12: 0.1uF, Capacitor_SMD:C_1206_3216Metric_Pad1.42x1.75mm_HandSolder, F.Cu at (113.2, 33.9)
- added C4: 0.1uF, Capacitor_SMD:C_1206_3216Metric_Pad1.42x1.75mm_HandSolder, F.Cu at (259.1, 119.1)
- added C5: 0.1uF, Capacitor_SMD:C_1206_3216Metric_Pad1.42x1.75mm_HandSolder, F.Cu at (248.9, 112.0)
- added C6: 0.1uF, Capacitor_SMD:C_1206_3216Metric_Pad1.42x1.75mm_HandSolder, F.Cu at (243.9, 114.2)
- added C7: 0.1uF, Capacitor_SMD:C_1206_3216Metric_Pad1.42x1.75mm_HandSolder, F.Cu at (248.9, 114.2)
- added C8: 0.1uF, Capacitor_SMD:C_1206_3216Metric_Pad1.42x1.75mm_HandSolder, F.Cu at (253.8, 112.0)
- added C9: 10uF, Capacitor_SMD:C_1206_3216Metric_Pad1.42x1.75mm_HandSolder, F.Cu at (165.4, 42.4)
- added MH1: M4, MountingHole:MountingHole_4.3mm_M4, F.Cu at (278.4, 91.2)
- added MH2: M4, MountingHole:MountingHole_4.3mm_M4, F.Cu at (261.9, 107.5)
- added MH3: M4, MountingHole:MountingHole_4.3mm_M4, F.Cu at (272.8, 100.4)
- added MH4: M4, MountingHole:MountingHole_4.3mm_M4, F.Cu at (271.1, 109.5)
- added R21: 4.7k, Resistor_SMD:R_1206_3216Metric_Pad1.42x1.75mm_HandSolder, F.Cu at (253.8, 114.2)
- added SW2: SW_Push, keyswitches:MX, F.Cu at (98.8, 38.8)
- added U3: LM1084-5.0, Package_TO_SOT_SMD:TO-263-3_TabPin2, F.Cu at (158.3, 60.7)
- C2, C3: footprint Capacitor_SMD:C_0603_1608Metric_Pad1.05x0.95mm_HandSolder -> Capacitor_SMD:C_1206_3216Metric_Pad1.42x1.75mm_HandSolder
- D4: value STATUS_0 -> WS2812B; footprint misc:3528_SMD_LED -> LED_SMD:LED_WS2812B_PLCC4_5.0x5.0mm_P3.2mm
- D5: value STATUS_1 -> WS2812B; footprint misc:3528_SMD_LED -> LED_SMD:LED_WS2812B_PLCC4_5.0x5.0mm_P3.2mm
- R1, R10, R11, R12, R13, R14, R15, R16, R17, R19, R2, R3, R4, R5, R6, R7, R8, R9: footprint Resistor_THT:R_Axial_DIN0309_L9.0mm_D3.2mm_P15.24mm_Horizontal -> Resistor_THT:R_Axial_DIN0309_L9.0mm_D3.2mm_P12.70mm_Horizontal
- R18: value R -> 4.7k; footprint Resistor_THT:R_Axial_DIN0309_L9.0mm_D3.2mm_P15.24mm_Horizontal -> Resistor_SMD:R_1206_3216Metric_Pad1.42x1.75mm_HandSolder
- R20: footprint Resistor_THT:R_Axial_DIN0309_L9.0mm_D3.2mm_P15.24mm_Horizontal -> Resistor_SMD:R_1206_3216Metric_Pad1.42x1.75mm_HandSolder
- moved D4 109.7 mm to (119.4, 32.2), turned to 180 degrees
- moved D6 11.9 mm to (187.2, 40.2)
Connections:
- D4 pad 1: /GND -> /5v
- D5 pad 1: /GND -> /5v
- D5 pad 2: Net-(D5-Pad2) -> Net-(D4-Pad4)
- D6 pad 2: Net-(D6-Pad2) -> Net-(D5-Pad4)
- R18 pad 1: Net-(D4-Pad2) -> Net-(R18-Pad1)
- R18 pad 2: /STATUS_LED_0 -> /i2c_SDA
- R19 pad 1: Net-(D5-Pad2) -> /PUSH_SW1
- R19 pad 2: /STATUS_LED_1 -> /3.3v
- U1 pad 12: /STATUS_LED_0 -> /RGB_DATA
- U1 pad 13: /STATUS_LED_1 -> /PUSH_SW1
Routing:
- net /STATUS_LED_0: track 81.7 -> 0.00 mm
- net Net-(BZ1-Pad1): track 69.6 -> 151.3 mm
- net Net-(R18-Pad1): track 0.00 -> 14.9 mm
- net Net-(D4-Pad2): track 14.9 -> 0.00 mm
- net Net-(D5-Pad2): track 13.6 -> 0.00 mm, vias 1 -> 0
- net /PUSH_SW1: track 0.00 -> 13.6 mm, vias 0 -> 1

Commit message: reworked mouse shape
Parts:
- MH1, MH2, MH3, MH4: value M4 -> M3; footprint MountingHole:MountingHole_4.3mm_M4 -> MountingHole:MountingHole_3.2mm_M3
- R1, R10, R11, R12, R13, R14, R15, R16, R2, R3, R4, R5, R6, R7, R8, R9: footprint Resistor_THT:R_Axial_DIN0309_L9.0mm_D3.2mm_P12.70mm_Horizontal -> Resistor_SMD:R_1206_3216Metric_Pad1.42x1.75mm_HandSolder
- R17, R19: value R -> R_PULL_UP; footprint Resistor_THT:R_Axial_DIN0309_L9.0mm_D3.2mm_P12.70mm_Horizontal -> Resistor_SMD:R_1206_3216Metric_Pad1.42x1.75mm_HandSolder
- R20: value R -> R_BZ
- SW1, SW2: value SW_Push -> TL3315NF160Q; footprint keyswitches:MX -> misc:KSC_SW
- moved BZ1 42.7 mm to (201.0, 64.2), turned to 270 degrees
- moved SW2 41.0 mm to (129.9, 65.5), turned to 270 degrees
- moved C3 37.7 mm to (177.6, 126.0)
- moved BT1 28.8 mm to (141.7, 70.1)
- moved J4 28.8 mm to (138.2, 67.6)
- moved U2 28.4 mm to (182.1, 66.8), turned to 90 degrees
- moved SW1 27.8 mm to (120.7, 65.6), turned to 270 degrees
- moved S1 27.5 mm to (140.5, 61.4)
- moved MH2 20.6 mm to (242.9, 99.7)
- moved U5 19.9 mm to (142.6, 77.9)
- moved U4 19.2 mm to (166.7, 78.1)
- moved M1 18.6 mm to (158.6, 87.3)
- moved M2 18.6 mm to (161.5, 87.3)
- moved U1 17.6 mm to (160.3, 114.9)
- moved T1 16.6 mm to (168.1, 129.2)
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Connections:
- C1 pad 1: /5v -> /3.3v
- C10 pad 1: /5v -> /3.3v
- C10 pad 2: Net-(C10-Pad2) -> /GND
- C11 pad 1: /5v -> /3.3v
- C12 pad 1: /5v -> /3.3v
- C2 pad 1: /5v -> /3.3v
- C3 pad 1: /5v -> /3.3v
- C4 pad 1: /5v -> /3.3v
- C5 pad 1: /5v -> /3.3v
- C6 pad 1: /5v -> /3.3v
- C7 pad 1: /5v -> /3.3v
- C8 pad 1: /5v -> /3.3v
- D0 pad 2: /5v -> /3.3v
- D1 pad 2: /5v -> /3.3v
- D10 pad 1: /5v -> /3.3v
- D11 pad 1: /5v -> /3.3v
- D2 pad 2: /5v -> /3.3v
- D3 pad 2: /5v -> /3.3v
- D4 pad 1: /5v -> /3.3v
- D5 pad 1: /5v -> /3.3v
- D6 pad 1: /5v -> /3.3v
- D7 pad 1: /5v -> /3.3v
- D8 pad 1: /5v -> /3.3v
- D9 pad 1: /5v -> /3.3v
- R18 pad 1: Net-(R18-Pad1) -> /3.3v
- R21 pad 1: Net-(R21-Pad1) -> /3.3v
- SW1 pad 1: /GND -> Net-(SW1-Pad1)
- SW1 pad 2: /PUSH_SW -> /GND
- SW2 pad 1: /GND -> Net-(SW2-Pad1)
- SW2 pad 2: /PUSH_SW1 -> /GND
- U1 pad 33: /5v -> /3.3v
- U2 pad 16: /5v -> /3.3v
- U2 pad 8: /5v -> /3.3v
- U3 pad 2: /5v -> /3.3v
- U4 pad 4: /5v -> /3.3v
- U5 pad 4: /5v -> /3.3v
Routing:
- net /5v: track 250.3 -> 0.00 mm, vias 1 -> 0
- net /3.3v: track 188.0 -> 0.00 mm, vias 1 -> 0
- net Net-(BZ1-Pad1): track 151.3 -> 0.00 mm, vias 2 -> 0
- net /OUT1: track 98.4 -> 0.00 mm
- net /STATUS_LED_1: track 88.2 -> 0.00 mm
- net /OUT2: track 70.8 -> 0.00 mm
- net /PUSH_SW: track 65.1 -> 0.00 mm
- net Net-(S1-Pad3): track 63.2 -> 0.00 mm, vias 1 -> 0
- net /OUT4: track 51.4 -> 0.00 mm, vias 1 -> 0
- net /M1_speed: track 46.5 -> 0.00 mm
- net /OUT3: track 45.0 -> 0.00 mm
- net /M2_backward: track 44.5 -> 0.00 mm
- net /Reciever_3: track 44.3 -> 0.00 mm
- net /M1_forward: track 35.2 -> 0.00 mm
- net /M2_speed: track 35.0 -> 0.00 mm
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Other:
- outline, holes or cut-outs redrawn

Commit message: Start of v3.0
Parts:
- BZ1: moved to F.Cu
- turned BZ1 to 90 degrees
Changed lines of the file:
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@@
   (general
     (thickness 1.6)
-    (drawings 43)
+    (drawings 41)
     (tracks 0)
     (zones 0)
@@
     (pad "" np_thru_hole circle (at -26.75 -9 180) (size 2.1844 2.1844) (drill 2.1844) (layers *.Cu *.Mask))
   )
-  (module "misc:9x5.5mm Buzzer" (layer B.Cu)
-    (at 200.9648 64.1858 270)
-    (fp_text reference BZ1 (at 0.381 5.6896 270) (layer B.SilkS)
-      (effects (font (size 1 1) (thickness 0.15)) (justify mirror))
+  (module "misc:9x5.5mm Buzzer" (layer F.Cu)
+    (at 200.9648 64.1858 90)
+    (fp_text reference BZ1 (at 0.381 -5.6896 90) (layer F.SilkS)
+      (effects (font (size 1 1) (thickness 0.15)))
     )
-    (fp_text value Buzzer (at -0.05 -6.8 270) (layer B.Fab)
-      (effects (font (size 1 1) (thickness 0.15)) (justify mirror))
+    (fp_text value Buzzer (at -0.05 6.8 90) (layer F.Fab)
+      (effects (font (size 1 1) (thickness 0.15)))
     )
-    (fp_circle (center 0 0) (end 4.4 1.1) (layer B.SilkS) (width 0.15))
-    (fp_text user - (at -2.55 -1.35 270) (layer B.SilkS)
-      (effects (font (size 1 1) (thickness 0.15)) (justify mirror))
+    (fp_circle (center 0 0) (end 4.4 -1.1) (layer F.SilkS) (width 0.15))
+    (fp_text user - (at -2.55 1.35 90) (layer F.SilkS)
+      (effects (font (size 1 1) (thickness 0.15)))
     )
-    (fp_text user + (at 2.5 -1.3 270) (layer B.SilkS)
-      (effects (font (size 1 1) (thickness 0.15)) (justify mirror))
+    (fp_text user + (at 2.5 1.3 90) (layer F.SilkS)
+      (effects (font (size 1 1) (thickness 0.15)))
     )
-    (pad 2 thru_hole circle (at -2.5 0 270) (size 1.524 1.524) (drill 0.762) (layers *.Cu *.Mask)
+    (pad 2 thru_hole circle (at -2.5 0 90) (size 1.524 1.524) (drill 0.762) (layers *.Cu *.Mask)
       (net 2 /GND))
-    (pad 1 thru_hole circle (at 2.5 -0.05 270) (size 1.524 1.524) (drill 0.762) (layers *.Cu *.Mask)
+    (pad 1 thru_hole circle (at 2.5 0.05 90) (size 1.524 1.524) (drill 0.762) (layers *.Cu *.Mask)
       (net 50 "Net-(BZ1-Pad1)"))
   )
@@
   (gr_line (start 207.3402 102.4128) (end 192.2272 102.4128) (layer Edge.Cuts) (width 0.15))
   (gr_line (start 112.5982 102.1588) (end 127.7112 102.1588) (layer Edge.Cuts) (width 0.15))
-  (dimension 10.9982 (width 0.3) (layer F.SilkS)
-    (gr_text "10.998 mm" (at 218.508 100.4951 90) (layer F.SilkS)
-      (effects (font (size 1.5 1.5) (thickness 0.3)))
-    )
-    (feature1 (pts (xy 144.9832 94.996) (xy 216.994421 94.996)))
-    (feature2 (pts (xy 144.9832 105.9942) (xy 216.994421 105.9942)))
-    (crossbar (pts (xy 216.408 105.9942) (xy 216.408 94.996)))
-    (arrow1a (pts (xy 216.408 94.996) (xy 216.994421 96.122504)))
-    (arrow1b (pts (xy 216.408 94.996) (xy 215.821579 96.122504)))
-    (arrow2a (pts (xy 216.408 105.9942) (xy 216.994421 104.867696)))
-    (arrow2b (pts (xy 216.408 105.9942) (xy 215.821579 104.867696)))
-  )
-  (dimension 26.823855 (width 0.3) (layer F.SilkS)
-    (gr_text "26.824 mm" (at 128.255363 118.054665 359.4031905) (layer F.SilkS)
-      (effects (font (size 1.5 1.5) (thickness 0.3)))
-    )
-    (feature1 (pts (xy 142.0114 85.09) (xy 141.682328 116.680868)))
-    (feature2 (pts (xy 115.189 84.8106) (xy 114.859928 116.401468)))
-    (crossbar (pts (xy 114.866037 115.815079) (xy 141.688437 116.094479)))
-    (arrow1a (pts (xy 141.688437 116.094479) (xy 140.555886 116.669134)))
-    (arrow1b (pts (xy 141.688437 116.094479) (xy 140.568103 115.496356)))
-    (arrow2a (pts (xy 114.866037 115.815079) (xy 115.986371 116.413202)))
-    (arrow2b (pts (xy 114.866037 115.815079) (xy 115.998588 115.240424)))
-  )
   (gr_text v2.0 (at 182.1942 55.9054 180) (layer B.SilkS)
     (effects (font (size 1.5 1.5) (thickness 0.3)) (justify mirror))

Commit message: working on layout
Parts:
- C1, C11, C12, C3, C5, C8, D10, D11, D4, D5, D6, D8, R20: moved to B.Cu
- moved C7 146.4 mm to (115.3, 57.5)
- moved MH4 145.6 mm to (128.9, 132.8)
- moved C4 123.2 mm to (154.6, 56.0), turned to 180 degrees
- moved C11 116.3 mm to (194.9, 114.0), turned to 90 degrees
- moved C6 113.9 mm to (147.5, 55.8), turned to 180 degrees
- moved D6 111.6 mm to (141.2, 141.0)
- moved MH2 110.9 mm to (132.5, 109.1)
- moved D4 108.4 mm to (201.3, 113.7)
- moved C1 103.9 mm to (147.2, 145.7)
- moved R21 96.4 mm to (160.7, 132.6), turned to 270 degrees
- moved D11 94.7 mm to (178.8, 141.0)
- moved MH1 92.7 mm to (187.4, 108.9)
- moved MH3 90.2 mm to (190.3, 133.4)
- moved C8 89.1 mm to (172.7, 145.1), turned to 180 degrees
- moved D10 84.6 mm to (115.3, 63.3), turned to 90 degrees
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Connections:
- C1 pad 1: /3.3v -> /5v
- C10 pad 1: /3.3v -> /5v
- C11 pad 1: /3.3v -> /5v
- C12 pad 1: /3.3v -> /5v
- C2 pad 1: /3.3v -> /5v
- C3 pad 1: /3.3v -> /5v
- C4 pad 1: /3.3v -> /5v
- C5 pad 1: /3.3v -> /5v
- C6 pad 1: /3.3v -> /5v
- C7 pad 1: /3.3v -> /5v
- C8 pad 1: /3.3v -> /5v
- D0 pad 2: /3.3v -> /5v
- D1 pad 2: /3.3v -> /5v
- D10 pad 1: /3.3v -> /5v
- D11 pad 1: /3.3v -> /5v
- D2 pad 2: /3.3v -> /5v
- D3 pad 2: /3.3v -> /5v
- D4 pad 1: /3.3v -> /5v
- D5 pad 1: /3.3v -> /5v
- D6 pad 1: /3.3v -> /5v
- D7 pad 1: /3.3v -> /5v
- D8 pad 1: /3.3v -> /5v
- D9 pad 1: /3.3v -> /5v
- U1 pad 33: /3.3v -> /5v
- U2 pad 16: /3.3v -> /5v
- U2 pad 8: /3.3v -> /5v
- U3 pad 2: /3.3v -> /5v
- U4 pad 4: /3.3v -> /5v
- U5 pad 4: /3.3v -> /5v
Other:
- board text added: "v3.0"
- board text removed: "IN"
- board text removed: "OUT"
- board text removed: "v2.0"
