File: pcb_files/mouse/mouse_v2.kicad_pcb (KiCad board)
At the start: 2 copper layers, 94.7 x 94.9 mm, 72 parts, among them J2 BT_Conn, J4 I2C_Conn, M1 Motor_DC, M2 Motor_DC, M3 CASTER_BALL, Q0 Q_Photo_NPN, Q1 Q_Photo_NPN, Q2 Q_Photo_NPN, Q3 Q_Photo_NPN, SW1 TL3315NF160Q, SW2 TL3315NF160Q, T0 Q_NMOS_DGS, T1 Q_NMOS_DGS, T2 Q_NMOS_DGS, T3 Q_NMOS_DGS, U1 Teensy3.2, U2 SN754410NE, U3 LM1084-5.0, U4 Encoder_3081, U5 Encoder_3081

Commit message: added usb c, rounded edges
Parts:
- added J1: USB_C_Receptacle, misc:USB_C_REDUCED_PINS, F.Cu at (198.8, 59.7)
- C7: moved to B.Cu
- moved C9 19.9 mm to (163.6, 72.3), turned to 90 degrees
- moved S1 14.8 mm to (184.4, 58.8)
- moved C5 6.61 mm to (197.8, 69.2), turned to 90 degrees
- moved D10 6.20 mm to (116.3, 69.4), turned to 180 degrees
- moved D8 6.10 mm to (203.7, 69.3), turned to 180 degrees
- moved C7 6.00 mm to (115.2, 63.5), turned to 180 degrees
Connections:
- C10 pad 1: /5v -> Net-(C10-Pad1)
- C9 pad 1: Net-(C9-Pad1) -> /vBatt
- S1 pad 1: Net-(C9-Pad1) -> Net-(C10-Pad1)
- S1 pad 2: /vBatt -> /5v
- S1 pad 3: Net-(S1-Pad3) -> /USB_VBUS
- U3 pad 2: /5v -> Net-(C10-Pad1)
- U3 pad 3: Net-(C9-Pad1) -> /vBatt
Other:
- board size 94.7 x 94.9 mm -> 94.8 x 94.9 mm

Commit message: started tracing
Parts:
- C4, D7: moved to B.Cu
- C5, D8: moved to F.Cu
- moved D5 66.4 mm to (179.8, 139.4), turned to 90 degrees
- moved C1 65.7 mm to (203.4, 111.7), turned to 180 degrees
- moved C12 65.2 mm to (184.7, 139.7), turned to 0 degrees
- moved D4 65.1 mm to (141.6, 139.7), turned to 90 degrees
- moved D6 64.9 mm to (200.9, 115.5), turned to 180 degrees
- moved D11 64.2 mm to (119.5, 116.5)
- moved C8 58.5 mm to (119.7, 120.2), turned to 0 degrees
- moved C11 57.3 mm to (146.0, 143.8), turned to 270 degrees
- moved C4 51.9 mm to (206.1, 63.3), turned to 90 degrees
- moved D8 50.7 mm to (154.2, 58.4), turned to 90 degrees
- moved D7 49.7 mm to (203.6, 68.9), turned to 180 degrees
- moved C5 44.1 mm to (154.1, 63.1), turned to 0 degrees
- moved R18 37.3 mm to (155.8, 131.4), turned to 90 degrees
- moved R1 22.9 mm to (205.2, 105.3), turned to 270 degrees
- moved R5 17.9 mm to (193.7, 109.4), turned to 180 degrees
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Routing:
- net /3.3v: track 0.00 -> 206.3 mm
- net /5v: track 0.00 -> 41.0 mm
- net /vBatt: track 0.00 -> 21.7 mm
- net /USB_VBUS: track 0.00 -> 16.7 mm
- net Net-(C10-Pad1): track 0.00 -> 15.0 mm
- net Net-(R5-Pad2): track 0.00 -> 9.59 mm
- net /USB_D-: track 0.00 -> 8.94 mm, vias 0 -> 1
- net /USB_D+: track 0.00 -> 8.77 mm
- net Net-(R13-Pad2): track 0.00 -> 4.51 mm
- net /i2c_SDA: track 0.00 -> 3.47 mm
- net /i2c_SCL: track 0.00 -> 3.43 mm
- net Net-(D0-Pad1): track 0.00 -> 2.41 mm

Commit message: wired emitters/recievers, 5v+3.3v bus on bottom
Parts:
- moved R1 21.2 mm to (186.1, 114.6), turned to 90 degrees
- moved R11 15.7 mm to (127.8, 114.6)
- moved T2 12.8 mm to (128.5, 108.2)
- moved T0 8.65 mm to (193.1, 108.7)
- moved R9 8.05 mm to (188.8, 114.6)
- moved MH1 7.19 mm to (182.0, 104.2)
- moved R13 5.39 mm to (191.7, 114.6)
- moved R5 5.31 mm to (194.7, 114.6), turned to 90 degrees
- moved MH2 4.59 mm to (137.0, 108.9)
- moved T3 4.13 mm to (154.6, 131.9)
- moved R15 3.74 mm to (133.8, 114.7)
- moved R3 3.59 mm to (130.9, 114.6), turned to 270 degrees
- moved R6 3.10 mm to (163.7, 137.3)
- moved R16 3.00 mm to (156.4, 137.3)
- moved T1 2.71 mm to (167.8, 131.9)
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Routing:
- net /5v: track 41.0 -> 151.9 mm
- net /Reciever_0: track 0.00 -> 49.4 mm
- net /Reciever_2: track 0.00 -> 40.2 mm, vias 0 -> 2
- net /Emitter_2: track 0.00 -> 26.6 mm
- net /Emitter_0: track 0.00 -> 26.5 mm
- net /Reciever_1: track 0.00 -> 21.5 mm
- net /Reciever_3: track 0.00 -> 19.4 mm
- net /Emitter_1: track 0.00 -> 15.3 mm
- net /Emitter_3: track 0.00 -> 12.9 mm
- net Net-(R12-Pad1): track 0.00 -> 12.4 mm
- net Net-(R11-Pad1): track 0.00 -> 11.2 mm
- net Net-(R10-Pad1): track 0.00 -> 9.74 mm
- net Net-(D2-Pad1): track 0.00 -> 8.91 mm
- net Net-(D1-Pad1): track 0.00 -> 8.47 mm
- net Net-(R6-Pad2): track 0.00 -> 7.59 mm
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Other:
- net class Default: clearance 0.2 -> 0.13; trace_width 0.25 -> 0.13
- rule trace_clearance: 0.2 -> 0.13
- rule trace_min: 0.2 -> 0.13

Commit message: teensy header for microusb breakout smd pads
Parts:
- added J3: Conn_01x04_Female, Connector_PinHeader_2.54mm:PinHeader_1x04_P2.54mm_Vertical, F.Cu at (175.5, 117.4)
Changed lines of the file:
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@@
   (general
     (thickness 1.6)
-    (drawings 37)
+    (drawings 38)
     (tracks 259)
     (zones 0)
-    (modules 73)
+    (modules 74)
     (nets 86)
   )
@@
     )
   )
+  (module Connector_PinHeader_2.54mm:PinHeader_1x04_P2.54mm_Vertical (layer F.Cu)
+    (at 175.45304 117.37848 180)
+    (descr "Through hole straight pin header, 1x04, 2.54mm pitch, single row")
+    (tags "Through hole pin header THT 1x04 2.54mm single row")
+    (fp_text reference J3 (at -1.32588 -2.60604 180) (layer F.SilkS)
+      (effects (font (size 1 1) (thickness 0.15)))
+    )
+    (fp_text value Conn_01x04_Female (at 0 9.95 180) (layer F.Fab)
+      (effects (font (size 1 1) (thickness 0.15)))
+    )
+    (fp_line (start -0.635 -1.27) (end 1.27 -1.27) (layer F.Fab) (width 0.1))
+    (fp_line (start 1.27 -1.27) (end 1.27 8.89) (layer F.Fab) (width 0.1))
+    (fp_line (start 1.27 8.89) (end -1.27 8.89) (layer F.Fab) (width 0.1))
+    (fp_line (start -1.27 8.89) (end -1.27 -0.635) (layer F.Fab) (width 0.1))
+    (fp_line (start -1.27 -0.635) (end -0.635 -1.27) (layer F.Fab) (width 0.1))
+    (fp_line (start -1.33 8.95) (end 1.33 8.95) (layer F.SilkS) (width 0.12))
+    (fp_line (start -1.33 1.27) (end -1.33 8.95) (layer F.SilkS) (width 0.12))
+    (fp_line (start 1.33 1.27) (end 1.33 8.95) (layer F.SilkS) (width 0.12))
+    (fp_line (start -1.33 1.27) (end 1.33 1.27) (layer F.SilkS) (width 0.12))
+    (fp_line (start -1.33 0) (end -1.33 -1.33) (layer F.SilkS) (width 0.12))
+    (fp_line (start -1.33 -1.33) (end 0 -1.33) (layer F.SilkS) (width 0.12))
+    (fp_line (start -1.8 -1.8) (end -1.8 9.4) (layer F.CrtYd) (width 0.05))
+    (fp_line (start -1.8 9.4) (end 1.8 9.4) (layer F.CrtYd) (width 0.05))
+    (fp_line (start 1.8 9.4) (end 1.8 -1.8) (layer F.CrtYd) (width 0.05))
+    (fp_line (start 1.8 -1.8) (end -1.8 -1.8) (layer F.CrtYd) (width 0.05))
+    (fp_text user %R (at 0 3.81 270) (layer F.Fab)
+      (effects (font (size 1 1) (thickness 0.15)))
+    )
+    (pad 1 thru_hole rect (at 0 0 180) (size 1.7 1.7) (drill 1) (layers *.Cu *.Mask)
+      (net 83 /USB_VBUS))
+    (pad 2 thru_hole oval (at 0 2.54 180) (size 1.7 1.7) (drill 1) (layers *.Cu *.Mask)
+      (net 84 /USB_D-))
+    (pad 3 thru_hole oval (at 0 5.08 180) (size 1.7 1.7) (drill 1) (layers *.Cu *.Mask)
+      (net 85 /USB_D+))
+    (pad 4 thru_hole oval (at 0 7.62 180) (size 1.7 1.7) (drill 1) (layers *.Cu *.Mask)
+      (net 2 /GND))
+    (model ${KISYS3DMOD}/Connector_PinHeader_2.54mm.3dshapes/PinHeader_1x04_P2.54mm_Vertical.wrl
+      (at (xyz 0 0 0))
+      (scale (xyz 1 1 1))
+      (rotate (xyz 0 0 0))
+    )
+  )
+  (dimension 5.02412 (width 0.3) (layer B.SilkS)
+    (gr_text "5.024 mm" (at 166.48742 109.79404 270) (layer B.SilkS)
+      (effects (font (size 1.5 1.5) (thickness 0.3)))
+    )
+    (feature1 (pts (xy 176.76876 112.3061) (xy 168.000999 112.3061)))
+    (feature2 (pts (xy 176.76876 107.28198) (xy 168.000999 107.28198)))
+    (crossbar (pts (xy 168.58742 107.28198) (xy 168.58742 112.3061)))
+    (arrow1a (pts (xy 168.58742 112.3061) (xy 168.000999 111.179596)))
+    (arrow1b (pts (xy 168.58742 112.3061) (xy 169.173841 111.179596)))
+    (arrow2a (pts (xy 168.58742 107.28198) (xy 168.000999 108.408484)))
+    (arrow2b (pts (xy 168.58742 107.28198) (xy 169.173841 108.408484)))
+  )
   (gr_arc (start 115.958619 58.023759) (end 115.92052 54.65318) (angle -89.35237371) (layer Edge.Cuts) (width 0.15))

Commit message: swapping pins on teensy to make tracing easier
Parts:
- moved C2 23.4 mm to (157.8, 78.3)
- moved C3 22.8 mm to (137.3, 68.1), turned to 270 degrees
- moved U4 10.9 mm to (177.7, 78.0), turned to 270 degrees
- moved R17 2.28 mm to (123.1, 57.4), turned to 180 degrees
- moved U2 1.67 mm to (157.9, 66.6)
- turned R19 to 180 degrees
- turned SW1 to 90 degrees
- turned SW2 to 90 degrees
Routing:
- net /OUT4: track 0.00 -> 30.0 mm
- net /M1_backward: track 0.00 -> 26.5 mm
- net /M1_forward: track 0.00 -> 24.8 mm
- net /OUT3: track 0.00 -> 24.2 mm
- net /5v: track 151.9 -> 166.0 mm
- net /OUT1: track 0.00 -> 6.94 mm
- net Net-(D8-Pad4): track 0.00 -> 6.65 mm
- net /PUSH_SW1: track 0.00 -> 3.99 mm
- net /PUSH_SW: track 0.00 -> 3.82 mm
- net /OUT2: track 0.00 -> 3.77 mm

Commit message: finished traces, except gnd net
Parts:
- moved R20 0.41 mm to (136.6, 60.6), turned to 270 degrees
Connections:
- U1 pad 8: /M2_encoder_A -> /M2_encoder_B
- U1 pad 9: /M2_encoder_B -> /M2_encoder_A
Routing:
- net /5v: track 166.0 -> 433.6 mm, vias 0 -> 4
- net /3.3v: track 206.2 -> 292.4 mm
- net /Buzzer: track 0.00 -> 76.7 mm, vias 0 -> 3
- net /USB_D+: track 8.77 -> 83.0 mm, vias 0 -> 2
- net Net-(D7-Pad4): track 0.00 -> 70.9 mm, vias 0 -> 1
- net Net-(D10-Pad4): track 0.00 -> 70.8 mm
- net /USB_D-: track 8.94 -> 78.9 mm, vias 1 -> 3
- net /PUSH_SW: track 3.82 -> 73.7 mm
- net /USB_VBUS: track 16.7 -> 85.0 mm, vias 0 -> 2
- net /PUSH_SW1: track 3.99 -> 67.0 mm
- net Net-(D6-Pad4): track 0.00 -> 62.4 mm
- net /M2_backward: track 0.00 -> 60.3 mm, vias 0 -> 1
- net /M1_speed: track 0.00 -> 49.5 mm, vias 0 -> 1
- net /RGB_DATA: track 0.00 -> 49.5 mm, vias 0 -> 1
- net /M2_forward: track 0.00 -> 49.0 mm, vias 0 -> 2
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
Commit message: ground planes, via stitches
Parts:
- removed MH3, MH4: M3, MountingHole:MountingHole_3.2mm_M3
- moved MH1 22.3 mm to (185.4, 126.2)
- moved MH2 17.4 mm to (134.7, 126.1)
Routing:
- net Net-(D4-Pad4): track 0.00 -> 47.6 mm, vias 1 -> 4
- net /GND: track 0.00 -> 35.1 mm, vias 1 -> 36
- net Net-(R6-Pad2): track 7.59 -> 4.50 mm
- net Net-(R12-Pad1): track 12.4 -> 9.64 mm
- net Net-(R10-Pad1): track 9.74 -> 8.73 mm
- net /5v: track 433.6 -> 434.3 mm
- net Net-(R5-Pad2): track 10.8 -> 11.0 mm, vias 0 -> 1

Commit message: added keep out under usb c port
Routing:
- net /USB_VBUS: track 85.0 -> 90.3 mm, vias 2 -> 3
- net /USB_D-: track 78.9 -> 81.9 mm
- net /GND: vias 36 -> 52
