File: pcb_files/mouse/_saved_mouse_v2.sch (KiCad schematic (older format))
At the start: 49 parts, among them J4 I2C_Conn, M1 Motor_DC, M2 Motor_DC, M3 CASTER_BALL, Q0 Q_Photo_NPN, Q1 Q_Photo_NPN, Q2 Q_Photo_NPN, Q3 Q_Photo_NPN, T0 Q_NMOS_DGS, T1 Q_NMOS_DGS, T2 Q_NMOS_DGS, T3 Q_NMOS_DGS, U1 Teensy4.0, U2 SN754410NE, U3 LM1085-5.0, U4 Encoder_3081, U5 Encoder_3081

Commit message: SMD Caps, Space for Skates, Smaller Switch
Parts:
- C2, C9: footprint Capacitor_THT:CP_Radial_D8.0mm_P3.80mm -> Capacitor_SMD:C_1206_3216Metric_Pad1.42x1.75mm_HandSolder
- C3: footprint Capacitor_THT:CP_Radial_D8.0mm_P5.00mm -> Capacitor_SMD:C_1206_3216Metric_Pad1.42x1.75mm_HandSolder
- S1: footprint misc:PW_SLIDE_SW -> misc:SWITCH_SLIDE_500SSP1S2M2QEA
Changed lines of the file:
@@
 F 0 "C2" H 4100 8650 50  0000 R CNN
 F 1 "0.1uF" H 4109 8745 50  0000 R CNN
-F 2 "Capacitor_THT:CP_Radial_D8.0mm_P3.80mm" H 4200 8700 50  0001 C CNN
+F 2 "Capacitor_SMD:C_1206_3216Metric_Pad1.42x1.75mm_HandSolder" H 4200 8700 50  0001 C CNN
 F 3 "~" H 4200 8700 50  0001 C CNN
 	1    4200 8700
@@
 F 0 "C3" H 4000 9050 50  0000 L CNN
 F 1 "1.0uF" H 3900 8950 50  0000 L CNN
-F 2 "Capacitor_THT:CP_Radial_D8.0mm_P5.00mm" H 4200 9000 50  0001 C CNN
+F 2 "Capacitor_SMD:C_1206_3216Metric_Pad1.42x1.75mm_HandSolder" H 4200 9000 50  0001 C CNN
 F 3 "~" H 4200 9000 50  0001 C CNN
 	1    4200 9000
@@
 F 0 "S1" H 5775 6254 50  0000 C CNN
 F 1 "EG1218" H 5775 6163 50  0000 C CNN
-F 2 "misc:PW_SLIDE_SW" H 5975 6175 50  0001 L CNN
+F 2 "misc:SWITCH_SLIDE_500SSP1S2M2QEA" H 5975 6175 50  0001 L CNN
 F 3 "http://spec_sheets.e-switch.com/specs/P040040.pdf" H 5975 6275 60  0001 L CNN
 F 4 "EG1903-ND" H 5975 6375 60  0001 L CNN "Digi-Key_PN"
@@
 F 0 "C9" H 4340 5996 50  0000 L CNN
 F 1 "10uF" H 4340 5905 50  0000 L CNN
-F 2 "Capacitor_THT:CP_Radial_D8.0mm_P3.80mm" H 4225 5950 50  0001 C CNN
+F 2 "Capacitor_SMD:C_1206_3216Metric_Pad1.42x1.75mm_HandSolder" H 4225 5950 50  0001 C CNN
 F 3 "~" H 4225 5950 50  0001 C CNN
 	1    4225 5950
