File: pcb_files/mouse/mouse_v2.sch (KiCad schematic (older format))
At the start: 49 parts, among them J4 I2C_Conn, M1 Motor_DC, M2 Motor_DC, M3 CASTER_BALL, Q0 Q_Photo_NPN, Q1 Q_Photo_NPN, Q2 Q_Photo_NPN, Q3 Q_Photo_NPN, T0 Q_NMOS_DGS, T1 Q_NMOS_DGS, T2 Q_NMOS_DGS, T3 Q_NMOS_DGS, U1 Teensy4.0, U2 SN754410NE, U3 LM1085-5.0, U4 Encoder_3081, U5 Encoder_3081

Commit message: Fixed reciever/emitter pins
Connections:
- net Emitter_0: now also U1.29 (22_A8_CTX1)
- net Reciever_0: now also U1.30 (23_A9_CRX1_MCLK1)
- net Reciever_1: now also U1.28 (21_A7_RX5_BCLK1)
- no-connect marks 30 -> 32
Changed lines of the file:
@@
 Text Label 5370 3010 0    50   ~ 0
 GND
-Text Label 9800 3450 0    50   ~ 0
+Text Label 9800 3525 0    50   ~ 0
 Reciever_0
-Text Label 9800 3650 0    50   ~ 0
+Text Label 7600 3625 2    50   ~ 0
 Reciever_1
 Text Label 7600 2925 2    50   ~ 0
@@
 Text Label 7600 3125 2    50   ~ 0
 Reciever_3
-Text Label 9800 3550 0    50   ~ 0
+Text Label 9800 3625 0    50   ~ 0
 Emitter_0
 Text Label 7600 3525 2    50   ~ 0
@@
 	1    0    0    -1
 $EndComp
+NoConn ~ 9800 3325
+NoConn ~ 9800 3425
 $EndSCHEMATC

Commit message: SMD Caps, Space for Skates, Smaller Switch
Parts:
- C2, C9: footprint Capacitor_THT:CP_Radial_D8.0mm_P3.80mm -> Capacitor_SMD:C_1206_3216Metric_Pad1.42x1.75mm_HandSolder
- C3: footprint Capacitor_THT:CP_Radial_D8.0mm_P5.00mm -> Capacitor_SMD:C_1206_3216Metric_Pad1.42x1.75mm_HandSolder
Changed lines of the file:
@@
 F 0 "C2" H 4100 8650 50  0000 R CNN
 F 1 "0.1uF" H 4109 8745 50  0000 R CNN
-F 2 "Capacitor_THT:CP_Radial_D8.0mm_P3.80mm" H 4200 8700 50  0001 C CNN
+F 2 "Capacitor_SMD:C_1206_3216Metric_Pad1.42x1.75mm_HandSolder" H 4200 8700 50  0001 C CNN
 F 3 "~" H 4200 8700 50  0001 C CNN
 	1    4200 8700
@@
 F 0 "C3" H 4000 9050 50  0000 L CNN
 F 1 "1.0uF" H 3900 8950 50  0000 L CNN
-F 2 "Capacitor_THT:CP_Radial_D8.0mm_P5.00mm" H 4200 9000 50  0001 C CNN
+F 2 "Capacitor_SMD:C_1206_3216Metric_Pad1.42x1.75mm_HandSolder" H 4200 9000 50  0001 C CNN
 F 3 "~" H 4200 9000 50  0001 C CNN
 	1    4200 9000
@@
 F 0 "C9" H 4340 5996 50  0000 L CNN
 F 1 "10uF" H 4340 5905 50  0000 L CNN
-F 2 "Capacitor_THT:CP_Radial_D8.0mm_P3.80mm" H 4225 5950 50  0001 C CNN
+F 2 "Capacitor_SMD:C_1206_3216Metric_Pad1.42x1.75mm_HandSolder" H 4225 5950 50  0001 C CNN
 F 3 "~" H 4225 5950 50  0001 C CNN
 	1    4225 5950

Commit message: Update on PCB reforms
Parts:
- removed M3: CASTER_BALL, misc:Mouse_caster, symbol Motor:Motor_DC
- added BZ1: Buzzer, misc:9x5.5mm Buzzer, symbol Device:Buzzer
- added D4, D5, D6: LED, LED_THT:LED_D5.0mm, symbol Device:LED
- added R18, R19, R20, R21: R, Resistor_THT:R_Axial_DIN0207_L6.3mm_D2.5mm_P10.16mm_Horizontal, symbol Device:R
- S1: footprint misc:PW_SLIDE_SW -> misc:SWITCH_SLIDE_500SSP1S2M2QEA
- U2: value SN754410NE -> SN754410NE (Half-Bridge)
- renumbered MH4 to SK1, MH3 to SK2
Connections:
- net GND: now also BZ1.2 (+), D4.1 (K), D5.1 (K), D6.1 (K)
- net Buzzer: now reaches U1.13 (11_MOSI_CTX1)
- net Buzzer: now also R18.1
- net LED_1: now reaches U1.20 (13_SCK_CRX1_LED)
- net LED_1: now also R19.2
- net LED_2: now reaches U1.25 (18_A4_SDA0)
- net LED_2: now also R20.2
- net LED_3: now reaches U1.26 (19_A5_SCL0)
- net LED_3: now also R21.2
- new net: BZ1.1 (-), R18.2
- new net: D4.2 (A), R19.1
- new net: D5.2 (A), R20.1
- new net: D6.2 (A), R21.1
- no-connect marks 32 -> 26
Other:
- note added: "Indicators\n"
- note added: "Mount Designators\n"
- note removed: "Caster and Motors\n"
- moved on the sheet: MH1, MH2, SK1, SK2
Changed lines of the file:
@@
 Text Label 7600 3225 2    50   ~ 0
 Emitter_3
-$Comp
-L Motor:Motor_DC M3
-U 1 1 5D240B05
-P 1425 6950
-F 0 "M3" H 1583 6946 50  0000 L CNN
-F 1 "CASTER_BALL" H 1583 6855 50  0000 L CNN
-F 2 "misc:Mouse_caster" H 1425 6860 50  0001 C CNN
-F 3 "~" H 1425 6860 50  0001 C CNN
-	1    1425 6950
-	1    0    0    -1
-$EndComp
 Text Label 7600 1125 2    50   ~ 0
 M1_forward
@@
 P 5400 9400
 F 0 "U2" H 5400 10370 50  0000 C CNN
-F 1 "SN754410NE" H 5400 10279 50  0000 C CNN
+F 1 "SN754410NE (Half-Bridge)" H 5400 10279 50  0000 C CNN
 F 2 "SN754410NE.kicad_mod:DIP254P762X508-16" H 5400 9400 50  0001 L BNN
 F 3 "PDIP-16 Texas Instruments" H 5400 9400 50  0001 L BNN
@@
 F 0 "S1" H 5775 6254 50  0000 C CNN
 F 1 "EG1218" H 5775 6163 50  0000 C CNN
-F 2 "misc:PW_SLIDE_SW" H 5975 6175 50  0001 L CNN
+F 2 "misc:SWITCH_SLIDE_500SSP1S2M2QEA" H 5975 6175 50  0001 L CNN
 F 3 "http://spec_sheets.e-switch.com/specs/P040040.pdf" H 5975 6275 60  0001 L CNN
 F 4 "EG1903-ND" H 5975 6375 60  0001 L CNN "Digi-Key_PN"
@@
 Text Label 9800 3225 0    50   ~ 0
 5v
-NoConn ~ 1425 6750
-NoConn ~ 1425 7250
-$Comp
-L Mechanical:MountingHole MH4
+$Comp
+L Mechanical:MountingHole SK1
 U 1 1 5E799FC8
-P 2000 6325
-F 0 "MH4" H 2100 6371 50  0000 L CNN
-F 1 "M3" H 2100 6280 50  0000 L CNN
-F 2 "MountingHole:MountingHole_3.2mm_M3" H 2000 6325 50  0001 C CNN
-F 3 "~" H 2000 6325 50  0001 C CNN
-	1    2000 6325
+P 2000 5550
+F 0 "SK1" H 2100 5596 50  0000 L CNN
+F 1 "M3" H 2100 5505 50  0000 L CNN
+F 2 "MountingHole:MountingHole_3.2mm_M3" H 2000 5550 50  0001 C CNN
+F 3 "~" H 2000 5550 50  0001 C CNN
+	1    2000 5550
 	1    0    0    -1
 $EndComp
@@
 L Mechanical:MountingHole MH2
 U 1 1 5E79A0A3
-P 1175 6350
-F 0 "MH2" H 1275 6396 50  0000 L CNN
-F 1 "M3" H 1275 6305 50  0000 L CNN
-F 2 "MountingHole:MountingHole_3.2mm_M3" H 1175 6350 50  0001 C CNN
-F 3 "~" H 1175 6350 50  0001 C CNN
-	1    1175 6350
+P 1175 5575
+F 0 "MH2" H 1275 5621 50  0000 L CNN
+F 1 "M3" H 1275 5530 50  0000 L CNN
+F 2 "MountingHole:MountingHole_3.2mm_M3" H 1175 5575 50  0001 C CNN
+F 3 "~" H 1175 5575 50  0001 C CNN
+	1    1175 5575
 	1    0    0    -1
 $EndComp
@@
 L Mechanical:MountingHole MH1
 U 1 1 5E79A15B
-P 1175 5950
-F 0 "MH1" H 1275 5996 50  0000 L CNN
-F 1 "M3" H 1275 5905 50  0000 L CNN
-F 2 "MountingHole:MountingHole_3.2mm_M3" H 1175 5950 50  0001 C CNN
-F 3 "~" H 1175 5950 50  0001 C CNN
-	1    1175 5950
-	1    0    0    -1
-$EndComp
-$Comp
-L Mechanical:MountingHole MH3
+P 1175 5175
+F 0 "MH1" H 1275 5221 50  0000 L CNN
+F 1 "M3" H 1275 5130 50  0000 L CNN
+F 2 "MountingHole:MountingHole_3.2mm_M3" H 1175 5175 50  0001 C CNN
+F 3 "~" H 1175 5175 50  0001 C CNN
+	1    1175 5175
+	1    0    0    -1
+$EndComp
+$Comp
+L Mechanical:MountingHole SK2
 U 1 1 5E79A200
-P 2000 5950
-F 0 "MH3" H 2100 5996 50  0000 L CNN
-F 1 "M3" H 2100 5905 50  0000 L CNN
-F 2 "MountingHole:MountingHole_3.2mm_M3" H 2000 5950 50  0001 C CNN
-F 3 "~" H 2000 5950 50  0001 C CNN
-	1    2000 5950
+P 2000 5175
+F 0 "SK2" H 2100 5221 50  0000 L CNN
+F 1 "M3" H 2100 5130 50  0000 L CNN
+F 2 "MountingHole:MountingHole_3.2mm_M3" H 2000 5175 50  0001 C CNN
+F 3 "~" H 2000 5175 50  0001 C CNN
+	1    2000 5175
 	1    0    0    -1
 $EndComp
@@
 Text Notes 6700 8000 2    79   ~ 0
 Power Supply
-Text Notes 2800 8000 2    79   ~ 0
-Caster and Motors\n
+Text Notes 2875 5950 2    79   ~ 0
+Mount Designators\n
 Wire Notes Line
 	2900 8100 2900 4950
@@
 	500  8100 6800 8100
 NoConn ~ 7600 2025
-NoConn ~ 7600 2125
-NoConn ~ 7600 3325
-NoConn ~ 7600 3425
 Wire Notes Line
 	6800 500  6800 11200
@@
 	8000 4350 8100 4350
 Connection ~ 8100 4350
-NoConn ~ 7600 2825
 Text Label 5400 5775 2    50   ~ 0
 VUSB
@@
 NoConn ~ 9800 3325
 NoConn ~ 9800 3425
+$Comp
+L Device:Buzzer BZ1
+U 1 1 5F35DDB2
+P 1075 6775
+F 0 "BZ1" H 1228 6804 50  0000 L CNN
+F 1 "Buzzer" H 1228 6713 50  0000 L CNN
+F 2 "misc:9x5.5mm Buzzer" V 1050 6875 50  0001 C CNN
+F 3 "~" V 1050 6875 50  0001 C CNN
+	1    1075 6775
+	0    -1   -1   0
+$EndComp
+$Comp
+L Device:LED D4
+U 1 1 5F361454
+P 2150 6300
+F 0 "D4" H 2141 6516 50  0000 C CNN
+F 1 "LED" H 2141 6425 50  0000 C CNN
+F 2 "LED_THT:LED_D5.0mm" H 2150 6300 50  0001 C CNN
+F 3 "~" H 2150 6300 50  0001 C CNN
+	1    2150 6300
+	1    0    0    -1
+$EndComp
+$Comp
+L Device:R R19
+U 1 1 5F367A92
+P 2425 6550
+F 0 "R19" H 2495 6596 50  0000 L CNN
+F 1 "R" H 2495 6505 50  0000 L CNN
+F 2 "Resistor_THT:R_Axial_DIN0207_L6.3mm_D2.5mm_P10.16mm_Horizontal" V 2355 6550 50  0001 C CNN
+F 3 "~" H 2425 6550 50  0001 C CNN
+	1    2425 6550
+	1    0    0    -1
+$EndComp
+Text Notes 2875 8025 2    79   ~ 0
+Indicators\n
+Wire Notes Line
+	2900 6000 475  6000
+Wire Wire Line
+	2425 6400 2425 6300
+Wire Wire Line
+	2425 6300 2300 6300
+$Comp
+L Device:LED D5
+U 1 1 5F396452
+P 2150 6825
+F 0 "D5" H 2141 7041 50  0000 C CNN
+F 1 "LED" H 2141 6950 50  0000 C CNN
+F 2 "LED_THT:LED_D5.0mm" H 2150 6825 50  0001 C CNN
+F 3 "~" H 2150 6825 50  0001 C CNN
+	1    2150 6825
+	1    0    0    -1
+$EndComp
+$Comp
+L Device:R R20
+U 1 1 5F396459
+P 2425 7075
+F 0 "R20" H 2495 7121 50  0000 L CNN
+F 1 "R" H 2495 7030 50  0000 L CNN
+F 2 "Resistor_THT:R_Axial_DIN0207_L6.3mm_D2.5mm_P10.16mm_Horizontal" V 2355 7075 50  0001 C CNN
+F 3 "~" H 2425 7075 50  0001 C CNN
+	1    2425 7075
+	1    0    0    -1
+$EndComp
+Wire Wire Line
+	2425 6925 2425 6825
+Wire Wire Line
+	2425 6825 2300 6825
+$Comp
+L Device:LED D6
+U 1 1 5F399A50
+P 2150 7350
+F 0 "D6" H 2141 7566 50  0000 C CNN
+F 1 "LED" H 2141 7475 50  0000 C CNN
+F 2 "LED_THT:LED_D5.0mm" H 2150 7350 50  0001 C CNN
+F 3 "~" H 2150 7350 50  0001 C CNN
+	1    2150 7350
+	1    0    0    -1
+$EndComp
+$Comp
+L Device:R R21
+U 1 1 5F399A57
+P 2425 7600
+F 0 "R21" H 2495 7646 50  0000 L CNN
+F 1 "R" H 2495 7555 50  0000 L CNN
+F 2 "Resistor_THT:R_Axial_DIN0207_L6.3mm_D2.5mm_P10.16mm_Horizontal" V 2355 7600 50  0001 C CNN
+F 3 "~" H 2425 7600 50  0001 C CNN
+	1    2425 7600
+	1    0    0    -1
+$EndComp
+Wire Wire Line
+	2425 7450 2425 7350
+Wire Wire Line
+	2425 7350 2300 7350
+Wire Wire Line
+	2000 6300 1800 6300
+Wire Wire Line
+	1800 6300 1800 6825
+Wire Wire Line
+	2000 7350 1800 7350
+Connection ~ 1800 7350
+Wire Wire Line
+	1800 7350 1800 7725
+Wire Wire Line
+	2000 6825 1800 6825
+Connection ~ 1800 6825
+Wire Wire Line
+	1800 6825 1800 7350
+Text Label 2500 6700 0    50   ~ 0
+LED_1
+Text Label 2500 7225 0    50   ~ 0
+LED_2
+Text Label 2500 7750 0    50   ~ 0
+LED_3
+Wire Wire Line
+	2500 6700 2425 6700
+Wire Wire Line
+	2500 7225 2425 7225
+Wire Wire Line
+	2500 7750 2425 7750
+Text Label 1800 7725 3    50   ~ 0
+GND
+$Comp
+L Device:R R18
+U 1 1 5F3C1532
+P 975 7150
+F 0 "R18" H 905 7104 50  0000 R CNN
+F 1 "R" H 905 7195 50  0000 R CNN
+F 2 "Resistor_THT:R_Axial_DIN0207_L6.3mm_D2.5mm_P10.16mm_Horizontal" V 905 7150 50  0001 C CNN
+F 3 "~" H 975 7150 50  0001 C CNN
+	1    975  7150
+	-1   0    0    1
+$EndComp
+Wire Wire Line
+	975  7000 975  6875
+Text Label 975  7300 3    50   ~ 0
+Buzzer
+Text Label 1350 6975 0    50   ~ 0
+GND
+Wire Wire Line
+	1175 6975 1175 6875
+Wire Wire Line
+	1175 6975 1350 6975
+Text Label 7600 3425 2    50   ~ 0
+LED_3
+Text Label 7600 3325 2    50   ~ 0
+LED_2
+Text Label 7600 2825 2    50   ~ 0
+LED_1
+Text Label 7600 2125 2    50   ~ 0
+Buzzer
 $EndSCHEMATC
