File: pcb_files/mouse/mouse_v2.sch (KiCad schematic (older format))
At the start: 56 parts, among them J4 I2C_Conn, M1 Motor_DC, M2 Motor_DC, Q0 Q_Photo_NPN, Q1 Q_Photo_NPN, Q2 Q_Photo_NPN, Q3 Q_Photo_NPN, T0 Q_NMOS_DGS, T1 Q_NMOS_DGS, T2 Q_NMOS_DGS, T3 Q_NMOS_DGS, U1 Teensy4.0, U2 SN754410NE (Half-Bridge), U3 LM1085-5.0, U4 Encoder_3081, U5 Encoder_3081

Commit message: updated buzzer footprinton pcb
Parts:
- BZ1: footprint misc:9x5.5mm Buzzer -> custom:CST-931AP_buzzer
Changed lines of the file:
@@
 EESchema Schematic File Version 4
-LIBS:mouse_v2-cache
-EELAYER 26 0
+EELAYER 30 0
 EELAYER END
 $Descr A3 16535 11693
@@
 F 0 "BZ1" H 1228 6804 50  0000 L CNN
 F 1 "Buzzer" H 1228 6713 50  0000 L CNN
-F 2 "misc:9x5.5mm Buzzer" V 1050 6875 50  0001 C CNN
+F 2 "custom:CST-931AP_buzzer" V 1050 6875 50  0001 C CNN
 F 3 "~" V 1050 6875 50  0001 C CNN
 	1    1075 6775
